Commit message: Add IMU plugin. Also change organization of lidar and sensor plugins

File: urdf/basic_sensors/lidar/velodyne.xacro (robot description, xacro)
@@ -91,6 +91,6 @@
                     </scan>
                     <range>
-                        <min>${collision_range}</min>
-                        <max>${max_range+1}</max>
+                        <min>${min_range}</min>
+                        <max>${max_range}</max>
                         <resolution>${resolution}</resolution>
                     </range>

File: urdf/basic_sensors/lidar/velodyne16.xacro (robot description, xacro)
@@ -1,5 +1,5 @@
 <robot name="velodyne16" xmlns:xacro="http://ros.org/wiki/xacro">
     <xacro:property name="M_PI" value="3.1415926535897931" />
-    <xacro:include filename="$(find agribot_description)/urdf/basic_sensors/velodyne.xacro"/>
+    <xacro:include filename="$(find agribot_description)/urdf/basic_sensors/lidar/velodyne.xacro"/>
     <xacro:macro    name="velodyne16"
                     params="*origin

File: urdf/basic_sensors/sonar/balluff_sonar.xacro (robot description, xacro)
@@ -1,5 +1,5 @@
 <robot name="balluff_sonar" xmlns:xacro="http://ros.org/wiki/xacro">
     <xacro:property name="M_PI" value="3.1415926535897931" />
-    <xacro:include filename="$(find agribot_description)/urdf/basic_sensors/sonar.xacro"/>
+    <xacro:include filename="$(find agribot_description)/urdf/basic_sensors/sonar/sonar.xacro"/>
     <xacro:macro    name="balluff_sonar"
                     params="*origin

File: urdf/basic_sensors/sonar/bosch_sonar.xacro (robot description, xacro)
@@ -1,5 +1,5 @@
 <robot name="bosch_sonar" xmlns:xacro="http://ros.org/wiki/xacro">
     <xacro:property name="M_PI" value="3.1415926535897931" />
-    <xacro:include filename="$(find agribot_description)/urdf/basic_sensors/sonar.xacro"/>
+    <xacro:include filename="$(find agribot_description)/urdf/basic_sensors/sonar/sonar.xacro"/>
     <xacro:macro    name="bosch_sonar"
                     params="*origin

File: urdf/sensors.xacro (robot description, xacro)
@@ -1,13 +1,9 @@
 <robot name="sensors" xmlns:xacro="http://ros.org/wiki/xacro">
-    <xacro:include filename="$(find agribot_description)/urdf/basic_sensors/velodyne16.xacro"/>
-    <xacro:include filename="$(find agribot_description)/urdf/basic_sensors/bosch_sonar.xacro"/>
-    <xacro:include filename="$(find agribot_description)/urdf/basic_sensors/balluff_sonar.xacro"/>
+    <xacro:include filename="$(find agribot_description)/urdf/basic_sensors/lidar/velodyne16.xacro"/>
+    <xacro:include filename="$(find agribot_description)/urdf/basic_sensors/lidar/benewake_ce30_c.xacro"/>
+    <xacro:include filename="$(find agribot_description)/urdf/basic_sensors/sonar/bosch_sonar.xacro"/>
+    <xacro:include filename="$(find agribot_description)/urdf/basic_sensors/sonar/balluff_sonar.xacro"/>
+    <xacro:include filename="$(find agribot_description)/urdf/basic_sensors/imu/imu.xacro"/>
     <xacro:macro name="agribot_sensors">
-        <link name="imu_link"/>
-        <joint name="imu_joint" type="fixed">
-            <origin xyz="0 0 0" rpy="0 0 0"/>
-            <parent link="chassis_link"/>
-            <child link="imu_link" />
-        </joint>
         <link name="magnetic_link"/>
         <joint name="magnetic_joint" type="fixed">
@@ -28,12 +24,34 @@
             <child link="inclinometer_link" />
         </joint>
-        <!-- <xacro:velodyne16>
-            <origin xyz="1.6 0 1.4" rpy="0 0 0" />
+        <xacro:imu>
+            <origin xyz="1.6 0 1.4" rpy="0 0.2 0" />
+            <xacro:property name="parent"               value="chassis_link"/>
+            <xacro:property name="robot_namespace"      value="agribot"/>
+            <xacro:property name="topic"                value="imu/raw"/>
+            <xacro:property name="name"                 value="imu"/>
+            <xacro:property name="hz"                   value="10.0"/>
+            <xacro:property name="accel_noise"          value="0.001"/>
+            <xacro:property name="gyro_noise"           value="0.001"/>
+            <xacro:property name="yaw_noise"            value="0.05"/>
+            <xacro:property name="yaw_drift"            value="0.01"/>
+            <xacro:property name="yaw_drift_freq"       value="1.0"/>
+        </xacro:imu>
+<!--
+        <xacro:velodyne16>
+            <origin xyz="1.6 0 1.4" rpy="0 0.2 0" />
             <xacro:property name="parent"               value="base_footprint"/>
-            <xacro:property name="topic"                value="/agribot/front_lidar/pc2"/>
-            <xacro:property name="name"                 value="front_lidar"/>
+            <xacro:property name="topic"                value="/agribot/front_lidar/v16/pc2"/>
+            <xacro:property name="name"                 value="front_lidar_v16"/>
             <xacro:property name="hz"                   value="1.0"/>
             <xacro:property name="visualize"            value="false"/>
         </xacro:velodyne16>
+        <xacro:benewake_ce30_c>
+            <origin xyz="1.6 0 1.4" rpy="0 0.4 0" />
+            <xacro:property name="parent"               value="base_footprint"/>
+            <xacro:property name="topic"                value="/agribot/front_lidar/ce30c/pc2"/>
+            <xacro:property name="name"                 value="front_lidar_ce30c"/>
+            <xacro:property name="hz"                   value="1.0"/>
+            <xacro:property name="visualize"            value="false"/>
+        </xacro:benewake_ce30_c>
         <xacro:bosch_sonar>
             <origin xyz="1.6 0.4 1.0" rpy="0 0 0" />
