Commit message: Add GPS+Heading plugin files. Also adjust imu.xacro

File: urdf/basic_sensors/imu/imu.xacro (robot description, xacro)
@@ -22,27 +22,27 @@
         <gazebo>
             <plugin name="imu_controller" filename="libgazebo_imu.so">
-              <updateRate> ${hz} </updateRate>
-              <robotNamespace> ${robot_namespace} </robotNamespace>
-              <bodyName> ${name}_link </bodyName>
-              <frameId> ${name}_link </frameId>
-              <topicName> ${topic} </topicName>
-              <!-- General noise  -->
-              <!-- If 0.0 [accel/rate/yaw]GaussianNoises are used -->
-              <gaussianNoise>0.0</gaussianNoise>
-              <!-- Accelerometer noise -->
-              <accelOffset>0.0 0.0 0.0</accelOffset>
-              <accelDrift>0.0 0.0 0.0</accelDrift>
-              <accelDriftFrequency>0.0 0.0 0.0</accelDriftFrequency>
-              <accelGaussianNoise> ${accel_noise} ${accel_noise} ${accel_noise} </accelGaussianNoise>
-              <!-- Gyroscope noise -->
-              <rateOffset>0.0 0.0 0.0</rateOffset>
-              <rateDrift>0.0 0.0 0.0</rateDrift>
-              <rateDriftFrequency>0.0 0.0 0.0</rateDriftFrequency>
-              <rateGaussianNoise> ${gyro_noise} ${gyro_noise} ${gyro_noise} </rateGaussianNoise>
-              <!-- Yaw noise -->
-              <yawOffset>0.0</yawOffset>
-              <yawDrift> ${yaw_drift} </yawDrift>
-              <yawDriftFrequency> ${yaw_drift_freq} </yawDriftFrequency>
-              <yawGaussianNoise> ${yaw_noise} </yawGaussianNoise>
+                <updateRate> ${hz} </updateRate>
+                <robotNamespace> ${robot_namespace} </robotNamespace>
+                <bodyName> ${name}_link </bodyName>
+                <frameId> ${name}_link </frameId>
+                <topicName> ${topic} </topicName>
+                <!-- General noise  -->
+                <!-- If 0.0 [accel/rate/yaw]GaussianNoises are used -->
+                <gaussianNoise>0.0</gaussianNoise>
+                <!-- Accelerometer noise -->
+                <accelOffset>0.0 0.0 0.0</accelOffset>
+                <accelDrift>0.0 0.0 0.0</accelDrift>
+                <accelDriftFrequency>0.0 0.0 0.0</accelDriftFrequency>
+                <accelGaussianNoise> ${accel_noise} ${accel_noise} ${accel_noise} </accelGaussianNoise>
+                <!-- Gyroscope noise -->
+                <rateOffset>0.0 0.0 0.0</rateOffset>
+                <rateDrift>0.0 0.0 0.0</rateDrift>
+                <rateDriftFrequency>0.0 0.0 0.0</rateDriftFrequency>
+                <rateGaussianNoise> ${gyro_noise} ${gyro_noise} ${gyro_noise} </rateGaussianNoise>
+                <!-- Yaw noise -->
+                <yawOffset>0.0</yawOffset>
+                <yawDrift> ${yaw_drift} </yawDrift>
+                <yawDriftFrequency> ${yaw_drift_freq} </yawDriftFrequency>
+                <yawGaussianNoise> ${yaw_noise} </yawGaussianNoise>
             </plugin>
         </gazebo>

File: urdf/sensors.xacro (robot description, xacro)
@@ -5,4 +5,5 @@
     <xacro:include filename="$(find agribot_description)/urdf/basic_sensors/sonar/balluff_sonar.xacro"/>
     <xacro:include filename="$(find agribot_description)/urdf/basic_sensors/imu/imu.xacro"/>
+    <xacro:include filename="$(find agribot_description)/urdf/basic_sensors/gps/gps.xacro"/>
     <xacro:macro name="agribot_sensors">
         <link name="magnetic_link"/>
@@ -11,10 +12,4 @@
             <parent link="chassis_link"/>
             <child link="magnetic_link" />
-        </joint>
-        <link name="gps_link"/>
-        <joint name="gps_joint" type="fixed">
-            <origin xyz="0 0 0" rpy="0 0 0"/>
-            <parent link="chassis_link"/>
-            <child link="gps_link" />
         </joint>
         <link name="inclinometer_link"/>
@@ -25,5 +20,5 @@
         </joint>
         <xacro:imu>
-            <origin xyz="1.6 0 1.4" rpy="0 0.2 0" />
+            <origin xyz="0 0 0" rpy="0 0 0" />
             <xacro:property name="parent"               value="chassis_link"/>
             <xacro:property name="robot_namespace"      value="agribot"/>
@@ -37,4 +32,24 @@
             <xacro:property name="yaw_drift_freq"       value="1.0"/>
         </xacro:imu>
+        <xacro:gps>
+            <origin xyz="0 0 0" rpy="0 0 0" />
+            <xacro:property name="parent"               value="chassis_link"/>
+            <xacro:property name="robot_namespace"      value="agribot"/>
+            <xacro:property name="topic"                value="gnss"/>
+            <xacro:property name="velocity_topic"       value="fix_velocity"/>
+            <xacro:property name="name"                 value="gps"/>
+            <xacro:property name="hz"                   value="10.0"/>
+            <xacro:property name="noise"                value="0.03"/>
+            <xacro:property name="velocity_noise"       value="0.3"/>
+            <!-- Moderna vineyard coordinates -->
+            <xacro:property name="reference_latitude"   value="51.26662409135839"/>
+            <xacro:property name="reference_longitude"  value="17.20327894189977"/>
+            <xacro:property name="reference_heading"    value="158.5507847682035"/>
+            <xacro:property name="reference_altitude"   value="193.7327916698572"/>
+            <!-- Use heading -->
+            <xacro:property name="publish_heading"      value="true"/>
+            <xacro:property name="heading_topic"        value="heading"/>
+            <xacro:property name="heading_noise"        value="0.01"/>
+        </xacro:gps>
 <!--
         <xacro:velodyne16>
