Commit message: Adjust some noise and config values in sensors.xacro

File: urdf/sensors.xacro (robot description, xacro)
@@ -1,34 +1,4 @@
 <robot name="sensors" xmlns:xacro="http://ros.org/wiki/xacro">
   <xacro:macro name="agribot_sensors">
-    <link name="inclinometer_link"/>
-    <joint name="inclinometer_joint" type="fixed">
-        <parent link="chassis_link"/>
-        <child link="inclinometer_link" />
-        <origin xyz="0 0 0" rpy="0 0 0"/>
-    </joint>
-    <gazebo>
-        <plugin name="inclinometer_controller" filename="libgazebo_inclinometer.so">
-        <updateRate>10.0</updateRate>
-        <robotNamespace>agribot</robotNamespace>
-        <bodyName>inclinometer_link</bodyName>
-        <frameId>inclinometer_link</frameId>
-        <topicName>inclinometer</topicName>
-        <Drift>10.0000000 10.0000000 10.0000000</Drift>
-        <DriftFrequency>10.0000000 10.0000000 10.0000000</DriftFrequency>
-        <GaussianNoise>10.0000000 10.0000000 10.0000000</GaussianNoise>
-        </plugin>
-    </gazebo>
-    <gazebo>
-        <plugin name="heading_controller" filename="libgazebo_heading.so">
-        <updateRate>10.0</updateRate>
-        <robotNamespace>agribot</robotNamespace>
-        <bodyName>gps_link</bodyName>
-        <frameId>gps_link</frameId>
-        <topicName>heading</topicName>
-        <Drift>10.0000000 10.0000000 10.0000000</Drift>
-        <DriftFrequency>10.0000000 10.0000000 10.0000000</DriftFrequency>
-        <GaussianNoise>10.0000000 10.0000000 10.0000000</GaussianNoise>
-        </plugin>
-    </gazebo>
     <link name="imu_link"/>
     <joint name="imu_joint" type="fixed">
@@ -38,26 +8,52 @@
     </joint>
     <gazebo>
-        <plugin name="imu_cotroller" filename="libgazebo_imu.so">
-        <updateRate>10</updateRate>
-        <robotNamespace>agribot</robotNamespace>
-        <bodyName>imu_link</bodyName>
-        <frameId>imu_link</frameId>
-        <topicName>imu</topicName>
-        <rpyOffset>0 0 0</rpyOffset>
-        <xyzOffset>0 0 0</xyzOffset>
-        <!-- <gaussianNoise>0.00000001</gaussianNoise>
-        <accelDrift>0.00000001 0.00000001 0.00000001</accelDrift>
-        <accelDriftFrequency>0.00000001 0.00000001 0.00000001</accelDriftFrequency>
-        <accelGaussianNoise>0.00000001 0.00000001 0.00000001</accelGaussianNoise> -->
-        <gaussianNoise>10.0000000</gaussianNoise>
-        <accelDrift>10.0000000 10.0000000 10.0000000</accelDrift>
-        <accelDriftFrequency>10.0000000 10.0000000 10.0000000</accelDriftFrequency>
-        <accelGaussianNoise>10.0000000 10.0000000 10.0000000</accelGaussianNoise>
-        <rateDrift>10.0 10.0 10.0</rateDrift>
-        <rateDriftFrequency>10.0 10.0 10.0</rateDriftFrequency>
-        <rateGaussianNoise>10.0 10.0 10.0</rateGaussianNoise>
-        <headingDrift>10.0 10.0 10.0</headingDrift>
-        <headingDriftFrequency>10.0 10.0 10.0</headingDriftFrequency>
-        <headingGaussianNoise>10.0 10.0 10.0</headingGaussianNoise>
+        <plugin name="imu_controller" filename="libgazebo_imu.so">
+          <updateRate>10.0</updateRate>
+          <robotNamespace>agribot</robotNamespace>
+          <bodyName>imu_link</bodyName>
+          <frameId>imu_link</frameId>
+          <topicName>imu/raw</topicName>
+          <!-- General noise  -->
+          <!-- If 0.0 [accel/rate/yaw]GaussianNoises are used -->
+          <gaussianNoise>0.0</gaussianNoise>
+          <!-- Accelerometer noise -->
+          <accelOffset>0.0 0.0 0.0</accelOffset>
+          <accelDrift>0.0 0.0 0.0</accelDrift>
+          <accelDriftFrequency>0.0 0.0 0.0</accelDriftFrequency>
+          <accelGaussianNoise>0.001 0.001 0.001</accelGaussianNoise>
+          <!-- Gyroscope noise -->
+          <rateOffset>0.0 0.0 0.0</rateOffset>
+          <rateDrift>0.0 0.0 0.0</rateDrift>
+          <rateDriftFrequency>0.0 0.0 0.0</rateDriftFrequency>
+          <rateGaussianNoise>0.01 0.01 0.01</rateGaussianNoise>
+          <!-- Yaw noise -->
+          <yawOffset>0.0</yawOffset>
+          <yawDrift>0.01</yawDrift>
+          <yawDriftFrequency>1.0</yawDriftFrequency>
+          <yawGaussianNoise>0.9</yawGaussianNoise>
+        </plugin>
+    </gazebo>
+    <link name="magnetic_link"/>
+    <joint name="magnetic_joint" type="fixed">
+        <parent link="chassis_link"/>
+        <child link="magnetic_link" />
+        <origin xyz="0 0 0" rpy="0 0 0"/>
+    </joint>
+    <gazebo>
+        <plugin name="magnetic_controller" filename="libgazebo_magnetic.so">
+          <updateRate>10.0</updateRate>
+          <robotNamespace>agribot</robotNamespace>
+          <bodyName>imu_link</bodyName>
+          <topicName>magnetic_field</topicName>
+          <!-- Magnetometer setup -->
+          <magnitude>1.0</magnitude>
+          <referenceHeading>0.0</referenceHeading>
+          <declination>0.0</declination>
+          <inclination>60.0</inclination>
+          <!-- Magnetometer noise -->
+          <offset>0.0 0.0 0.0</offset>
+          <drift>0.0 0.0 0.0</drift>
+          <driftFrequency>0.0 0.0 0.0</driftFrequency>
+          <gaussianNoise>0.01 0.01 0.01</gaussianNoise>
         </plugin>
     </gazebo>
@@ -70,39 +66,60 @@
     <gazebo>
         <plugin name="gps_controller" filename="libgazebo_gps.so">
-        <updateRate>10.0</updateRate>
-        <robotNamespace>agribot</robotNamespace>
-        <bodyName>gps_link</bodyName>
-        <frameId>gps_link</frameId>
-        <topicName>gnss</topicName>
-        <velocityTopicName>fix_velocity</velocityTopicName>
-        <!-- <drift>5.0 5.0 5.0</drift>
-        <gaussianNoise>0.1 0.1 0.1</gaussianNoise>
-        <velocityDrift>0 0 0</velocityDrift>
-        <velocityGaussianNoise>0.1 0.1 0.1</velocityGaussianNoise> -->
-        <drift>10.0 10.0 10.0</drift>
-        <gaussianNoise>10.0 10.0 10.0</gaussianNoise>
-        <velocityDrift>10 10 10</velocityDrift>
-        <velocityGaussianNoise>10.0 10.0 10.0</velocityGaussianNoise>
+          <updateRate>10.0</updateRate>
+          <robotNamespace>agribot</robotNamespace>
+          <bodyName>gps_link</bodyName>
+          <frameId>gps_link</frameId>
+          <topicName>gnss</topicName>
+          <velocityTopicName>fix_velocity</velocityTopicName>
+          <!-- Reference values -->
+          <referenceLatitude>49.9</referenceLatitude>
+          <referenceLongitude>8.9</referenceLongitude>
+          <referenceHeading>0.0</referenceHeading>
+          <referenceAltitude>0.0</referenceAltitude>
+          <!-- GPS noise -->
+          <offset>0.0 0.0 0.0</offset>
+          <gaussianNoise>2.0 2.0 2.0</gaussianNoise>
+          <drift>0.0 0.0 0.0</drift>
+          <driftFrequency>0.0 0.0 0.0</driftFrequency>
+          <!-- Velocity noise -->
+          <velocityOffset>0.0 0.0 0.0</velocityOffset>
+          <velocityGaussianNoise>0.5 0.5 0.5</velocityGaussianNoise>
+          <velocityDrift>0.0 0.0 0.0</velocityDrift>
+          <velocityDriftFrequency>0.0 0.0 0.0</velocityDriftFrequency>
+          <!-- Flags -->
+          <status>STATUS_FIX</status>
+          <service>SERVICE_GPS</service>
         </plugin>
     </gazebo>
-    <link name="magnetic_link"/>
-    <joint name="magnetic_joint" type="fixed">
+    <gazebo>
+        <plugin name="heading_controller" filename="libgazebo_heading.so">
+          <updateRate>10.0</updateRate>
+          <robotNamespace>agribot</robotNamespace>
+          <bodyName>gps_link</bodyName>
+          <frameId>gps_link</frameId>
+          <topicName>heading</topicName>
+          <!-- Heading noise -->
+          <Drift>0.0 0.0 0.0</Drift>
+          <DriftFrequency>0.0 0.0 0.0</DriftFrequency>
+          <GaussianNoise>0.01 0.01 0.01</GaussianNoise>
+        </plugin>
+    </gazebo>
+    <link name="inclinometer_link"/>
+    <joint name="inclinometer_joint" type="fixed">
         <parent link="chassis_link"/>
-        <child link="magnetic_link" />
+        <child link="inclinometer_link" />
         <origin xyz="0 0 0" rpy="0 0 0"/>
     </joint>
     <gazebo>
-        <plugin name="magnetic_controller" filename="libgazebo_magnetic.so">
-        <updateRate>10.0</updateRate>
-        <robotNamespace>agribot</robotNamespace>
-        <bodyName>magnetic_link</bodyName>
-        <topicName>magnetic_field</topicName>
-        <!-- <drift>5.0 5.0 5.0</drift>
-        <gaussianNoise>0.1 0.1 0.1</gaussianNoise>
-        <velocityDrift>0 0 0</velocityDrift>
-        <velocityGaussianNoise>0.1 0.1 0.1</velocityGaussianNoise> -->
-        <Drift>10.0000000 10.0000000 10.0000000</Drift>
-        <DriftFrequency>10.0000000 10.0000000 10.0000000</DriftFrequency>
-        <GaussianNoise>10.0000000 10.0000000 10.0000000</GaussianNoise>
+        <plugin name="inclinometer_controller" filename="libgazebo_inclinometer.so">
+          <updateRate>10.0</updateRate>
+          <robotNamespace>agribot</robotNamespace>
+          <bodyName>inclinometer_link</bodyName>
+          <frameId>inclinometer_link</frameId>
+          <topicName>inclinometer</topicName>
+          <!-- Inclinometer noise -->
+          <Drift>0.0 0.0 0.0</Drift>
+          <DriftFrequency>0.0 0.0 0.0</DriftFrequency>
+          <GaussianNoise>0.01 0.01 0.01</GaussianNoise>
         </plugin>
     </gazebo>

Commit message: Update simulation parameters of sensors

File: urdf/sensors.xacro (robot description, xacro)
@@ -26,10 +26,10 @@
           <rateDrift>0.0 0.0 0.0</rateDrift>
           <rateDriftFrequency>0.0 0.0 0.0</rateDriftFrequency>
-          <rateGaussianNoise>0.01 0.01 0.01</rateGaussianNoise>
+          <rateGaussianNoise>0.001 0.001 0.001</rateGaussianNoise>
           <!-- Yaw noise -->
           <yawOffset>0.0</yawOffset>
           <yawDrift>0.01</yawDrift>
           <yawDriftFrequency>1.0</yawDriftFrequency>
-          <yawGaussianNoise>0.9</yawGaussianNoise>
+          <yawGaussianNoise>0.05</yawGaussianNoise>
         </plugin>
     </gazebo>
@@ -38,4 +38,5 @@
         <parent link="chassis_link"/>
         <child link="magnetic_link" />
+        <!-- <origin xyz="0 0 0" rpy="0 0 3.14159265"/> -->
         <origin xyz="0 0 0" rpy="0 0 0"/>
     </joint>
@@ -44,16 +45,18 @@
           <updateRate>10.0</updateRate>
           <robotNamespace>agribot</robotNamespace>
-          <bodyName>imu_link</bodyName>
+          <bodyName>magnetic_link</bodyName>
+          <frameId>magnetic_link</frameId>
           <topicName>magnetic_field</topicName>
           <!-- Magnetometer setup -->
           <magnitude>1.0</magnitude>
           <referenceHeading>0.0</referenceHeading>
-          <declination>0.0</declination>
-          <inclination>60.0</inclination>
+          <!-- Parking Drzewna -->
+          <declination>5.0741</declination>
+          <inclination>67.0937</inclination>
           <!-- Magnetometer noise -->
           <offset>0.0 0.0 0.0</offset>
           <drift>0.0 0.0 0.0</drift>
           <driftFrequency>0.0 0.0 0.0</driftFrequency>
-          <gaussianNoise>0.01 0.01 0.01</gaussianNoise>
+          <gaussianNoise>1.1e-14 1.1e-14 1.1e-14</gaussianNoise>
         </plugin>
     </gazebo>
@@ -73,16 +76,17 @@
           <velocityTopicName>fix_velocity</velocityTopicName>
           <!-- Reference values -->
-          <referenceLatitude>49.9</referenceLatitude>
-          <referenceLongitude>8.9</referenceLongitude>
+          <!-- Parking Drzewna -->
+          <referenceLatitude>51.113448886283525</referenceLatitude>
+          <referenceLongitude>17.019922397662153</referenceLongitude>
           <referenceHeading>0.0</referenceHeading>
           <referenceAltitude>0.0</referenceAltitude>
           <!-- GPS noise -->
           <offset>0.0 0.0 0.0</offset>
-          <gaussianNoise>2.0 2.0 2.0</gaussianNoise>
+          <gaussianNoise>0.03 0.03 0.03</gaussianNoise>
           <drift>0.0 0.0 0.0</drift>
           <driftFrequency>0.0 0.0 0.0</driftFrequency>
           <!-- Velocity noise -->
           <velocityOffset>0.0 0.0 0.0</velocityOffset>
-          <velocityGaussianNoise>0.5 0.5 0.5</velocityGaussianNoise>
+          <velocityGaussianNoise>0.3 0.3 0.3</velocityGaussianNoise>
           <velocityDrift>0.0 0.0 0.0</velocityDrift>
           <velocityDriftFrequency>0.0 0.0 0.0</velocityDriftFrequency>

Commit message: Add basic velodyne and sonar templates. Also add derived velodyne16, balluff_sonar and bosch_sonar templates

File: urdf/sensors.xacro (robot description, xacro)
@@ -1,29 +1,55 @@
 <robot name="sensors" xmlns:xacro="http://ros.org/wiki/xacro">
-  <xacro:macro name="agribot_sensors">
-    <link name="imu_link"/>
-    <joint name="imu_joint" type="fixed">
-        <parent link="chassis_link"/>
-        <child link="imu_link" />
-        <origin xyz="0 0 0" rpy="0 0 0"/>
-    </joint>
-    <link name="magnetic_link"/>
-    <joint name="magnetic_joint" type="fixed">
-        <parent link="chassis_link"/>
-        <child link="magnetic_link" />
-        <!-- <origin xyz="0 0 0" rpy="0 0 3.14159265"/> -->
-        <origin xyz="0 0 0" rpy="0 0 0"/>
-    </joint>
-    <link name="gps_link"/>
-    <joint name="gps_joint" type="fixed">
-        <parent link="chassis_link"/>
-        <child link="gps_link" />
-        <origin xyz="0 0 0" rpy="0 0 0"/>
-    </joint>
-    <link name="inclinometer_link"/>
-    <joint name="inclinometer_joint" type="fixed">
-        <parent link="chassis_link"/>
-        <child link="inclinometer_link" />
-        <origin xyz="0 0 0" rpy="0 0 0"/>
-    </joint>
-  </xacro:macro>
+    <xacro:include filename="$(find agribot_description)/urdf/basic_sensors/velodyne16.xacro"/>
+    <xacro:include filename="$(find agribot_description)/urdf/basic_sensors/bosch_sonar.xacro"/>
+    <xacro:include filename="$(find agribot_description)/urdf/basic_sensors/balluff_sonar.xacro"/>
+    <xacro:macro name="agribot_sensors">
+        <link name="imu_link"/>
+        <joint name="imu_joint" type="fixed">
+            <origin xyz="0 0 0" rpy="0 0 0"/>
+            <parent link="chassis_link"/>
+            <child link="imu_link" />
+        </joint>
+        <link name="magnetic_link"/>
+        <joint name="magnetic_joint" type="fixed">
+            <origin xyz="0 0 0" rpy="0 0 0"/>
+            <parent link="chassis_link"/>
+            <child link="magnetic_link" />
+        </joint>
+        <link name="gps_link"/>
+        <joint name="gps_joint" type="fixed">
+            <origin xyz="0 0 0" rpy="0 0 0"/>
+            <parent link="chassis_link"/>
+            <child link="gps_link" />
+        </joint>
+        <link name="inclinometer_link"/>
+        <joint name="inclinometer_joint" type="fixed">
+            <origin xyz="0 0 0" rpy="0 0 0"/>
+            <parent link="chassis_link"/>
+            <child link="inclinometer_link" />
+        </joint>
+        <xacro:velodyne16>
+            <origin xyz="1.6 0 1.4" rpy="0 0 0" />
+            <xacro:property name="parent"               value="base_footprint"/>
+            <xacro:property name="topic"                value="/agribot/front_lidar/pc2"/>
+            <xacro:property name="name"                 value="front_lidar"/>
+            <xacro:property name="hz"                   value="1.0"/>
+            <xacro:property name="visualize"            value="false"/>
+        </xacro:velodyne16>
+        <xacro:bosch_sonar>
+            <origin xyz="1.6 0.4 1.0" rpy="0 0 0" />
+            <xacro:property name="parent"               value="base_footprint"/>
+            <xacro:property name="topic"                value="/agribot/front_left_sonar"/>
+            <xacro:property name="name"                 value="front_left_sonar"/>
+            <xacro:property name="hz"                   value="10.0"/>
+            <xacro:property name="visualize"            value="false"/>
+        </xacro:bosch_sonar>
+        <xacro:balluff_sonar>
+            <origin xyz="1.6 -0.4 1.0" rpy="0 0 0" />
+            <xacro:property name="parent"               value="base_footprint"/>
+            <xacro:property name="topic"                value="/agribot/front_right_sonar"/>
+            <xacro:property name="name"                 value="front_right_sonar"/>
+            <xacro:property name="hz"                   value="10.0"/>
+            <xacro:property name="visualize"            value="false"/>
+        </xacro:balluff_sonar>
+    </xacro:macro>
 </robot>

Commit message: Add inclinometer plugin files

File: urdf/sensors.xacro (robot description, xacro)
@@ -6,4 +6,5 @@
     <xacro:include filename="$(find agribot_description)/urdf/basic_sensors/imu/imu.xacro"/>
     <xacro:include filename="$(find agribot_description)/urdf/basic_sensors/gps/gps.xacro"/>
+    <xacro:include filename="$(find agribot_description)/urdf/basic_sensors/inclinometer/inclinometer.xacro"/>
     <xacro:macro name="agribot_sensors">
         <link name="magnetic_link"/>
@@ -12,10 +13,4 @@
             <parent link="chassis_link"/>
             <child link="magnetic_link" />
-        </joint>
-        <link name="inclinometer_link"/>
-        <joint name="inclinometer_joint" type="fixed">
-            <origin xyz="0 0 0" rpy="0 0 0"/>
-            <parent link="chassis_link"/>
-            <child link="inclinometer_link" />
         </joint>
         <xacro:imu>
@@ -52,4 +47,13 @@
             <xacro:property name="heading_noise"        value="0.01"/>
         </xacro:gps>
+        <xacro:inclinometer>
+            <origin xyz="0 0 0" rpy="0 0 0" />
+            <xacro:property name="parent"               value="chassis_link"/>
+            <xacro:property name="robot_namespace"      value="agribot"/>
+            <xacro:property name="topic"                value="inclinometer"/>
+            <xacro:property name="name"                 value="inclinometer"/>
+            <xacro:property name="hz"                   value="10.0"/>
+            <xacro:property name="noise"                value="0.01"/>
+        </xacro:inclinometer>
 <!--
         <xacro:velodyne16>

Commit message: Add magnetometer plugin files

File: urdf/sensors.xacro (robot description, xacro)
@@ -7,11 +7,6 @@
     <xacro:include filename="$(find agribot_description)/urdf/basic_sensors/gps/gps.xacro"/>
     <xacro:include filename="$(find agribot_description)/urdf/basic_sensors/inclinometer/inclinometer.xacro"/>
+    <xacro:include filename="$(find agribot_description)/urdf/basic_sensors/magnetometer/magnetometer.xacro"/>
     <xacro:macro name="agribot_sensors">
-        <link name="magnetic_link"/>
-        <joint name="magnetic_joint" type="fixed">
-            <origin xyz="0 0 0" rpy="0 0 0"/>
-            <parent link="chassis_link"/>
-            <child link="magnetic_link" />
-        </joint>
         <xacro:imu>
             <origin xyz="0 0 0" rpy="0 0 0" />
@@ -56,4 +51,19 @@
             <xacro:property name="noise"                value="0.01"/>
         </xacro:inclinometer>
+        <xacro:magnetometer>
+            <origin xyz="0 0 0" rpy="0 0 0" />
+            <xacro:property name="parent"               value="chassis_link"/>
+            <xacro:property name="robot_namespace"      value="agribot"/>
+            <xacro:property name="topic"                value="magnetic_field"/>
+            <xacro:property name="name"                 value="magnetometer"/>
+            <xacro:property name="hz"                   value="10.0"/>
+            <xacro:property name="magnitude"            value="1.0"/>
+            <xacro:property name="reference_heading"    value="158.5507847682035"/>
+            <xacro:property name="declination"          value="5.0741"/>
+            <xacro:property name="inclination"          value="67.0937"/>
+            <xacro:property name="noise"                value="1.1e-14"/>
+            <!-- <xacro:property name="noise"                value="1.1e-8"/> -->
+            <!-- <xacro:property name="noise"                value="1.1e-5"/> -->
+        </xacro:magnetometer>
 <!--
         <xacro:velodyne16>

Commit message: Add separate xacro file for perception sensors

File: urdf/sensors.xacro (robot description, xacro)
@@ -1,7 +1,4 @@
 <robot name="sensors" xmlns:xacro="http://ros.org/wiki/xacro">
-    <xacro:include filename="$(find agribot_description)/urdf/basic_sensors/lidar/velodyne16.xacro"/>
-    <xacro:include filename="$(find agribot_description)/urdf/basic_sensors/lidar/benewake_ce30_c.xacro"/>
-    <xacro:include filename="$(find agribot_description)/urdf/basic_sensors/sonar/bosch_sonar.xacro"/>
-    <xacro:include filename="$(find agribot_description)/urdf/basic_sensors/sonar/balluff_sonar.xacro"/>
+    <xacro:include filename="$(find agribot_description)/urdf/perception_sensors.xacro"/>
     <xacro:include filename="$(find agribot_description)/urdf/basic_sensors/imu/imu.xacro"/>
     <xacro:include filename="$(find agribot_description)/urdf/basic_sensors/gps/gps.xacro"/>
@@ -66,37 +63,6 @@
             <!-- <xacro:property name="noise"                value="1.1e-5"/> -->
         </xacro:magnetometer>
-<!--
-        <xacro:velodyne16>
-            <origin xyz="1.6 0 1.4" rpy="0 0.2 0" />
-            <xacro:property name="parent"               value="base_footprint"/>
-            <xacro:property name="topic"                value="/agribot/front_lidar/v16/pc2"/>
-            <xacro:property name="name"                 value="front_lidar_v16"/>
-            <xacro:property name="hz"                   value="1.0"/>
-            <xacro:property name="visualize"            value="false"/>
-        </xacro:velodyne16>
-        <xacro:benewake_ce30_c>
-            <origin xyz="1.6 0 1.4" rpy="0 0.4 0" />
-            <xacro:property name="parent"               value="base_footprint"/>
-            <xacro:property name="topic"                value="/agribot/front_lidar/ce30c/pc2"/>
-            <xacro:property name="name"                 value="front_lidar_ce30c"/>
-            <xacro:property name="hz"                   value="1.0"/>
-            <xacro:property name="visualize"            value="false"/>
-        </xacro:benewake_ce30_c>
-        <xacro:bosch_sonar>
-            <origin xyz="1.6 0.4 1.0" rpy="0 0 0" />
-            <xacro:property name="parent"               value="base_footprint"/>
-            <xacro:property name="topic"                value="/agribot/front_left_sonar"/>
-            <xacro:property name="name"                 value="front_left_sonar"/>
-            <xacro:property name="hz"                   value="10.0"/>
-            <xacro:property name="visualize"            value="false"/>
-        </xacro:bosch_sonar>
-        <xacro:balluff_sonar>
-            <origin xyz="1.6 -0.4 1.0" rpy="0 0 0" />
-            <xacro:property name="parent"               value="base_footprint"/>
-            <xacro:property name="topic"                value="/agribot/front_right_sonar"/>
-            <xacro:property name="name"                 value="front_right_sonar"/>
-            <xacro:property name="hz"                   value="10.0"/>
-            <xacro:property name="visualize"            value="false"/>
-        </xacro:balluff_sonar> -->
+        <!-- Add perception sensors -->
+        <!-- <xacro:perception_sensors /> -->
     </xacro:macro>
 </robot>
