Commit message: Chagned topic to service

File: urdf/tools_sensors.xacro (robot description, xacro)
@@ -6,5 +6,5 @@
         <xacro:property name="parent"               value="chassis_link"/>
         <xacro:property name="robot_namespace"      value="agribot"/>
-        <xacro:property name="topic"                value="rfid/tags"/>
+        <xacro:property name="service"              value="tags"/>
         <xacro:property name="name"                 value="rfid"/>
       </xacro:rfid>

File: urdf/tools_sensors/rfid/rfid.xacro (robot description, xacro)
@@ -5,5 +5,5 @@
                           name:=^
                           robot_namespace:=^
-                          topic:=^
+                          service:=^
                           ">
         <joint name="${name}_joint" type="fixed">
@@ -18,5 +18,5 @@
                 <bodyName> ${name}_link </bodyName>
                 <frameId> ${name}_link </frameId>
-                <topicName> ${topic} </topicName>
+                <serviceName> ${service} </serviceName>
             </plugin>
         </gazebo>
