Commit message: Replace old imu plugin with new (imu_sensor.xacro)

File: urdf/basic_sensors.xacro (robot description, xacro)
@@ -1,4 +1,4 @@
 <robot name="sensors" xmlns:xacro="http://ros.org/wiki/xacro">
-    <xacro:include filename="$(find agribot_description)/urdf/basic_sensors/imu/imu.xacro"/>
+    <xacro:include filename="$(find agribot_description)/urdf/basic_sensors/imu/imu_sensor.xacro"/>
     <xacro:include filename="$(find agribot_description)/urdf/basic_sensors/gps/gps.xacro"/>
     <xacro:include filename="$(find agribot_description)/urdf/basic_sensors/inclinometer/inclinometer.xacro"/>
@@ -10,17 +10,13 @@
         <xacro:property name="reference_heading"    value="158.5507847682035"/>
         <xacro:property name="reference_altitude"   value="193.7327916698572"/>
-        <xacro:imu>
+        <xacro:imu_sensor>
             <origin xyz="0 0 0" rpy="0 0 0" />
             <xacro:property name="parent"               value="chassis_link"/>
-            <xacro:property name="robot_namespace"      value="agribot"/>
-            <xacro:property name="topic"                value="imu/raw"/>
+            <xacro:property name="topic"                value="agribot/imu/raw"/>
             <xacro:property name="name"                 value="imu"/>
             <xacro:property name="hz"                   value="10.0"/>
-            <xacro:property name="accel_noise"          value="0.001"/>
-            <xacro:property name="gyro_noise"           value="0.001"/>
-            <xacro:property name="yaw_noise"            value="0.05"/>
-            <xacro:property name="yaw_drift"            value="0.01"/>
-            <xacro:property name="yaw_drift_freq"       value="1.0"/>
-        </xacro:imu>
+            <xacro:property name="accel_noise"          value="0.0"/>
+            <xacro:property name="gyro_noise"           value="0.0"/>
+        </xacro:imu_sensor>
         <xacro:gps>
             <origin xyz="0 0 0" rpy="0 0 0" />

File: urdf/basic_sensors/imu/legacy_imu.xacro (robot description, xacro)
@@ -1,5 +1,5 @@
-<robot name="imu" xmlns:xacro="http://www.ros.org/wiki/xacro">
+<robot name="legacy_imu" xmlns:xacro="http://www.ros.org/wiki/xacro">
     <!-- Basic sonar macro  -->
-    <xacro:macro  name="imu"
+    <xacro:macro  name="legacy_imu"
                   params="*origin
                           parent:=^

Commit message: Change magnetometer plugin settings

File: urdf/basic_sensors.xacro (robot description, xacro)
@@ -10,4 +10,7 @@
         <xacro:property name="reference_heading"    value="158.5507847682035"/>
         <xacro:property name="reference_altitude"   value="193.7327916698572"/>
+        <!-- Magnetometer simulation plugin -->
+        <xacro:property name="declination"   value="-5.2809"/>
+        <xacro:property name="inclination"   value="-67.2494"/>
         <xacro:imu_sensor>
             <origin xyz="0 0 0" rpy="0 0 0" />
@@ -50,10 +53,6 @@
             <xacro:property name="name"                 value="magnetometer"/>
             <xacro:property name="hz"                   value="10.0"/>
-            <xacro:property name="magnitude"            value="1.0"/>
-            <xacro:property name="declination"          value="5.0741"/>
-            <xacro:property name="inclination"          value="67.0937"/>
-            <xacro:property name="noise"                value="1.1e-14"/>
-            <!-- <xacro:property name="noise"                value="1.1e-8"/> -->
-            <!-- <xacro:property name="noise"                value="1.1e-5"/> -->
+            <xacro:property name="magnitude"            value="4.97604e-5"/>
+            <xacro:property name="noise"                value="3.2e-7"/>
         </xacro:magnetometer>
     </xacro:macro>

Commit message: Move inclination and declination parameters to environmental variables

File: urdf/basic_sensors.xacro (robot description, xacro)
@@ -5,4 +5,6 @@
     <xacro:include filename="$(find agribot_description)/urdf/basic_sensors/magnetometer/magnetometer.xacro"/>
     <xacro:macro name="basic_sensors">
+        <!-- NOTE: Simulation properties are passed in robot_description.xml file -->
+        <!-- Position on earth -->
         <xacro:property name="reference_latitude"   value="$(arg simulation_latitude)"/>
         <xacro:property name="reference_longitude"  value="$(arg simulation_longitude)"/>
@@ -10,6 +12,6 @@
         <xacro:property name="reference_altitude"   value="$(arg simulation_altitude)"/>
         <!-- Magnetometer simulation plugin -->
-        <xacro:property name="declination"   value="-5.2809"/>
-        <xacro:property name="inclination"   value="-67.2494"/>
+        <xacro:property name="declination"   value="$(arg simulation_declination)"/>
+        <xacro:property name="inclination"   value="$(arg simulation_inclination)"/>
         <xacro:imu_sensor>
             <origin xyz="0 0 0" rpy="0 0 0" />

Commit message: Move sensor simulation parameters to config repo

File: urdf/basic_sensors.xacro (robot description, xacro)
@@ -6,5 +6,5 @@
     <xacro:macro name="basic_sensors">
         <!-- NOTE: Simulation properties are passed in robot_description.xml file -->
-        <!-- Position on earth -->
+        <!-- Position on Earth -->
         <xacro:property name="reference_latitude"   value="$(arg simulation_latitude)"/>
         <xacro:property name="reference_longitude"  value="$(arg simulation_longitude)"/>
@@ -20,6 +20,6 @@
             <xacro:property name="name"                 value="imu"/>
             <xacro:property name="hz"                   value="10.0"/>
-            <xacro:property name="accel_noise"          value="0.0"/>
-            <xacro:property name="gyro_noise"           value="0.0"/>
+            <xacro:property name="accel_noise"          value="$(arg simulation_accelerometer_noise)"/>
+            <xacro:property name="gyro_noise"           value="$(arg simulation_gyroscope_noise)"/>
         </xacro:imu_sensor>
         <xacro:gps>
@@ -31,10 +31,10 @@
             <xacro:property name="name"                 value="gps"/>
             <xacro:property name="hz"                   value="10.0"/>
-            <xacro:property name="noise"                value="0.03"/>
-            <xacro:property name="velocity_noise"       value="0.3"/>
+            <xacro:property name="noise"                value="$(arg simulation_gps_noise)"/>
+            <xacro:property name="velocity_noise"       value="$(arg simulation_gps_velocity_noise)"/>
             <!-- Use heading -->
-            <xacro:property name="publish_heading"      value="true"/>
+            <xacro:property name="publish_heading"      value="$(arg simulation_gps_publish_heading)"/>
             <xacro:property name="heading_topic"        value="heading"/>
-            <xacro:property name="heading_noise"        value="0.01"/>
+            <xacro:property name="heading_noise"        value="$(arg simulation_gps_heading_noise)"/>
         </xacro:gps>
         <xacro:inclinometer>
@@ -45,5 +45,5 @@
             <xacro:property name="name"                 value="inclinometer"/>
             <xacro:property name="hz"                   value="10.0"/>
-            <xacro:property name="noise"                value="0.01"/>
+            <xacro:property name="noise"                value="$(arg simulation_inclinometer_noise)"/>
         </xacro:inclinometer>
         <xacro:magnetometer>
@@ -54,6 +54,6 @@
             <xacro:property name="name"                 value="magnetometer"/>
             <xacro:property name="hz"                   value="10.0"/>
-            <xacro:property name="magnitude"            value="4.97604e-5"/>
-            <xacro:property name="noise"                value="3.2e-7"/>
+            <xacro:property name="magnitude"            value="$(arg simulation_magnetometer_magnitude)"/>
+            <xacro:property name="noise"                value="$(arg simulation_magnetometer_noise)"/>
         </xacro:magnetometer>
     </xacro:macro>

Commit message: Change IMU and magnetometer topics for use with imu_transformer

File: urdf/basic_sensors.xacro (robot description, xacro)
@@ -17,5 +17,5 @@
             <origin xyz="0 0 0" rpy="0 0 0" />
             <xacro:property name="parent"               value="chassis_link"/>
-            <xacro:property name="topic"                value="agribot/imu/raw"/>
+            <xacro:property name="topic"                value="/agribot/imu/raw/data"/>
             <xacro:property name="name"                 value="imu"/>
             <xacro:property name="hz"                   value="10.0"/>
@@ -51,5 +51,5 @@
             <xacro:property name="parent"               value="chassis_link"/>
             <xacro:property name="robot_namespace"      value="agribot"/>
-            <xacro:property name="topic"                value="magnetic_field"/>
+            <xacro:property name="topic"                value="imu/raw/mag"/>
             <xacro:property name="name"                 value="magnetometer"/>
             <xacro:property name="hz"                   value="10.0"/>

Commit message: Rotate IMU tf

File: urdf/basic_sensors.xacro (robot description, xacro)
@@ -15,5 +15,5 @@
         <xacro:property name="inclination"   value="$(arg simulation_inclination)"/>
         <xacro:imu_sensor>
-            <origin xyz="0 0 0" rpy="0 0 0" />
+            <origin xyz="0 0 0" rpy="0 0 ${M_PI/2}" />
             <xacro:property name="parent"               value="chassis_link"/>
             <xacro:property name="topic"                value="/agribot/imu/raw/data"/>

Commit message: Change direction of imu_link rotation

File: urdf/basic_sensors.xacro (robot description, xacro)
@@ -15,5 +15,5 @@
         <xacro:property name="inclination"   value="$(arg simulation_inclination)"/>
         <xacro:imu_sensor>
-            <origin xyz="0 0 0" rpy="0 0 ${M_PI/2}" />
+            <origin xyz="0 0 0" rpy="0 0 ${-M_PI/2}" />
             <xacro:property name="parent"               value="chassis_link"/>
             <xacro:property name="topic"                value="/agribot/imu/raw/data"/>

Commit message: Rotate magnetometer frame

File: urdf/basic_sensors.xacro (robot description, xacro)
@@ -48,5 +48,5 @@
         </xacro:inclinometer>
         <xacro:magnetometer>
-            <origin xyz="0 0 0" rpy="0 0 0" />
+            <origin xyz="0 0 0" rpy="0 0 ${-M_PI/2}" />
             <xacro:property name="parent"               value="chassis_link"/>
             <xacro:property name="robot_namespace"      value="agribot"/>

Commit message: Change direction of rotation for imu and magnetometer links

File: urdf/basic_sensors.xacro (robot description, xacro)
@@ -15,5 +15,5 @@
         <xacro:property name="inclination"   value="$(arg simulation_inclination)"/>
         <xacro:imu_sensor>
-            <origin xyz="0 0 0" rpy="0 0 ${-M_PI/2}" />
+            <origin xyz="0 0 0" rpy="0 0 ${M_PI/2}" />
             <xacro:property name="parent"               value="chassis_link"/>
             <xacro:property name="topic"                value="/agribot/imu/raw/data"/>
@@ -48,5 +48,5 @@
         </xacro:inclinometer>
         <xacro:magnetometer>
-            <origin xyz="0 0 0" rpy="0 0 ${-M_PI/2}" />
+            <origin xyz="0 0 0" rpy="0 0 ${M_PI/2}" />
             <xacro:property name="parent"               value="chassis_link"/>
             <xacro:property name="robot_namespace"      value="agribot"/>

Commit message: Include imu mount angle when simulating reference_heading in gazebo

File: urdf/basic_sensors.xacro (robot description, xacro)
@@ -5,9 +5,10 @@
     <xacro:include filename="$(find agribot_description)/urdf/basic_sensors/magnetometer/magnetometer.xacro"/>
     <xacro:macro name="basic_sensors">
+        <xacro:property name="chassis_to_imu_yaw" value="${M_PI/2}"/>
         <!-- NOTE: Simulation properties are passed in robot_description.xml file -->
         <!-- Position on Earth -->
         <xacro:property name="reference_latitude"   value="$(arg simulation_latitude)"/>
         <xacro:property name="reference_longitude"  value="$(arg simulation_longitude)"/>
-        <xacro:property name="reference_heading"    value="$(arg simulation_heading)"/>
+        <xacro:property name="reference_heading"    value="${$(arg simulation_heading) - degrees(chassis_to_imu_yaw)}"/>
         <xacro:property name="reference_altitude"   value="$(arg simulation_altitude)"/>
         <!-- Magnetometer simulation plugin -->
@@ -15,5 +16,5 @@
         <xacro:property name="inclination"   value="$(arg simulation_inclination)"/>
         <xacro:imu_sensor>
-            <origin xyz="0 0 0" rpy="0 0 ${M_PI/2}" />
+            <origin xyz="0 0 0" rpy="0 0 ${chassis_to_imu_yaw}" />
             <xacro:property name="parent"               value="chassis_link"/>
             <xacro:property name="topic"                value="/agribot/imu/raw/data"/>
@@ -48,5 +49,5 @@
         </xacro:inclinometer>
         <xacro:magnetometer>
-            <origin xyz="0 0 0" rpy="0 0 ${M_PI/2}" />
+            <origin xyz="0 0 0" rpy="0 0 ${chassis_to_imu_yaw}" />
             <xacro:property name="parent"               value="chassis_link"/>
             <xacro:property name="robot_namespace"      value="agribot"/>

Commit message: Correct reference heading setting - split it into separate reference heading for gps and magnetometer, as magnetometer heading is affected by imu mount angle and gps reference heading is "global" value independent of imu mount position

File: urdf/basic_sensors.xacro (robot description, xacro)
@@ -10,5 +10,4 @@
         <xacro:property name="reference_latitude"   value="$(arg simulation_latitude)"/>
         <xacro:property name="reference_longitude"  value="$(arg simulation_longitude)"/>
-        <xacro:property name="reference_heading"    value="${$(arg simulation_heading) - degrees(chassis_to_imu_yaw)}"/>
         <xacro:property name="reference_altitude"   value="$(arg simulation_altitude)"/>
         <!-- Magnetometer simulation plugin -->
@@ -32,4 +31,5 @@
             <xacro:property name="name"                 value="gps"/>
             <xacro:property name="hz"                   value="10.0"/>
+            <xacro:property name="reference_heading"  value="${$(arg simulation_heading)}"/>
             <xacro:property name="noise"                value="$(arg simulation_gps_noise)"/>
             <xacro:property name="velocity_noise"       value="$(arg simulation_gps_velocity_noise)"/>
@@ -55,4 +55,5 @@
             <xacro:property name="name"                 value="magnetometer"/>
             <xacro:property name="hz"                   value="10.0"/>
+            <xacro:property name="reference_heading"  value="${$(arg simulation_heading) - degrees(chassis_to_imu_yaw)}"/>
             <xacro:property name="magnitude"            value="$(arg simulation_magnetometer_magnitude)"/>
             <xacro:property name="noise"                value="$(arg simulation_magnetometer_noise)"/>

Commit message: Add bynav and hydrabox links as dual_antenna_gps macros. TODO: add gazebo plugins

File: urdf/basic_sensors.xacro (robot description, xacro)
@@ -2,4 +2,5 @@
     <xacro:include filename="$(find agribot_description)/urdf/basic_sensors/imu/imu_sensor.xacro"/>
     <xacro:include filename="$(find agribot_description)/urdf/basic_sensors/gps/gps.xacro"/>
+    <xacro:include filename="$(find agribot_description)/urdf/basic_sensors/gps/dual_antenna_gps.xacro"/>
     <xacro:include filename="$(find agribot_description)/urdf/basic_sensors/inclinometer/inclinometer.xacro"/>
     <xacro:include filename="$(find agribot_description)/urdf/basic_sensors/magnetometer/magnetometer.xacro"/>
@@ -14,4 +15,14 @@
         <xacro:property name="declination"   value="$(arg simulation_declination)"/>
         <xacro:property name="inclination"   value="$(arg simulation_inclination)"/>
+        <xacro:dual_antenna_gps>
+          <origin xyz="0 0 0" rpy="0 0 0" />
+          <xacro:property name="parent"               value="chassis_link"/>
+          <xacro:property name="name"                 value="bynav"/>
+        </xacro:dual_antenna_gps>
+        <xacro:dual_antenna_gps>
+          <origin xyz="0 0 0" rpy="0 0 0" />
+          <xacro:property name="parent"               value="chassis_link"/>
+          <xacro:property name="name"                 value="hydrabox"/>
+        </xacro:dual_antenna_gps>
         <xacro:imu_sensor>
             <origin xyz="0 0 0" rpy="0 0 ${chassis_to_imu_yaw}" />

Commit message: Add plugins for hydrabox and bynav

File: urdf/basic_sensors.xacro (robot description, xacro)
@@ -19,4 +19,13 @@
           <xacro:property name="parent"               value="chassis_link"/>
           <xacro:property name="name"                 value="bynav"/>
+          <xacro:property name="robot_namespace"      value="agribot"/>
+          <xacro:property name="topic"                value="gnss/bynav"/>
+          <xacro:property name="velocity_topic"       value="gnss_velocity/bynav"/>
+          <xacro:property name="hz"                   value="10.0"/>
+          <xacro:property name="reference_heading"  value="${$(arg simulation_heading)}"/>
+          <xacro:property name="noise"                value="$(arg simulation_gps_noise)"/>
+          <xacro:property name="velocity_noise"       value="$(arg simulation_gps_velocity_noise)"/> -->
+          <xacro:property name="heading_topic"        value="heading/bynav"/>
+          <xacro:property name="heading_noise"        value="$(arg simulation_gps_heading_noise)"/>
         </xacro:dual_antenna_gps>
         <xacro:dual_antenna_gps>
@@ -24,4 +33,13 @@
           <xacro:property name="parent"               value="chassis_link"/>
           <xacro:property name="name"                 value="hydrabox"/>
+          <xacro:property name="robot_namespace"      value="agribot"/>
+          <xacro:property name="topic"                value="gnss/hydrabox"/>
+          <xacro:property name="velocity_topic"       value="gnss_velocity/hydrabox"/>
+          <xacro:property name="hz"                   value="10.0"/>
+          <xacro:property name="reference_heading"  value="${$(arg simulation_heading)}"/>
+          <xacro:property name="noise"                value="$(arg simulation_gps_noise)"/>
+          <xacro:property name="velocity_noise"       value="$(arg simulation_gps_velocity_noise)"/>
+          <xacro:property name="heading_topic"        value="heading/hydrabox"/>
+          <xacro:property name="heading_noise"        value="$(arg simulation_gps_heading_noise)"/>
         </xacro:dual_antenna_gps>
         <xacro:imu_sensor>

File: urdf/basic_sensors/gps/dual_antenna_gps.xacro (robot description, xacro)
@@ -4,12 +4,22 @@
                                                parent:=^
                                                name:=^
+                                               robot_namespace:=^
+                                               topic:=^
+                                               velocity_topic:=^
+                                               hz:=^
+                                               reference_latitude:=^
+                                               reference_longitude:=^
+                                               reference_heading:=^
+                                               reference_altitude:=^
+                                               noise:=^
+                                               velocity_noise:=^
+                                               publish_heading:=^|false
+                                               heading_topic:=^|heading
+                                               heading_noise:=^|0.00
                                                ">
-    <joint name="${name}_joint" type="fixed">
+    <xacro:gps>
       <xacro:insert_block name="origin" />
-      <parent link="${parent}" />
-      <child link="${name}_link" />
-    </joint>
-    <link name="${name}_link" />
-    <!-- TODO(olek) - add gazebo plugins -->
+      <xacro:property name="publish_heading" value="true" />
+    </xacro:gps>
   </xacro:macro>
 </robot>
