Commit message: Remove old (regular) GPS, IMU and magnetometer

File: urdf/basic_sensors.xacro (robot description, xacro)
@@ -43,29 +43,4 @@
           <xacro:property name="heading_noise"        value="$(arg simulation_gps_heading_noise)"/>
         </xacro:dual_antenna_gps>
-        <xacro:imu_sensor>
-            <origin xyz="0 0 0" rpy="0 0 ${chassis_to_imu_yaw}" />
-            <xacro:property name="parent"               value="chassis_link"/>
-            <xacro:property name="topic"                value="/agribot/imu/raw/data"/>
-            <xacro:property name="name"                 value="imu"/>
-            <xacro:property name="hz"                   value="10.0"/>
-            <xacro:property name="accel_noise"          value="$(arg simulation_accelerometer_noise)"/>
-            <xacro:property name="gyro_noise"           value="$(arg simulation_gyroscope_noise)"/>
-        </xacro:imu_sensor>
-        <xacro:gps>
-            <origin xyz="0 0 0" rpy="0 0 0" />
-            <xacro:property name="parent"               value="chassis_link"/>
-            <xacro:property name="robot_namespace"      value="agribot"/>
-            <xacro:property name="topic"                value="gnss"/>
-            <xacro:property name="velocity_topic"       value="fix_velocity"/>
-            <xacro:property name="name"                 value="gps"/>
-            <xacro:property name="hz"                   value="10.0"/>
-            <xacro:property name="reference_heading"  value="${$(arg simulation_heading)}"/>
-            <xacro:property name="noise"                value="$(arg simulation_gps_noise)"/>
-            <xacro:property name="velocity_noise"       value="$(arg simulation_gps_velocity_noise)"/>
-            <!-- Use heading -->
-            <xacro:property name="publish_heading"      value="$(arg simulation_gps_publish_heading)"/>
-            <xacro:property name="heading_topic"        value="heading"/>
-            <xacro:property name="heading_noise"        value="$(arg simulation_gps_heading_noise)"/>
-        </xacro:gps>
         <xacro:inclinometer>
             <origin xyz="0 0 0" rpy="0 0 0" />
@@ -77,15 +52,4 @@
             <xacro:property name="noise"                value="$(arg simulation_inclinometer_noise)"/>
         </xacro:inclinometer>
-        <xacro:magnetometer>
-            <origin xyz="0 0 0" rpy="0 0 ${chassis_to_imu_yaw}" />
-            <xacro:property name="parent"               value="chassis_link"/>
-            <xacro:property name="robot_namespace"      value="agribot"/>
-            <xacro:property name="topic"                value="imu/raw/mag"/>
-            <xacro:property name="name"                 value="magnetometer"/>
-            <xacro:property name="hz"                   value="10.0"/>
-            <xacro:property name="reference_heading"  value="${$(arg simulation_heading) - degrees(chassis_to_imu_yaw)}"/>
-            <xacro:property name="magnitude"            value="$(arg simulation_magnetometer_magnitude)"/>
-            <xacro:property name="noise"                value="$(arg simulation_magnetometer_noise)"/>
-        </xacro:magnetometer>
     </xacro:macro>
 </robot>

Commit message: Remove old Imu and Magnetometer parameters

File: urdf/basic_sensors.xacro (robot description, xacro)
@@ -1,10 +1,6 @@
 <robot name="sensors" xmlns:xacro="http://ros.org/wiki/xacro">
-    <xacro:include filename="$(find agribot_description)/urdf/basic_sensors/imu/imu_sensor.xacro"/>
-    <xacro:include filename="$(find agribot_description)/urdf/basic_sensors/gps/gps.xacro"/>
     <xacro:include filename="$(find agribot_description)/urdf/basic_sensors/gps/dual_antenna_gps.xacro"/>
     <xacro:include filename="$(find agribot_description)/urdf/basic_sensors/inclinometer/inclinometer.xacro"/>
-    <xacro:include filename="$(find agribot_description)/urdf/basic_sensors/magnetometer/magnetometer.xacro"/>
     <xacro:macro name="basic_sensors">
-        <xacro:property name="chassis_to_imu_yaw" value="${M_PI/2}"/>
         <!-- NOTE: Simulation properties are passed in robot_description.xml file -->
         <!-- Position on Earth -->
@@ -12,7 +8,5 @@
         <xacro:property name="reference_longitude"  value="$(arg simulation_longitude)"/>
         <xacro:property name="reference_altitude"   value="$(arg simulation_altitude)"/>
-        <!-- Magnetometer simulation plugin -->
-        <xacro:property name="declination"   value="$(arg simulation_declination)"/>
-        <xacro:property name="inclination"   value="$(arg simulation_inclination)"/>
+        <xacro:property name="reference_heading"  value="$(arg simulation_heading)"/>
         <xacro:dual_antenna_gps>
           <origin xyz="0 0 0" rpy="0 0 0" />
@@ -23,7 +17,6 @@
           <xacro:property name="velocity_topic"       value="gnss_velocity/bynav"/>
           <xacro:property name="hz"                   value="10.0"/>
-          <xacro:property name="reference_heading"  value="${$(arg simulation_heading)}"/>
           <xacro:property name="noise"                value="$(arg simulation_gps_noise)"/>
-          <xacro:property name="velocity_noise"       value="$(arg simulation_gps_velocity_noise)"/> -->
+          <xacro:property name="velocity_noise"       value="$(arg simulation_gps_velocity_noise)"/>
           <xacro:property name="heading_topic"        value="heading/bynav"/>
           <xacro:property name="heading_noise"        value="$(arg simulation_gps_heading_noise)"/>
@@ -37,5 +30,4 @@
           <xacro:property name="velocity_topic"       value="gnss_velocity/hydrabox"/>
           <xacro:property name="hz"                   value="10.0"/>
-          <xacro:property name="reference_heading"  value="${$(arg simulation_heading)}"/>
           <xacro:property name="noise"                value="$(arg simulation_gps_noise)"/>
           <xacro:property name="velocity_noise"       value="$(arg simulation_gps_velocity_noise)"/>

File: urdf/basic_sensors/gps/dual_antenna_gps.xacro (robot description, xacro)
@@ -1,3 +1,4 @@
 <robot name="dual_antenna_gps" xmlns:xacro="http://www.ros.org/wiki/xacro">
+  <xacro:include filename="$(find agribot_description)/urdf/basic_sensors/gps/gps.xacro" />
   <!-- Basic sonar macro  -->
   <xacro:macro name="dual_antenna_gps" params="*origin

Commit message: Add separate GPS noise parameters for bynav and hydrabox

File: urdf/basic_sensors.xacro (robot description, xacro)
@@ -17,8 +17,8 @@
           <xacro:property name="velocity_topic"       value="gnss_velocity/bynav"/>
           <xacro:property name="hz"                   value="10.0"/>
-          <xacro:property name="noise"                value="$(arg simulation_gps_noise)"/>
-          <xacro:property name="velocity_noise"       value="$(arg simulation_gps_velocity_noise)"/>
+          <xacro:property name="noise"                value="$(arg simulation_bynav_position_noise)"/>
+          <xacro:property name="velocity_noise"       value="$(arg simulation_bynav_velocity_noise)"/>
           <xacro:property name="heading_topic"        value="heading/bynav"/>
-          <xacro:property name="heading_noise"        value="$(arg simulation_gps_heading_noise)"/>
+          <xacro:property name="heading_noise"        value="$(arg simulation_bynav_heading_noise)"/>
         </xacro:dual_antenna_gps>
         <xacro:dual_antenna_gps>
@@ -30,8 +30,8 @@
           <xacro:property name="velocity_topic"       value="gnss_velocity/hydrabox"/>
           <xacro:property name="hz"                   value="10.0"/>
-          <xacro:property name="noise"                value="$(arg simulation_gps_noise)"/>
-          <xacro:property name="velocity_noise"       value="$(arg simulation_gps_velocity_noise)"/>
+          <xacro:property name="noise"                value="$(arg simulation_hydrabox_position_noise)"/>
+          <xacro:property name="velocity_noise"       value="$(arg simulation_hydrabox_velocity_noise)"/>
           <xacro:property name="heading_topic"        value="heading/hydrabox"/>
-          <xacro:property name="heading_noise"        value="$(arg simulation_gps_heading_noise)"/>
+          <xacro:property name="heading_noise"        value="$(arg simulation_hydrabox_heading_noise)"/>
         </xacro:dual_antenna_gps>
         <xacro:inclinometer>
