Commit message: Agribot model v1

File: urdf/agribot.urdf.xacro (robot description, xacro)
@@ -3,33 +3,54 @@
   <xacro:include filename="$(find agribot_description)/urdf/common_properties.xacro"/>
   <xacro:include filename="$(find agribot_description)/urdf/agribot.gazebo"/>
-  <xacro:include filename="$(find agribot_description)/urdf/basic_links/base.xacro"/>
+  <xacro:include filename="$(find agribot_description)/urdf/basic_links/cart.xacro"/>
   <xacro:include filename="$(find agribot_description)/urdf/basic_links/wheel.xacro"/>
-  <xacro:include filename="$(find agribot_description)/urdf/basic_links/caster.xacro"/>
   <link name="base_footprint"/>
-  <joint name="base_joint" type="fixed">
+  <joint name="chassis_joint" type="fixed">
     <parent link="base_footprint"/>
-    <child link="base_link" />
-    <origin xyz="0 0 ${wheel_radius}" rpy="0 0 0"/>
+    <child link="chassis_link" />
+    <origin xyz="0 0 ${3*wheel_radius+chassis_heigth/2}" rpy="0 0 0"/>
   </joint>
-  <xacro:agribot_base name="base_link" />
-  <joint name="wheel_left_joint" type="continuous">
-    <parent link="base_link"/>
-    <child link="wheel_left_link"/>
-    <origin xyz="${(base_lenght/2)-wheel_radius} ${(base_width+wheel_width)/2} 0.0" rpy="${-M_PI/2} 0 0"/>
-    <axis xyz="0 0 1"/>
-  </joint>
-  <xacro:agribot_wheel name="wheel_left_link" />
-  <joint name="wheel_right_joint" type="continuous">
-    <parent link="base_link"/>
-    <child link="wheel_right_link"/>
-    <origin xyz="${(base_lenght/2)-wheel_radius} ${-(base_width+wheel_width)/2} 0.0" rpy="${-M_PI/2} 0 0"/>
-    <axis xyz="0 0 1"/>
-  </joint>
-  <xacro:agribot_wheel name="wheel_right_link" />
-  <joint name="caster_back_right_joint" type="fixed">
-    <parent link="base_link"/>
-    <child link="caster_back"/>
-    <origin xyz="${caster_lenght-(base_lenght/2)} 0.0 ${-(base_height+caster_height)/2}" rpy="0.0 0.0 0.0"/>
-  </joint>
-  <xacro:agribot_caster name="caster_back" />
+  <xacro:agribot_chassis name="chassis_link" />
+      <joint name="front_cart_joint" type="continuous">
+        <parent link="chassis_link"/>
+        <child link="front_cart_link"/>
+        <origin xyz="${(chassis_length/2)-cart_lenght/2} 0.0 ${-3*wheel_radius}" rpy="0 0 0"/>
+        <axis xyz="0 0 1"/>
+      </joint>
+      <xacro:agribot_cart name="front_cart_link" />
+          <joint name="front_left_wheel_joint" type="continuous">
+              <parent link="front_cart_link"/>
+              <child link="front_left_wheel_link"/>
+              <origin xyz="0.0 ${(chassis_width+wheel_width)/2} ${-wheel_radius}" rpy="${-M_PI/2} 0 0"/>
+              <axis xyz="0 0 1"/>
+            </joint>
+            <xacro:agribot_wheel name="front_left_wheel_link" />
+            <joint name="front_right_wheel_joint" type="continuous">
+              <parent link="front_cart_link"/>
+              <child link="front_right_wheel_link"/>
+              <origin xyz="0.0 ${-(chassis_width+wheel_width)/2} ${-wheel_radius}" rpy="${-M_PI/2} 0 0"/>
+              <axis xyz="0 0 1"/>
+            </joint>
+            <xacro:agribot_wheel name="front_right_wheel_link" />
+      <joint name="back_cart_joint" type="continuous">
+        <parent link="chassis_link"/>
+        <child link="back_cart_link"/>
+        <origin xyz="${-(chassis_length/2)+cart_lenght/2} 0.0 ${-3*wheel_radius}" rpy="0 0 0"/>
+        <axis xyz="0 0 1"/>
+      </joint>
+      <xacro:agribot_cart name="back_cart_link" />
+          <joint name="back_left_wheel_joint" type="continuous">
+              <parent link="back_cart_link"/>
+              <child link="back_left_wheel_link"/>
+              <origin xyz="0.0 ${(chassis_width+wheel_width)/2} ${-wheel_radius}" rpy="${-M_PI/2} 0 0"/>
+              <axis xyz="0 0 1"/>
+            </joint>
+            <xacro:agribot_wheel name="back_left_wheel_link" />
+            <joint name="back_right_wheel_joint" type="continuous">
+              <parent link="back_cart_link"/>
+              <child link="back_right_wheel_link"/>
+              <origin xyz="0.0 ${-(chassis_width+wheel_width)/2} ${-wheel_radius}" rpy="${-M_PI/2} 0 0"/>
+              <axis xyz="0 0 1"/>
+            </joint>
+            <xacro:agribot_wheel name="back_right_wheel_link" />
 </robot>

File: urdf/basic_links/chassis.xacro (robot description, xacro)
@@ -1,12 +1,12 @@
-<robot name="base" xmlns:xacro="http://ros.org/wiki/xacro">
-    <xacro:property name="base_lenght" value="0.2" />
-    <xacro:property name="base_width" value="0.2" />
-    <xacro:property name="base_height" value="0.01" />
-    <xacro:macro name="agribot_base" params="name">
+<robot name="chassis" xmlns:xacro="http://ros.org/wiki/xacro">
+    <xacro:property name="chassis_length" value="1" />
+    <xacro:property name="chassis_width" value="0.2" />
+    <xacro:property name="chassis_heigth" value="0.2" />
+    <xacro:macro name="agribot_chassis" params="name">
         <link name="${name}">
           <visual>
             <origin xyz="0.0 0.0 0.0" rpy="0 0 0"/>
             <geometry>
-               <box size="${base_lenght} ${base_width} ${base_height}" />
+               <box size="${chassis_length} ${chassis_width} ${chassis_heigth}" />
             </geometry>
             <material name="blue"/>
@@ -15,5 +15,5 @@
             <origin xyz="0.0 0.0 0.0" rpy="0 0 0"/>
             <geometry>
-              <box size="${base_lenght} ${base_width} ${base_height}"/>
+              <box size="${chassis_length} ${chassis_width} ${chassis_heigth}"/>
             </geometry>
           </collision>

Commit message: Agribot model v1.01

File: urdf/agribot.urdf.xacro (robot description, xacro)
@@ -5,9 +5,10 @@
   <xacro:include filename="$(find agribot_description)/urdf/basic_links/cart.xacro"/>
   <xacro:include filename="$(find agribot_description)/urdf/basic_links/wheel.xacro"/>
+  <xacro:include filename="$(find agribot_description)/urdf/basic_links/support.xacro"/>
   <link name="base_footprint"/>
   <joint name="chassis_joint" type="fixed">
     <parent link="base_footprint"/>
     <child link="chassis_link" />
-    <origin xyz="0 0 ${3*wheel_radius+chassis_heigth/2}" rpy="0 0 0"/>
+    <origin xyz="0 0 ${3*wheel_radius+chassis_height/2 + 1}" rpy="0 0 0"/>
   </joint>
   <xacro:agribot_chassis name="chassis_link" />
@@ -15,8 +16,15 @@
         <parent link="chassis_link"/>
         <child link="front_cart_link"/>
-        <origin xyz="${(chassis_length/2)-cart_lenght/2} 0.0 ${-3*wheel_radius}" rpy="0 0 0"/>
+        <origin xyz="${(chassis_length/2)-cart_lenght/2} 0.0 ${(chassis_height+cart_height)/(-2)}" rpy="0 0 0"/>
         <axis xyz="0 0 1"/>
       </joint>
       <xacro:agribot_cart name="front_cart_link" />
+          <joint name="front_support_joint" type="fixed">
+              <parent link="front_cart_link"/>
+              <child link="front_support_link"/>
+              <origin xyz="0.0 0.0 ${-cart_height/2-support_height/2}" rpy="0 0 0"/>
+              <axis xyz="0 0 1"/>
+          </joint>
+          <xacro:agribot_support name="front_support_link" />
           <joint name="front_left_wheel_joint" type="continuous">
               <parent link="front_cart_link"/>
@@ -36,8 +44,15 @@
         <parent link="chassis_link"/>
         <child link="back_cart_link"/>
-        <origin xyz="${-(chassis_length/2)+cart_lenght/2} 0.0 ${-3*wheel_radius}" rpy="0 0 0"/>
+        <origin xyz="${-(chassis_length/2)+cart_lenght/2} 0.0 ${(chassis_height+cart_height)/(-2)}" rpy="0 0 0"/>
         <axis xyz="0 0 1"/>
       </joint>
       <xacro:agribot_cart name="back_cart_link" />
+          <joint name="back_support_joint" type="fixed">
+            <parent link="back_cart_link"/>
+            <child link="back_support_link"/>
+            <origin xyz="0.0 0.0 ${-cart_height/2-support_height/2}" rpy="0 0 0"/>
+            <axis xyz="0 0 1"/>
+          </joint>
+          <xacro:agribot_support name="back_support_link" />
           <joint name="back_left_wheel_joint" type="continuous">
               <parent link="back_cart_link"/>

File: urdf/basic_links/chassis.xacro (robot description, xacro)
@@ -2,5 +2,5 @@
     <xacro:property name="chassis_length" value="1" />
     <xacro:property name="chassis_width" value="0.2" />
-    <xacro:property name="chassis_heigth" value="0.2" />
+    <xacro:property name="chassis_height" value="0.2" />
     <xacro:macro name="agribot_chassis" params="name">
         <link name="${name}">
@@ -8,5 +8,5 @@
             <origin xyz="0.0 0.0 0.0" rpy="0 0 0"/>
             <geometry>
-               <box size="${chassis_length} ${chassis_width} ${chassis_heigth}" />
+               <box size="${chassis_length} ${chassis_width} ${chassis_height}" />
             </geometry>
             <material name="blue"/>
@@ -15,10 +15,10 @@
             <origin xyz="0.0 0.0 0.0" rpy="0 0 0"/>
             <geometry>
-              <box size="${chassis_length} ${chassis_width} ${chassis_heigth}"/>
+              <box size="${chassis_length} ${chassis_width} ${chassis_height}"/>
             </geometry>
           </collision>
           <inertial>
             <origin xyz="0.0 0.0 0.0" rpy="0 0 0"/>
-            <mass value="1"/>
+            <mass value="10"/>
             <inertia ixx="0.01" ixy="0.0" ixz="0.0"
                      iyy="0.01" iyz="0.0"

Commit message: Agribot description with ros_controller

File: urdf/agribot.urdf.xacro (robot description, xacro)
@@ -10,5 +10,5 @@
     <parent link="base_footprint"/>
     <child link="chassis_link" />
-    <origin xyz="0 0 ${3*wheel_radius+chassis_height/2 + 1}" rpy="0 0 0"/>
+    <origin xyz="0 0 ${3*wheel_radius+chassis_height/2}" rpy="0 0 0"/>
   </joint>
   <xacro:agribot_chassis name="chassis_link" />

File: urdf/basic_links/support.xacro (robot description, xacro)
@@ -4,5 +4,5 @@
     <xacro:property name="support_length" value="${chassis_width*2}" />
     <xacro:property name="support_width" value="${wheel_width}" />
-    <xacro:property name="support_height" value="${wheel_radius*0.5}" />
+    <xacro:property name="support_height" value="${wheel_radius*0.99}" />
     <xacro:macro name="agribot_support" params="name">
         <link name="${name}">

Commit message: Remove unnecessary things

File: urdf/agribot.urdf.xacro (robot description, xacro)
@@ -13,59 +13,59 @@
   </joint>
   <xacro:agribot_chassis name="chassis_link" />
-      <joint name="front_cart_joint" type="continuous">
-        <parent link="chassis_link"/>
-        <child link="front_cart_link"/>
-        <origin xyz="${(chassis_length/2)-cart_lenght/2} 0.0 ${(chassis_height+cart_height)/(-2)}" rpy="0 0 0"/>
-        <axis xyz="0 0 1"/>
-      </joint>
-      <xacro:agribot_cart name="front_cart_link" />
-          <joint name="front_support_joint" type="fixed">
-              <parent link="front_cart_link"/>
-              <child link="front_support_link"/>
-              <origin xyz="0.0 0.0 ${-cart_height/2-support_height/2}" rpy="0 0 0"/>
-              <axis xyz="0 0 1"/>
-          </joint>
-          <xacro:agribot_support name="front_support_link" />
-          <joint name="front_left_wheel_joint" type="continuous">
-              <parent link="front_cart_link"/>
-              <child link="front_left_wheel_link"/>
-              <origin xyz="0.0 ${(chassis_width+wheel_width)/2} ${-wheel_radius}" rpy="${-M_PI/2} 0 0"/>
-              <axis xyz="0 0 1"/>
-            </joint>
-            <xacro:agribot_wheel name="front_left_wheel_link" />
-            <joint name="front_right_wheel_joint" type="continuous">
-              <parent link="front_cart_link"/>
-              <child link="front_right_wheel_link"/>
-              <origin xyz="0.0 ${-(chassis_width+wheel_width)/2} ${-wheel_radius}" rpy="${-M_PI/2} 0 0"/>
-              <axis xyz="0 0 1"/>
-            </joint>
-            <xacro:agribot_wheel name="front_right_wheel_link" />
-      <joint name="back_cart_joint" type="continuous">
-        <parent link="chassis_link"/>
-        <child link="back_cart_link"/>
-        <origin xyz="${-(chassis_length/2)+cart_lenght/2} 0.0 ${(chassis_height+cart_height)/(-2)}" rpy="0 0 0"/>
-        <axis xyz="0 0 1"/>
-      </joint>
-      <xacro:agribot_cart name="back_cart_link" />
-          <joint name="back_support_joint" type="fixed">
-            <parent link="back_cart_link"/>
-            <child link="back_support_link"/>
-            <origin xyz="0.0 0.0 ${-cart_height/2-support_height/2}" rpy="0 0 0"/>
-            <axis xyz="0 0 1"/>
-          </joint>
-          <xacro:agribot_support name="back_support_link" />
-          <joint name="back_left_wheel_joint" type="continuous">
-              <parent link="back_cart_link"/>
-              <child link="back_left_wheel_link"/>
-              <origin xyz="0.0 ${(chassis_width+wheel_width)/2} ${-wheel_radius}" rpy="${-M_PI/2} 0 0"/>
-              <axis xyz="0 0 1"/>
-            </joint>
-            <xacro:agribot_wheel name="back_left_wheel_link" />
-            <joint name="back_right_wheel_joint" type="continuous">
-              <parent link="back_cart_link"/>
-              <child link="back_right_wheel_link"/>
-              <origin xyz="0.0 ${-(chassis_width+wheel_width)/2} ${-wheel_radius}" rpy="${-M_PI/2} 0 0"/>
-              <axis xyz="0 0 1"/>
-            </joint>
-            <xacro:agribot_wheel name="back_right_wheel_link" />
+  <joint name="front_cart_joint" type="continuous">
+    <parent link="chassis_link"/>
+    <child link="front_cart_link"/>
+    <origin xyz="${(chassis_length/2)-cart_lenght/2} 0.0 ${(chassis_height+cart_height)/(-2)}" rpy="0 0 0"/>
+    <axis xyz="0 0 1"/>
+  </joint>
+  <xacro:agribot_cart name="front_cart_link" />
+  <joint name="front_support_joint" type="fixed">
+    <parent link="front_cart_link"/>
+    <child link="front_support_link"/>
+    <origin xyz="0.0 0.0 ${-cart_height/2-support_height/2}" rpy="0 0 0"/>
+    <axis xyz="0 0 1"/>
+  </joint>
+  <xacro:agribot_support name="front_support_link" />
+  <joint name="front_left_wheel_joint" type="continuous">
+    <parent link="front_cart_link"/>
+    <child link="front_left_wheel_link"/>
+    <origin xyz="0.0 ${(chassis_width+wheel_width)/2} ${-wheel_radius}" rpy="${-M_PI/2} 0 0"/>
+    <axis xyz="0 0 1"/>
+  </joint>
+  <xacro:agribot_wheel name="front_left_wheel_link" />
+  <joint name="front_right_wheel_joint" type="continuous">
+    <parent link="front_cart_link"/>
+    <child link="front_right_wheel_link"/>
+    <origin xyz="0.0 ${-(chassis_width+wheel_width)/2} ${-wheel_radius}" rpy="${-M_PI/2} 0 0"/>
+    <axis xyz="0 0 1"/>
+  </joint>
+  <xacro:agribot_wheel name="front_right_wheel_link" />
+  <joint name="back_cart_joint" type="continuous">
+    <parent link="chassis_link"/>
+    <child link="back_cart_link"/>
+    <origin xyz="${-(chassis_length/2)+cart_lenght/2} 0.0 ${(chassis_height+cart_height)/(-2)}" rpy="0 0 0"/>
+    <axis xyz="0 0 1"/>
+  </joint>
+  <xacro:agribot_cart name="back_cart_link" />
+  <joint name="back_support_joint" type="fixed">
+    <parent link="back_cart_link"/>
+    <child link="back_support_link"/>
+    <origin xyz="0.0 0.0 ${-cart_height/2-support_height/2}" rpy="0 0 0"/>
+    <axis xyz="0 0 1"/>
+  </joint>
+  <xacro:agribot_support name="back_support_link" />
+  <joint name="back_left_wheel_joint" type="continuous">
+    <parent link="back_cart_link"/>
+    <child link="back_left_wheel_link"/>
+    <origin xyz="0.0 ${(chassis_width+wheel_width)/2} ${-wheel_radius}" rpy="${-M_PI/2} 0 0"/>
+    <axis xyz="0 0 1"/>
+  </joint>
+  <xacro:agribot_wheel name="back_left_wheel_link" />
+  <joint name="back_right_wheel_joint" type="continuous">
+    <parent link="back_cart_link"/>
+    <child link="back_right_wheel_link"/>
+    <origin xyz="0.0 ${-(chassis_width+wheel_width)/2} ${-wheel_radius}" rpy="${-M_PI/2} 0 0"/>
+    <axis xyz="0 0 1"/>
+  </joint>
+  <xacro:agribot_wheel name="back_right_wheel_link" />
 </robot>

Commit message: Removed support, changed link type to revolute, added limits to cart joints

File: urdf/agribot.urdf.xacro (robot description, xacro)
@@ -13,18 +13,12 @@
   </joint>
   <xacro:agribot_chassis name="chassis_link" />
-  <joint name="front_cart_joint" type="continuous">
+  <joint name="front_cart_joint" type="revolute">
     <parent link="chassis_link"/>
     <child link="front_cart_link"/>
+    <limit lower="${-M_PI/4}" upper="${M_PI/4}" effort="1000.0" velocity="1000.0"/>
     <origin xyz="${(chassis_length/2)-cart_lenght/2} 0.0 ${(chassis_height+cart_height)/(-2)}" rpy="0 0 0"/>
     <axis xyz="0 0 1"/>
   </joint>
   <xacro:agribot_cart name="front_cart_link" />
-  <joint name="front_support_joint" type="fixed">
-    <parent link="front_cart_link"/>
-    <child link="front_support_link"/>
-    <origin xyz="0.0 0.0 ${-cart_height/2-support_height/2}" rpy="0 0 0"/>
-    <axis xyz="0 0 1"/>
-  </joint>
-  <xacro:agribot_support name="front_support_link" />
   <joint name="front_left_wheel_joint" type="continuous">
     <parent link="front_cart_link"/>
@@ -41,18 +35,12 @@
   </joint>
   <xacro:agribot_wheel name="front_right_wheel_link" />
-  <joint name="back_cart_joint" type="continuous">
+  <joint name="back_cart_joint" type="revolute">
     <parent link="chassis_link"/>
     <child link="back_cart_link"/>
+    <limit lower="${-M_PI/4}" upper="${M_PI/4}"  effort="1000.0" velocity="1000.0"/>
     <origin xyz="${-(chassis_length/2)+cart_lenght/2} 0.0 ${(chassis_height+cart_height)/(-2)}" rpy="0 0 0"/>
     <axis xyz="0 0 1"/>
   </joint>
   <xacro:agribot_cart name="back_cart_link" />
-  <joint name="back_support_joint" type="fixed">
-    <parent link="back_cart_link"/>
-    <child link="back_support_link"/>
-    <origin xyz="0.0 0.0 ${-cart_height/2-support_height/2}" rpy="0 0 0"/>
-    <axis xyz="0 0 1"/>
-  </joint>
-  <xacro:agribot_support name="back_support_link" />
   <joint name="back_left_wheel_joint" type="continuous">
     <parent link="back_cart_link"/>

Commit message: Fixed model size to real world values. With bigger mass the model breaks.

File: urdf/agribot.urdf.xacro (robot description, xacro)
@@ -57,3 +57,9 @@
   </joint>
   <xacro:agribot_wheel name="back_right_wheel_link" />
+  <gazebo>
+    <plugin name="agribot_controller" filename="libgazebo_ros_agribot.so">
+      <wheelSeparation> ${chassis_width+wheel_width} </wheelSeparation>
+      <wheelRadius> ${wheel_radius} </wheelRadius>
+    </plugin>
+  </gazebo>
 </robot>

File: urdf/basic_links/cart.xacro (robot description, xacro)
@@ -22,5 +22,6 @@
           <inertial>
             <origin xyz="0.0 0.0 0.0" rpy="0 0 0"/>
-            <mass value="1"/>
+            <!-- <mass value="1"/> -->
+            <mass value="1.00"/>
             <inertia ixx="0.01" ixy="0.0" ixz="0.0"
                      iyy="0.01" iyz="0.0"

File: urdf/basic_links/chassis.xacro (robot description, xacro)
@@ -1,6 +1,9 @@
 <robot name="chassis" xmlns:xacro="http://ros.org/wiki/xacro">
-    <xacro:property name="chassis_length" value="1" />
+    <!-- <xacro:property name="chassis_length" value="1" />
     <xacro:property name="chassis_width" value="0.2" />
-    <xacro:property name="chassis_height" value="0.2" />
+    <xacro:property name="chassis_height" value="0.2" /> -->
+    <xacro:property name="chassis_length" value="2.42" />
+    <xacro:property name="chassis_width" value="1.05" />
+    <xacro:property name="chassis_height" value="1.3" />
     <xacro:macro name="agribot_chassis" params="name">
         <link name="${name}">
@@ -20,5 +23,6 @@
           <inertial>
             <origin xyz="0.0 0.0 0.0" rpy="0 0 0"/>
-            <mass value="10"/>
+            <!-- <mass value="10"/> -->
+            <mass value="1.600"/>
             <inertia ixx="0.01" ixy="0.0" ixz="0.0"
                      iyy="0.01" iyz="0.0"

File: urdf/basic_links/wheel.xacro (robot description, xacro)
@@ -1,5 +1,7 @@
 <robot name="wheel" xmlns:xacro="http://ros.org/wiki/xacro">
-    <xacro:property name="wheel_width" value="0.02" />
-    <xacro:property name="wheel_radius" value="0.04" />
+    <!-- <xacro:property name="wheel_width" value="0.02" />
+    <xacro:property name="wheel_radius" value="0.04" /> -->
+    <xacro:property name="wheel_width" value="0.025" />
+    <xacro:property name="wheel_radius" value="0.16" />
     <xacro:macro name="agribot_wheel" params="name">
         <link name="${name}">
@@ -19,5 +21,6 @@
           <inertial>
             <origin xyz="0 0 0" />
-            <mass value="0.01" />
+            <!-- <mass value="0.01" /> -->
+            <mass value="0.50" />
             <inertia ixx="0.001" ixy="0.0" ixz="0.0"
                      iyy="0.001" iyz="0.0"
