Commit message: Added IMU,GPS and magnetometer plugins.

File: urdf/agribot.urdf.xacro (robot description, xacro)
@@ -61,4 +61,70 @@
       <wheelSeparation> ${chassis_width+wheel_width} </wheelSeparation>
       <wheelRadius> ${wheel_radius} </wheelRadius>
+      <chasisLength>${chassis_length-2*wheel_radius}</chasisLength>
+    </plugin>
+  </gazebo>
+  <link name="imu_link"/>
+  <joint name="imu_joint" type="fixed">
+    <parent link="chassis_link"/>
+    <child link="imu_link" />
+    <origin xyz="0 0 0" rpy="0 0 0"/>
+  </joint>
+  <gazebo>
+    <plugin name="imu_cotroller" filename="libhector_gazebo_ros_imu.so">
+      <updateRate>10</updateRate>
+      <robotNamespace>agribot</robotNamespace>
+      <bodyName>imu_link</bodyName>
+      <frameId>imu_link</frameId>
+      <topicName>imu</topicName>
+      <rpyOffset>0 0 0</rpyOffset>
+      <xyzOffset>0 0 0</xyzOffset>
+      <gaussianNoise>0.00000001</gaussianNoise>
+      <accelDrift>0.00000001 0.00000001 0.00000001</accelDrift>
+      <accelDriftFrequency>0.00000001 0.00000001 0.00000001</accelDriftFrequency>
+      <accelGaussianNoise>0.00000001 0.00000001 0.00000001</accelGaussianNoise>
+      <rateDrift>0.0 0.0 0.0</rateDrift>
+      <rateDriftFrequency>0.0 0.0 0.0</rateDriftFrequency>
+      <rateGaussianNoise>0.0 0.0 0.0</rateGaussianNoise>
+      <headingDrift>0.0 0.0 0.0</headingDrift>
+      <headingDriftFrequency>0.0 0.0 0.0</headingDriftFrequency>
+      <headingGaussianNoise>0.0 0.0 0.0</headingGaussianNoise>
+    </plugin>
+  </gazebo>
+  <link name="gps_link"/>
+  <joint name="gps_joint" type="fixed">
+    <parent link="chassis_link"/>
+    <child link="gps_link" />
+    <origin xyz="0 0 0" rpy="0 0 0"/>
+  </joint>
+  <gazebo>
+    <plugin name="gps_controller" filename="libhector_gazebo_ros_gps.so">
+      <updateRate>10.0</updateRate>
+      <robotNamespace>agribot</robotNamespace>
+      <bodyName>gps_link</bodyName>
+      <frameId>gps_link</frameId>
+      <topicName>fix</topicName>
+      <velocityTopicName>fix_velocity</velocityTopicName>
+      <drift>5.0 5.0 5.0</drift>
+      <gaussianNoise>0.1 0.1 0.1</gaussianNoise>
+      <velocityDrift>0 0 0</velocityDrift>
+      <velocityGaussianNoise>0.1 0.1 0.1</velocityGaussianNoise>
+    </plugin>
+  </gazebo>
+  <link name="magnetic_link"/>
+  <joint name="magnetic_joint" type="fixed">
+    <parent link="chassis_link"/>
+    <child link="magnetic_link" />
+    <origin xyz="0 0 0" rpy="0 0 0"/>
+  </joint>
+  <gazebo>
+    <plugin name="magnetic_controller" filename="libhector_gazebo_ros_magnetic.so">
+      <updateRate>10.0</updateRate>
+      <robotNamespace>agribot</robotNamespace>
+      <bodyName>magnetic_link</bodyName>
+      <topicName>magnetic_field</topicName>
+      <drift>5.0 5.0 5.0</drift>
+      <gaussianNoise>0.1 0.1 0.1</gaussianNoise>
+      <velocityDrift>0 0 0</velocityDrift>
+      <velocityGaussianNoise>0.1 0.1 0.1</velocityGaussianNoise>
     </plugin>
   </gazebo>

Commit message: Added all sensors.

File: urdf/agribot.urdf.xacro (robot description, xacro)
@@ -16,5 +16,5 @@
     <parent link="chassis_link"/>
     <child link="front_cart_link"/>
-    <limit lower="${-M_PI/4}" upper="${M_PI/4}" effort="1000.0" velocity="1000.0"/>
+    <limit lower="${-45*M_PI/180}" upper="${45*M_PI/180}" effort="1000.0" velocity="1000.0"/>
     <origin xyz="${(chassis_length/2)-cart_lenght/2} 0.0 ${(chassis_height+cart_height)/(-2)}" rpy="0 0 0"/>
     <axis xyz="0 0 1"/>
@@ -38,5 +38,5 @@
     <parent link="chassis_link"/>
     <child link="back_cart_link"/>
-    <limit lower="${-M_PI/4}" upper="${M_PI/4}"  effort="1000.0" velocity="1000.0"/>
+    <limit lower="${-45*M_PI/180}" upper="${45*M_PI/180}"  effort="1000.0" velocity="1000.0"/>
     <origin xyz="${-(chassis_length/2)+cart_lenght/2} 0.0 ${(chassis_height+cart_height)/(-2)}" rpy="0 0 0"/>
     <axis xyz="0 0 1"/>
@@ -64,7 +64,18 @@
     </plugin>
   </gazebo>
+  <link name="inclinometer_link"/>
+  <joint name="inclinometer_joint" type="fixed">
+    <parent link="chassis_link"/>
+    <child link="inclinometer_link" />
+    <origin xyz="0 0 0" rpy="0 0 0"/>
+  </joint>
   <gazebo>
     <plugin name="inclinometer_controller" filename="libgazebo_inclinometer.so">
-      <inclinometerLink>"base_footprint"</inclinometerLink>
+      <inclinometerLink>"inclinometer_link"</inclinometerLink>
+    </plugin>
+  </gazebo>
+  <gazebo>
+    <plugin name="heading_controller" filename="libgazebo_heading.so">
+      <headingLink>"gps_link"</headingLink>
     </plugin>
   </gazebo>
@@ -76,7 +87,7 @@
   </joint>
   <gazebo>
-    <plugin name="imu_cotroller" filename="libhector_gazebo_ros_imu.so">
+    <plugin name="imu_cotroller" filename="libgazebo_imu.so">
       <updateRate>10</updateRate>
-      <robotNamespace>simulation</robotNamespace>
+      <robotNamespace>agribot</robotNamespace>
       <bodyName>imu_link</bodyName>
       <frameId>imu_link</frameId>
@@ -103,7 +114,7 @@
   </joint>
   <gazebo>
-    <plugin name="gps_controller" filename="libhector_gazebo_ros_gps.so">
+    <plugin name="gps_controller" filename="libgazebo_gps.so">
       <updateRate>10.0</updateRate>
-      <robotNamespace>simulation</robotNamespace>
+      <robotNamespace>agribot</robotNamespace>
       <bodyName>gps_link</bodyName>
       <frameId>gps_link</frameId>
@@ -123,7 +134,7 @@
   </joint>
   <gazebo>
-    <plugin name="magnetic_controller" filename="libhector_gazebo_ros_magnetic.so">
+    <plugin name="magnetic_controller" filename="libgazebo_magnetic.so">
       <updateRate>10.0</updateRate>
-      <robotNamespace>simulation</robotNamespace>
+      <robotNamespace>agribot</robotNamespace>
       <bodyName>magnetic_link</bodyName>
       <topicName>magnetic_field</topicName>

Commit message: Splitted sensors into separate xacro.

File: urdf/agribot.urdf.xacro (robot description, xacro)
@@ -3,4 +3,5 @@
   <xacro:include filename="$(find agribot_description)/urdf/common_properties.xacro"/>
   <xacro:include filename="$(find agribot_description)/urdf/agribot.gazebo"/>
+  <xacro:include filename="$(find agribot_description)/urdf/sensors.xacro"/>
   <xacro:include filename="$(find agribot_description)/urdf/basic_links/cart.xacro"/>
   <xacro:include filename="$(find agribot_description)/urdf/basic_links/wheel.xacro"/>
@@ -64,84 +65,4 @@
     </plugin>
   </gazebo>
-  <link name="inclinometer_link"/>
-  <joint name="inclinometer_joint" type="fixed">
-    <parent link="chassis_link"/>
-    <child link="inclinometer_link" />
-    <origin xyz="0 0 0" rpy="0 0 0"/>
-  </joint>
-  <gazebo>
-    <plugin name="inclinometer_controller" filename="libgazebo_inclinometer.so">
-      <inclinometerLink>"inclinometer_link"</inclinometerLink>
-    </plugin>
-  </gazebo>
-  <gazebo>
-    <plugin name="heading_controller" filename="libgazebo_heading.so">
-      <headingLink>"gps_link"</headingLink>
-    </plugin>
-  </gazebo>
-  <link name="imu_link"/>
-  <joint name="imu_joint" type="fixed">
-    <parent link="chassis_link"/>
-    <child link="imu_link" />
-    <origin xyz="0 0 0" rpy="0 0 0"/>
-  </joint>
-  <gazebo>
-    <plugin name="imu_cotroller" filename="libgazebo_imu.so">
-      <updateRate>10</updateRate>
-      <robotNamespace>agribot</robotNamespace>
-      <bodyName>imu_link</bodyName>
-      <frameId>imu_link</frameId>
-      <topicName>imu</topicName>
-      <rpyOffset>0 0 0</rpyOffset>
-      <xyzOffset>0 0 0</xyzOffset>
-      <gaussianNoise>0.00000001</gaussianNoise>
-      <accelDrift>0.00000001 0.00000001 0.00000001</accelDrift>
-      <accelDriftFrequency>0.00000001 0.00000001 0.00000001</accelDriftFrequency>
-      <accelGaussianNoise>0.00000001 0.00000001 0.00000001</accelGaussianNoise>
-      <rateDrift>0.0 0.0 0.0</rateDrift>
-      <rateDriftFrequency>0.0 0.0 0.0</rateDriftFrequency>
-      <rateGaussianNoise>0.0 0.0 0.0</rateGaussianNoise>
-      <headingDrift>0.0 0.0 0.0</headingDrift>
-      <headingDriftFrequency>0.0 0.0 0.0</headingDriftFrequency>
-      <headingGaussianNoise>0.0 0.0 0.0</headingGaussianNoise>
-    </plugin>
-  </gazebo>
-  <link name="gps_link"/>
-  <joint name="gps_joint" type="fixed">
-    <parent link="chassis_link"/>
-    <child link="gps_link" />
-    <origin xyz="0 0 0" rpy="0 0 0"/>
-  </joint>
-  <gazebo>
-    <plugin name="gps_controller" filename="libgazebo_gps.so">
-      <updateRate>10.0</updateRate>
-      <robotNamespace>agribot</robotNamespace>
-      <bodyName>gps_link</bodyName>
-      <frameId>gps_link</frameId>
-      <topicName>fix</topicName>
-      <velocityTopicName>fix_velocity</velocityTopicName>
-      <drift>5.0 5.0 5.0</drift>
-      <gaussianNoise>0.1 0.1 0.1</gaussianNoise>
-      <velocityDrift>0 0 0</velocityDrift>
-      <velocityGaussianNoise>0.1 0.1 0.1</velocityGaussianNoise>
-    </plugin>
-  </gazebo>
-  <link name="magnetic_link"/>
-  <joint name="magnetic_joint" type="fixed">
-    <parent link="chassis_link"/>
-    <child link="magnetic_link" />
-    <origin xyz="0 0 0" rpy="0 0 0"/>
-  </joint>
-  <gazebo>
-    <plugin name="magnetic_controller" filename="libgazebo_magnetic.so">
-      <updateRate>10.0</updateRate>
-      <robotNamespace>agribot</robotNamespace>
-      <bodyName>magnetic_link</bodyName>
-      <topicName>magnetic_field</topicName>
-      <drift>5.0 5.0 5.0</drift>
-      <gaussianNoise>0.1 0.1 0.1</gaussianNoise>
-      <velocityDrift>0 0 0</velocityDrift>
-      <velocityGaussianNoise>0.1 0.1 0.1</velocityGaussianNoise>
-    </plugin>
-  </gazebo>
+  <xacro:agribot_sensors/>
 </robot>

Commit message: Add front_cart_footprint to agribot.urdf

File: urdf/agribot.urdf.xacro (robot description, xacro)
@@ -14,4 +14,10 @@
   </joint>
   <xacro:agribot_chassis name="chassis_link" />
+  <joint name="front_cart_joint_fixed" type="fixed">
+      <parent link="base_footprint"/>
+      <child link="front_cart_footprint" />
+      <origin xyz="${(chassis_length/2)-cart_lenght/2} 0 0" rpy="0 0 0"/>
+  </joint>
+  <link name="front_cart_footprint"/>
   <joint name="front_cart_joint" type="revolute">
     <parent link="chassis_link"/>

Commit message: Change organisation of launch files: separate robot_model and robot_model_robomaker launches. Add use_perception_sensors arg to agribot.urdf.xacro

File: urdf/agribot.urdf.xacro (robot description, xacro)
@@ -2,9 +2,11 @@
 <robot name="agribot" xmlns:xacro="http://ros.org/wiki/xacro">
   <xacro:include filename="$(find agribot_description)/urdf/common_properties.xacro"/>
-  <xacro:include filename="$(find agribot_description)/urdf/sensors.xacro"/>
+  <xacro:include filename="$(find agribot_description)/urdf/basic_sensors.xacro"/>
+  <xacro:include filename="$(find agribot_description)/urdf/perception_sensors.xacro"/>
   <xacro:include filename="$(find agribot_description)/urdf/basic_links/cart.xacro"/>
   <xacro:include filename="$(find agribot_description)/urdf/basic_links/wheel.xacro"/>
   <xacro:include filename="$(find agribot_description)/urdf/basic_links/support.xacro"/>
   <xacro:include filename="$(find agribot_description)/urdf/agribot.gazebo"/>
+  <xacro:arg name="use_perception_sensors" default="false" />
   <link name="base_footprint"/>
   <joint name="chassis_joint" type="fixed">
@@ -64,4 +66,9 @@
   </joint>
   <xacro:agribot_wheel name="back_right_wheel_link" />
-  <xacro:agribot_sensors/>
+  <!-- Load basic sensors -->
+  <xacro:basic_sensors/>
+  <!-- Load perception sensors -->
+  <xacro:if value="$(arg use_perception_sensors)">
+    <xacro:perception_sensors/>
+  </xacro:if>
 </robot>

File: urdf/basic_sensors.xacro (robot description, xacro)
@@ -1,9 +1,8 @@
 <robot name="sensors" xmlns:xacro="http://ros.org/wiki/xacro">
-    <xacro:include filename="$(find agribot_description)/urdf/perception_sensors.xacro"/>
     <xacro:include filename="$(find agribot_description)/urdf/basic_sensors/imu/imu.xacro"/>
     <xacro:include filename="$(find agribot_description)/urdf/basic_sensors/gps/gps.xacro"/>
     <xacro:include filename="$(find agribot_description)/urdf/basic_sensors/inclinometer/inclinometer.xacro"/>
     <xacro:include filename="$(find agribot_description)/urdf/basic_sensors/magnetometer/magnetometer.xacro"/>
-    <xacro:macro name="agribot_sensors">
+    <xacro:macro name="basic_sensors">
         <!-- Moderna vineyard coordinates -->
         <xacro:property name="reference_latitude"   value="51.26662409135839"/>
@@ -62,6 +61,4 @@
             <!-- <xacro:property name="noise"                value="1.1e-5"/> -->
         </xacro:magnetometer>
-        <!-- Add perception sensors -->
-        <!-- <xacro:perception_sensors /> -->
     </xacro:macro>
 </robot>

File: urdf/perception_sensors.xacro (robot description, xacro)
@@ -24,5 +24,5 @@
             <xacro:property name="hz"                   value="1.0"/>
             <xacro:property name="visualize"            value="false"/>
-        </xacro:benewake_ce30_c>
+        </xacro:benewake_ce30_c> -->
         <xacro:livox_horizon>
             <origin xyz="1.3 0 1.25" rpy="0 0.5 0" />
@@ -33,5 +33,5 @@
             <xacro:property name="visualize"            value="false"/>
         </xacro:livox_horizon>
-        <xacro:robosense_bpearl>
+        <!-- <xacro:robosense_bpearl>
             <origin xyz="1.3 0 1.25" rpy="0 ${M_PI/2} 0" />
             <xacro:property name="parent"               value="base_footprint"/>

Commit message: Add proper mass and inertia to urdf. Remove wheel geometry

File: urdf/agribot.urdf.xacro (robot description, xacro)
@@ -5,7 +5,7 @@
   <xacro:include filename="$(find agribot_description)/urdf/perception_sensors.xacro"/>
   <xacro:include filename="$(find agribot_description)/urdf/tools_sensors.xacro"/>
+  <xacro:include filename="$(find agribot_description)/urdf/basic_links/chassis.xacro"/>
   <xacro:include filename="$(find agribot_description)/urdf/basic_links/cart.xacro"/>
   <xacro:include filename="$(find agribot_description)/urdf/basic_links/wheel.xacro"/>
-  <xacro:include filename="$(find agribot_description)/urdf/basic_links/support.xacro"/>
   <xacro:include filename="$(find agribot_description)/urdf/agribot.gazebo"/>
   <xacro:arg name="use_perception_sensors" default="false" />
@@ -14,5 +14,5 @@
     <parent link="base_footprint"/>
     <child link="chassis_link" />
-    <origin xyz="0 0 ${3*wheel_radius+chassis_height/2}" rpy="0 0 0"/>
+    <origin xyz="0 0 ${(chassis_height/2)+(cart_height/2)+2*wheel_radius}" rpy="0 0 0"/>
   </joint>
   <xacro:agribot_chassis name="chassis_link" />
@@ -34,5 +34,5 @@
     <parent link="front_cart_link"/>
     <child link="front_left_wheel_link"/>
-    <origin xyz="0.0 ${(chassis_width+wheel_width)/2} ${-wheel_radius}" rpy="${-M_PI/2} 0 0"/>
+    <origin xyz="0.0 ${(cart_width+wheel_width)/2} ${-cart_height/2}" rpy="${-M_PI/2} 0 0"/>
     <axis xyz="0 0 1"/>
   </joint>
@@ -41,5 +41,5 @@
     <parent link="front_cart_link"/>
     <child link="front_right_wheel_link"/>
-    <origin xyz="0.0 ${-(chassis_width+wheel_width)/2} ${-wheel_radius}" rpy="${-M_PI/2} 0 0"/>
+    <origin xyz="0.0 ${-(cart_width+wheel_width)/2} ${-cart_height/2}" rpy="${-M_PI/2} 0 0"/>
     <axis xyz="0 0 1"/>
   </joint>
@@ -56,5 +56,5 @@
     <parent link="back_cart_link"/>
     <child link="back_left_wheel_link"/>
-    <origin xyz="0.0 ${(chassis_width+wheel_width)/2} ${-wheel_radius}" rpy="${-M_PI/2} 0 0"/>
+    <origin xyz="0.0 ${(cart_width+wheel_width)/2} ${-cart_height/2}" rpy="${-M_PI/2} 0 0"/>
     <axis xyz="0 0 1"/>
   </joint>
@@ -63,5 +63,5 @@
     <parent link="back_cart_link"/>
     <child link="back_right_wheel_link"/>
-    <origin xyz="0.0 ${-(chassis_width+wheel_width)/2} ${-wheel_radius}" rpy="${-M_PI/2} 0 0"/>
+    <origin xyz="0.0 ${-(cart_width+wheel_width)/2} ${-cart_height/2}" rpy="${-M_PI/2} 0 0"/>
     <axis xyz="0 0 1"/>
   </joint>

File: urdf/basic_links/cart.xacro (robot description, xacro)
@@ -1,8 +1,7 @@
 <robot name="base" xmlns:xacro="http://ros.org/wiki/xacro">
-    <xacro:include filename="$(find agribot_description)/urdf/basic_links/wheel.xacro"/>
-    <xacro:include filename="$(find agribot_description)/urdf/basic_links/chassis.xacro"/>
-    <xacro:property name="cart_lenght" value="${wheel_radius*2}" />
-    <xacro:property name="cart_width" value="${chassis_width}" />
-    <xacro:property name="cart_height" value="${wheel_radius*2}" />
+    <xacro:property name="cart_lenght" value="0.4" />
+    <xacro:property name="cart_width" value="0.6" />
+    <xacro:property name="cart_height" value="0.3" />
+    <xacro:property name="cart_mass" value="500" />
     <xacro:macro name="agribot_cart" params="name">
         <link name="${name}">
@@ -22,22 +21,23 @@
           <collision>
             <xacro:if value="${name == 'back_cart_link'}">
-              <origin xyz="-0.25 0.0 0.3" rpy="0 0 1.57"/>
+              <origin xyz="0.0 0.0 -0.01" rpy="0 0 0"/>
               <material name="white"/>
             </xacro:if>
             <xacro:if value="${name == 'front_cart_link'}">
-              <origin xyz="0.25 0.0 0.3" rpy="0 0 -1.57"/>
+              <origin xyz="0.0 0.0 -0.01" rpy="0 0 0"/>
               <material name="green"/>
             </xacro:if>
             <geometry>
-              <mesh filename="package://agribot_description/meshes/agribot_cart.stl" scale="0.01 0.01 0.01"/>
+               <box size="${cart_lenght} ${cart_width} ${cart_height}" />
             </geometry>
           </collision>
           <inertial>
             <origin xyz="0.0 0.0 0.0" rpy="0 0 0"/>
-            <!-- <mass value="1"/> -->
-            <mass value="1.00"/>
-            <inertia ixx="0.01" ixy="0.0" ixz="0.0"
-                     iyy="0.01" iyz="0.0"
-                     izz="0.01" />
+            <!-- Moments of inertia taken from-->
+            <!-- https://en.wikipedia.org/wiki/List_of_moments_of_inertia#List_of_3D_inertia_tensors-->
+            <mass value="${cart_mass}"/>
+            <inertia ixx="${cart_mass*(cart_height*cart_height+cart_width*cart_width)/12}" ixy="0.0" ixz="0.0"
+                     iyy="${cart_mass*(cart_lenght*cart_lenght+cart_width*cart_width)/12}" iyz="0.0"
+                     izz="${cart_mass*(cart_lenght*cart_lenght+cart_height*cart_height)/12}" />
           </inertial>
         </link>

File: urdf/basic_links/chassis.xacro (robot description, xacro)
@@ -1,9 +1,7 @@
 <robot name="chassis" xmlns:xacro="http://ros.org/wiki/xacro">
-    <!-- <xacro:property name="chassis_length" value="1" />
-    <xacro:property name="chassis_width" value="0.2" />
-    <xacro:property name="chassis_height" value="0.2" /> -->
     <xacro:property name="chassis_length" value="2.42" />
     <xacro:property name="chassis_width" value="1.05" />
     <xacro:property name="chassis_height" value="1.3" />
+    <xacro:property name="chassis_mass" value="2000" />
     <xacro:macro name="agribot_chassis" params="name">
         <link name="${name}">
@@ -16,7 +14,7 @@
           </visual>
           <collision>
-            <origin xyz="0.0 0.0 0" rpy="0 0 1.57"/>
+            <origin xyz="0.0 0.0 0" rpy="0 0 0"/>
             <geometry>
-              <mesh filename="package://agribot_description/meshes/agribot_chassis.stl" scale="0.01 0.01 0.01"/>
+               <box size="${chassis_length} ${chassis_width} ${chassis_height}" />
             </geometry>
             <material name="green"/>
@@ -24,9 +22,10 @@
           <inertial>
             <origin xyz="0.0 0.0 0.0" rpy="0 0 0"/>
-            <!-- <mass value="10"/> -->
-            <mass value="1.600"/>
-            <inertia ixx="0.01" ixy="0.0" ixz="0.0"
-                     iyy="0.01" iyz="0.0"
-                     izz="0.01" />
+            <!-- Moments of inertia taken from-->
+            <!-- https://en.wikipedia.org/wiki/List_of_moments_of_inertia#List_of_3D_inertia_tensors-->
+            <mass value="${chassis_mass}"/>
+            <inertia ixx="${chassis_mass*(chassis_height*chassis_height+chassis_width*chassis_width)/12}" ixy="0.0" ixz="0.0"
+                     iyy="${chassis_mass*(chassis_length*chassis_length+chassis_width*chassis_width)/12}" iyz="0.0"
+                     izz="${chassis_mass*(chassis_length*chassis_length+chassis_height*chassis_height)/12}" />
           </inertial>
         </link>

File: urdf/basic_links/wheel.xacro (robot description, xacro)
@@ -1,9 +1,14 @@
 <robot name="wheel" xmlns:xacro="http://ros.org/wiki/xacro">
-    <!-- <xacro:property name="wheel_width" value="0.02" />
-    <xacro:property name="wheel_radius" value="0.04" /> -->
-    <xacro:property name="wheel_width" value="0.025" />
-    <xacro:property name="wheel_radius" value="0.16" />
+    <xacro:property name="wheel_width" value="0.2" />
+    <xacro:property name="wheel_radius" value="0.2" />
+    <xacro:property name="wheel_mass" value="500" />
     <xacro:macro name="agribot_wheel" params="name">
         <link name="${name}">
+          <visual>
+            <origin rpy="0 0 0" xyz="0 0 0"/>
+            <geometry>
+              <cylinder length="${wheel_width}" radius="${wheel_radius}"/>
+            </geometry>
+          </visual>
           <collision>
             <origin rpy="0 0 0" xyz="0 0 0"/>
@@ -14,9 +19,10 @@
           <inertial>
             <origin xyz="0 0 0" />
-            <!-- <mass value="0.01" /> -->
-            <mass value="0.50" />
-            <inertia ixx="0.001" ixy="0.0" ixz="0.0"
-                     iyy="0.001" iyz="0.0"
-                     izz="0.001" />
+            <!-- Moments of inertia taken from-->
+            <!-- https://en.wikipedia.org/wiki/List_of_moments_of_inertia#List_of_3D_inertia_tensors-->
+            <mass value="${wheel_mass}" />
+            <inertia ixx="${wheel_mass*(3*wheel_radius*wheel_radius+wheel_width*wheel_width)/12}" ixy="0.0" ixz="0.0"
+                     iyy="${wheel_mass*(3*wheel_radius*wheel_radius+wheel_width*wheel_width)/12}" iyz="0.0"
+                     izz="${wheel_mass*(wheel_radius*wheel_radius)/2}" />
           </inertial>
         </link>

Commit message: Remove front_cart_joint_fixed

File: urdf/agribot.urdf.xacro (robot description, xacro)
@@ -17,10 +17,4 @@
   </joint>
   <xacro:agribot_chassis name="chassis_link" />
-  <joint name="front_cart_joint_fixed" type="fixed">
-      <parent link="base_footprint"/>
-      <child link="front_cart_footprint" />
-      <origin xyz="${(chassis_length/2)-cart_lenght/2} 0 0" rpy="0 0 0"/>
-  </joint>
-  <link name="front_cart_footprint"/>
   <joint name="front_cart_joint" type="revolute">
     <parent link="chassis_link"/>
