Commit message: Add stiffness and damping coefficient only to wheels

File: urdf/agribot.urdf.xacro (robot description, xacro)
@@ -8,5 +8,4 @@
   <xacro:include filename="$(find agribot_description)/urdf/basic_links/cart.xacro"/>
   <xacro:include filename="$(find agribot_description)/urdf/basic_links/wheel.xacro"/>
-  <xacro:include filename="$(find agribot_description)/urdf/agribot.gazebo"/>
   <xacro:arg name="perception_sensors" default="false" />
   <link name="base_footprint"/>
@@ -61,4 +60,17 @@
   </joint>
   <xacro:agribot_wheel name="back_right_wheel_link" />
+ <gazebo>
+    <plugin name="agribot_controller" filename="libgazebo_ros_agribot.so">
+      <wheelSeparation> ${chassis_width+wheel_width} </wheelSeparation>
+      <wheelRadius> ${wheel_radius} </wheelRadius>
+      <chasisLength>${chassis_length-2*wheel_radius}</chasisLength>
+      <broadcastTF>false</broadcastTF> <!-- set this paremeter to false when localization is used-->
+      <odometryTopic>/agribot/odometry</odometryTopic>
+      <encoderTopic>/agribot/encoder/caterpillar</encoderTopic>
+      <odometryFrame>odom</odometryFrame>
+      <robotBaseFrame>base_footprint</robotBaseFrame>
+      <updateRate>10.000000</updateRate>
+    </plugin>
+  </gazebo>
   <!-- Load basic sensors -->
   <xacro:basic_sensors/>

File: urdf/basic_links/wheel.xacro (robot description, xacro)
@@ -1,6 +1,6 @@
 <robot name="wheel" xmlns:xacro="http://ros.org/wiki/xacro">
     <xacro:property name="wheel_width" value="0.2" />
-    <xacro:property name="wheel_radius" value="0.2" />
-    <xacro:property name="wheel_mass" value="500" />
+    <xacro:property name="wheel_radius" value="0.16" />
+    <xacro:property name="wheel_mass" value="50" />
     <xacro:macro name="agribot_wheel" params="name">
         <link name="${name}">
@@ -27,4 +27,10 @@
           </inertial>
         </link>
+        <gazebo reference="${name}">
+          <mu1>0.1</mu1>
+          <mu2>0.1</mu2>
+          <kp>5e9</kp>
+          <kd>10.0</kd>
+        </gazebo>
     </xacro:macro>
 </robot>

Commit message: Revert basic links parameters

File: urdf/agribot.urdf.xacro (robot description, xacro)
@@ -5,7 +5,7 @@
   <xacro:include filename="$(find agribot_description)/urdf/perception_sensors.xacro"/>
   <xacro:include filename="$(find agribot_description)/urdf/tools_sensors.xacro"/>
+  <xacro:include filename="$(find agribot_description)/urdf/basic_links/wheel.xacro"/>
   <xacro:include filename="$(find agribot_description)/urdf/basic_links/chassis.xacro"/>
   <xacro:include filename="$(find agribot_description)/urdf/basic_links/cart.xacro"/>
-  <xacro:include filename="$(find agribot_description)/urdf/basic_links/wheel.xacro"/>
   <xacro:arg name="perception_sensors" default="false" />
   <link name="base_footprint"/>

File: urdf/basic_links/cart.xacro (robot description, xacro)
@@ -1,6 +1,6 @@
 <robot name="base" xmlns:xacro="http://ros.org/wiki/xacro">
-    <xacro:property name="cart_lenght" value="0.4" />
-    <xacro:property name="cart_width" value="0.6" />
-    <xacro:property name="cart_height" value="0.3" />
+    <xacro:property name="cart_lenght" value="${wheel_radius*2}" />
+    <xacro:property name="cart_width" value="${chassis_width}" />
+    <xacro:property name="cart_height" value="${wheel_radius*2}" />
     <xacro:property name="cart_mass" value="500" />
     <xacro:macro name="agribot_cart" params="name">
@@ -21,9 +21,9 @@
           <collision>
             <xacro:if value="${name == 'back_cart_link'}">
-              <origin xyz="0.0 0.0 -0.01" rpy="0 0 0"/>
+              <origin xyz="0.0 0.0 0.0" rpy="0 0 0"/>
               <material name="white"/>
             </xacro:if>
             <xacro:if value="${name == 'front_cart_link'}">
-              <origin xyz="0.0 0.0 -0.01" rpy="0 0 0"/>
+              <origin xyz="0.0 0.0 0.0" rpy="0 0 0"/>
               <material name="green"/>
             </xacro:if>

File: urdf/basic_links/wheel.xacro (robot description, xacro)
@@ -1,4 +1,4 @@
 <robot name="wheel" xmlns:xacro="http://ros.org/wiki/xacro">
-    <xacro:property name="wheel_width" value="0.2" />
+    <xacro:property name="wheel_width" value="0.025" />
     <xacro:property name="wheel_radius" value="0.16" />
     <xacro:property name="wheel_mass" value="50" />

Commit message: Add perception plugins argument

File: urdf/agribot.urdf.xacro (robot description, xacro)
@@ -9,4 +9,5 @@
   <xacro:include filename="$(find agribot_description)/urdf/basic_links/cart.xacro"/>
   <xacro:arg name="perception_sensors" default="false" />
+  <xacro:arg name="perception_plugins" default="true" />
   <link name="base_footprint"/>
   <joint name="chassis_joint" type="fixed">
@@ -79,5 +80,7 @@
   <!-- Load perception sensors -->
   <xacro:if value="$(arg perception_sensors)">
-    <xacro:perception_sensors/>
+    <xacro:perception_sensors>
+      <xacro:property name="perception_plugins_arg" value="$(arg perception_plugins)"/>
+    </xacro:perception_sensors>
   </xacro:if>
 </robot>

File: urdf/basic_sensors/lidar/livox_horizon.xacro (robot description, xacro)
@@ -9,4 +9,5 @@
                             hz:=^
                             visualize:=^
+                            perception_plugins:=^
                             ">
         <!-- Call basic velodyne lidar and pass arguments -->
@@ -28,4 +29,5 @@
             <xacro:property name="max_vertical_angle"       value="${12.55*M_PI/180.0}"/>
             <xacro:property name="resolution"               value="0.001"/>
+            <xacro:property name="perception_plugins_arg"       value="${perception_plugins}"/>
         </xacro:velodyne>
     </xacro:macro>

File: urdf/basic_sensors/lidar/velodyne.xacro (robot description, xacro)
@@ -19,4 +19,5 @@
                         resolution:=^
                         collision_range:=0.3
+                        perception_plugins_arg:=^
                         ">
         <joint name="${name}_base_mount_joint" type="fixed">
@@ -68,46 +69,48 @@
             </visual>
         </link>
-        <!-- Gazebo requires the velodyne_gazebo_plugins package -->
-        <gazebo reference="${name}_link">
-            <sensor type="ray" name="${name}">
-                <pose>0 0 0 0 0 0</pose>
-                <visualize>${visualize}</visualize>
-                <update_rate>${hz}</update_rate>
-                <always_on>true</always_on>
-                <ray>
-                    <scan>
-                        <horizontal>
-                            <samples>${samples}</samples>
-                            <resolution>1</resolution>
-                            <min_angle>${min_horizontal_angle}</min_angle>
-                            <max_angle>${max_horizontal_angle}</max_angle>
-                        </horizontal>
-                        <vertical>
-                            <samples>${lasers}</samples>
-                            <resolution>1</resolution>
-                            <min_angle>${min_vertical_angle}</min_angle>
-                            <max_angle>${max_vertical_angle}</max_angle>
-                        </vertical>
-                    </scan>
-                    <range>
-                        <min>${min_range}</min>
-                        <max>${max_range}</max>
-                        <resolution>${resolution}</resolution>
-                    </range>
-                    <noise>
-                        <type>gaussian</type>
-                        <mean>0.0</mean>
-                        <stddev>0.0</stddev>
-                    </noise>
-                </ray>
-                <plugin name="gazebo_ros_laser_controller" filename="libgazebo_ros_velodyne_laser.so">
-                    <topicName>${topic}</topicName>
-                    <frameName>${name}_link</frameName>
-                    <min_range>${min_range}</min_range>
-                    <max_range>${max_range}</max_range>
-                    <gaussianNoise>${noise}</gaussianNoise>
-                </plugin>
-            </sensor>
-        </gazebo>
+        <xacro:if value="${perception_plugins_arg}">
+            <!-- Gazebo requires the velodyne_gazebo_plugins package -->
+            <gazebo reference="${name}_link">
+                <sensor type="ray" name="${name}">
+                    <pose>0 0 0 0 0 0</pose>
+                    <visualize>${visualize}</visualize>
+                    <update_rate>${hz}</update_rate>
+                    <always_on>true</always_on>
+                    <ray>
+                        <scan>
+                            <horizontal>
+                                <samples>${samples}</samples>
+                                <resolution>1</resolution>
+                                <min_angle>${min_horizontal_angle}</min_angle>
+                                <max_angle>${max_horizontal_angle}</max_angle>
+                            </horizontal>
+                            <vertical>
+                                <samples>${lasers}</samples>
+                                <resolution>1</resolution>
+                                <min_angle>${min_vertical_angle}</min_angle>
+                                <max_angle>${max_vertical_angle}</max_angle>
+                            </vertical>
+                        </scan>
+                        <range>
+                            <min>${min_range}</min>
+                            <max>${max_range}</max>
+                            <resolution>${resolution}</resolution>
+                        </range>
+                        <noise>
+                            <type>gaussian</type>
+                            <mean>0.0</mean>
+                            <stddev>0.0</stddev>
+                        </noise>
+                    </ray>
+                    <plugin name="gazebo_ros_laser_controller" filename="libgazebo_ros_velodyne_laser.so">
+                        <topicName>${topic}</topicName>
+                        <frameName>${name}_link</frameName>
+                        <min_range>${min_range}</min_range>
+                        <max_range>${max_range}</max_range>
+                        <gaussianNoise>${noise}</gaussianNoise>
+                    </plugin>
+                </sensor>
+            </gazebo>
+        </xacro:if>
     </xacro:macro>
 </robot>

File: urdf/basic_sensors/sonar/balluff_sonar.xacro (robot description, xacro)
@@ -9,4 +9,5 @@
                             hz:=^
                             visualize:=^
+                            perception_plugins:=^
                             ">
         <!-- Call basic sonar and pass arguments -->
@@ -32,4 +33,5 @@
             <!-- <xacro:property name="max_vertical_angle"       value="${5.9*M_PI/180.0}"/> -->
             <xacro:property name="resolution"               value="0.0018"/>
+            <xacro:property name="perception_plugins_arg"  value="${perception_plugins}"/>
         </xacro:sonar>
     </xacro:macro>

File: urdf/basic_sensors/sonar/bosch_sonar.xacro (robot description, xacro)
@@ -9,4 +9,5 @@
                             hz:=^
                             visualize:=^
+                            perception_plugins:=^
                             ">
         <!-- Call basic sonar and pass arguments -->
@@ -27,4 +28,5 @@
             <xacro:property name="max_vertical_angle"       value="${30.0*M_PI/180.0}"/>
             <xacro:property name="resolution"               value="0.001"/>
+            <xacro:property name="perception_plugins_arg"  value="${perception_plugins}"/>
             <!-- Generation 6 BOSCH sensor -->
             <!-- <xacro:property name="min_range"                value="0.15"/>

File: urdf/basic_sensors/sonar/sonar.xacro (robot description, xacro)
@@ -16,4 +16,5 @@
                           max_vertical_angle:=^
                           resolution:=^
+                          perception_plugins_arg:=^
                           ">
         <joint name="${name}_joint" type="fixed">
@@ -23,38 +24,40 @@
         </joint>
         <link name="${name}_link"/>
-        <gazebo reference="${name}_link">
-            <sensor type="ray" name="${name}">
-                <pose>0 0 0 0 0 0</pose>
-                <visualize>${visualize}</visualize>
-                <update_rate>${hz}</update_rate>
-                <always_on>true</always_on>
-                <ray>
-                <scan>
-                    <horizontal>
-                        <samples>10</samples>
-                        <resolution>1</resolution>
-                        <min_angle>${min_horizontal_angle}</min_angle>
-                        <max_angle>${max_horizontal_angle}</max_angle>
-                    </horizontal>
-                    <vertical>
-                        <samples>10</samples>
-                        <resolution>1</resolution>
-                        <min_angle>${min_vertical_angle}</min_angle>
-                        <max_angle>${max_vertical_angle}</max_angle>
-                    </vertical>
-                </scan>
-                <range>
-                    <min>${min_range}</min>
-                    <max>${max_range}</max>
-                    <resolution>${resolution}</resolution>
-                </range>
-                </ray>
-                <plugin name="gazebo_ros_front_sonar_controller" filename="libhector_gazebo_ros_sonar.so">
-                    <topicName>${topic}</topicName>
-                    <frameId>${name}_link</frameId>
-                    <gaussianNoise>${noise}</gaussianNoise>
-                </plugin>
-            </sensor>
-        </gazebo>
+        <xacro:if value="${perception_plugins_arg}">
+            <gazebo reference="${name}_link">
+                <sensor type="ray" name="${name}">
+                    <pose>0 0 0 0 0 0</pose>
+                    <visualize>${visualize}</visualize>
+                    <update_rate>${hz}</update_rate>
+                    <always_on>true</always_on>
+                    <ray>
+                    <scan>
+                        <horizontal>
+                            <samples>10</samples>
+                            <resolution>1</resolution>
+                            <min_angle>${min_horizontal_angle}</min_angle>
+                            <max_angle>${max_horizontal_angle}</max_angle>
+                        </horizontal>
+                        <vertical>
+                            <samples>10</samples>
+                            <resolution>1</resolution>
+                            <min_angle>${min_vertical_angle}</min_angle>
+                            <max_angle>${max_vertical_angle}</max_angle>
+                        </vertical>
+                    </scan>
+                    <range>
+                        <min>${min_range}</min>
+                        <max>${max_range}</max>
+                        <resolution>${resolution}</resolution>
+                    </range>
+                    </ray>
+                    <plugin name="gazebo_ros_front_sonar_controller" filename="libhector_gazebo_ros_sonar.so">
+                        <topicName>${topic}</topicName>
+                        <frameId>${name}_link</frameId>
+                        <gaussianNoise>${noise}</gaussianNoise>
+                    </plugin>
+                </sensor>
+            </gazebo>
+        </xacro:if>
     </xacro:macro>
 </robot>

File: urdf/perception_sensors.xacro (robot description, xacro)
@@ -7,5 +7,7 @@
   <xacro:include filename="$(find agribot_description)/urdf/basic_sensors/sonar/bosch_sonar.xacro"/>
   <xacro:include filename="$(find agribot_description)/urdf/basic_sensors/sonar/balluff_sonar.xacro"/>
-  <xacro:macro name="perception_sensors">
+  <xacro:macro  name="perception_sensors"
+              params="perception_plugins_arg:=^
+                     ">
     <!-- Lidars -->
     <!-- <xacro:velodyne16>
@@ -32,4 +34,5 @@
       <xacro:property name="hz"                   value="1.0"/>
       <xacro:property name="visualize"            value="false"/>
+      <xacro:property name="perception_plugins"   value="${perception_plugins_arg}"/>
     </xacro:livox_horizon>
     <!-- <xacro:robosense_bpearl>
@@ -49,4 +52,5 @@
       <xacro:property name="hz"                   value="10.0"/>
       <xacro:property name="visualize"            value="true"/>
+      <xacro:property name="perception_plugins"   value="${perception_plugins_arg}"/>
     </xacro:bosch_sonar>
     <xacro:bosch_sonar>
@@ -57,4 +61,5 @@
       <xacro:property name="hz"                   value="10.0"/>
       <xacro:property name="visualize"            value="true"/>
+      <xacro:property name="perception_plugins"   value="${perception_plugins_arg}"/>
     </xacro:bosch_sonar>
     <xacro:balluff_sonar>
@@ -73,4 +78,5 @@
       <xacro:property name="hz"                   value="10.0"/>
       <xacro:property name="visualize"            value="true"/>
+      <xacro:property name="perception_plugins"   value="${perception_plugins_arg}"/>
     </xacro:bosch_sonar>
     <xacro:bosch_sonar>
@@ -81,4 +87,5 @@
       <xacro:property name="hz"                   value="10.0"/>
       <xacro:property name="visualize"            value="true"/>
+      <xacro:property name="perception_plugins"   value="${perception_plugins_arg}"/>
     </xacro:bosch_sonar>
     <!-- Left side sonars -->
@@ -90,4 +97,5 @@
       <xacro:property name="hz"                   value="10.0"/>
       <xacro:property name="visualize"            value="true"/>
+      <xacro:property name="perception_plugins"   value="${perception_plugins_arg}"/>
     </xacro:bosch_sonar>
     <xacro:bosch_sonar>
@@ -98,4 +106,5 @@
       <xacro:property name="hz"                   value="10.0"/>
       <xacro:property name="visualize"            value="true"/>
+      <xacro:property name="perception_plugins"   value="${perception_plugins_arg}"/>
     </xacro:bosch_sonar>
     <!-- Right side sonars -->
@@ -107,4 +116,5 @@
       <xacro:property name="hz"                   value="10.0"/>
       <xacro:property name="visualize"            value="true"/>
+      <xacro:property name="perception_plugins"   value="${perception_plugins_arg}"/>
     </xacro:bosch_sonar>
     <xacro:bosch_sonar>
@@ -115,4 +125,5 @@
       <xacro:property name="hz"                   value="10.0"/>
       <xacro:property name="visualize"            value="true"/>
+      <xacro:property name="perception_plugins"   value="${perception_plugins_arg}"/>
     </xacro:bosch_sonar>
     <!-- Back bumper sonars -->
@@ -124,4 +135,5 @@
       <xacro:property name="hz"                   value="10.0"/>
       <xacro:property name="visualize"            value="true"/>
+      <xacro:property name="perception_plugins"   value="${perception_plugins_arg}"/>
     </xacro:bosch_sonar>
     <xacro:bosch_sonar>
@@ -132,4 +144,5 @@
       <xacro:property name="hz"                   value="10.0"/>
       <xacro:property name="visualize"            value="true"/>
+      <xacro:property name="perception_plugins"   value="${perception_plugins_arg}"/>
     </xacro:bosch_sonar>
     <xacro:balluff_sonar>
@@ -140,4 +153,5 @@
       <xacro:property name="hz"                   value="10.0"/>
       <xacro:property name="visualize"            value="true"/>
+      <xacro:property name="perception_plugins"   value="${perception_plugins_arg}"/>
     </xacro:balluff_sonar>
     <xacro:bosch_sonar>
@@ -148,4 +162,5 @@
       <xacro:property name="hz"                   value="10.0"/>
       <xacro:property name="visualize"            value="true"/>
+      <xacro:property name="perception_plugins"   value="${perception_plugins_arg}"/>
     </xacro:bosch_sonar>
     <xacro:bosch_sonar>
@@ -156,4 +171,5 @@
       <xacro:property name="hz"                   value="10.0"/>
       <xacro:property name="visualize"            value="true"/>
+      <xacro:property name="perception_plugins"   value="${perception_plugins_arg}"/>
     </xacro:bosch_sonar>
   </xacro:macro>

Commit message: Adding tpl to agribot model in progress

File: urdf/agribot.urdf.xacro (robot description, xacro)
@@ -8,4 +8,5 @@
   <xacro:include filename="$(find agribot_description)/urdf/basic_links/chassis.xacro"/>
   <xacro:include filename="$(find agribot_description)/urdf/basic_links/cart.xacro"/>
+  <xacro:include filename="$(find agribot_description)/urdf/basic_links/tpl.xacro"/>
   <xacro:arg name="perception_sensors" default="false" />
   <xacro:arg name="perception_plugins" default="true" />
@@ -61,4 +62,11 @@
   </joint>
   <xacro:agribot_wheel name="back_right_wheel_link" />
+  <joint name="back_tpl_joint" type="fixed">
+    <parent link="back_cart_link"/>
+    <child link="back_tpl_link"/>
+    <origin xyz="0.0 ${-(cart_width+wheel_width)} ${-cart_height}" rpy="0 0 0"/>
+    <axis xyz="0 0 1"/>
+  </joint>
+  <xacro:agribot_tpl name="back_tpl_link" />
  <gazebo>
     <plugin name="agribot_controller" filename="libgazebo_ros_agribot.so">
