Commit message: TPL model in progress

File: urdf/agribot.urdf.xacro (robot description, xacro)
@@ -48,4 +48,11 @@
   </joint>
   <xacro:agribot_cart name="back_cart_link" />
+  <joint name="front_tpl_joint" type="fixed">
+    <parent link="front_cart_link"/>
+    <child link="front_tpl_link"/>
+    <origin xyz="${(cart_lenght+tpl_len)/2} 0.0 -0.02" rpy="0 0 0"/>
+    <axis xyz="0 0 1"/>
+  </joint>
+  <xacro:agribot_tpl_base name="front_tpl_link" />
   <joint name="back_left_wheel_joint" type="continuous">
     <parent link="back_cart_link"/>
@@ -65,8 +72,15 @@
     <parent link="back_cart_link"/>
     <child link="back_tpl_link"/>
-    <origin xyz="0.0 ${-(cart_width+wheel_width)} ${-cart_height}" rpy="0 0 0"/>
+    <origin xyz="${-(cart_lenght+tpl_len)/2} 0.0 -0.02" rpy="0 0 0"/>
     <axis xyz="0 0 1"/>
   </joint>
-  <xacro:agribot_tpl name="back_tpl_link" />
+  <xacro:agribot_tpl_base name="back_tpl_link" />
+  <joint name="back_tpl_cyl_joint" type="fixed">
+    <parent link="back_tpl_link"/>
+    <child link="back_tpl_cyl_link"/>
+    <origin xyz="${-(cart_lenght+tpl_len)/2} 0.0 -0.02" rpy="0 0 0"/>
+    <axis xyz="0 0 1"/>
+  </joint>
+  <xacro:agribot_tpl_cylinder name="back_tpl_cyl_link" />
  <gazebo>
     <plugin name="agribot_controller" filename="libgazebo_ros_agribot.so">

File: urdf/basic_links/tpl.xacro (robot description, xacro)
@@ -1,28 +1,78 @@
 <robot name="tpl" xmlns:xacro="http://ros.org/wiki/xacro">
-    <xacro:property name="tpl_width" value="0.25" />
-    <xacro:property name="tpl_mass" value="500" />
-    <xacro:property name="tpl_radius" value="500" />
-        <xacro:macro name="agribot_tpl" params="name">
-        <link name="${name}">
-          <visual>
-            <geometry>
-              <cylinder length="${tpl_width}" radius="${tpl_radius}"/>
-            </geometry>
-          </visual>
-          <collision>
-            <geometry>
-               <cylinder length="${tpl_width}" radius="${tpl_radius}"/>
-            </geometry>
-          </collision>
-          <inertial>
-            <origin xyz="0.0 0.0 0.0" rpy="0 0 0"/>
-            <!-- Moments of inertia taken from-->
-            <!-- https://en.wikipedia.org/wiki/List_of_moments_of_inertia#List_of_3D_inertia_tensors-->
-            <mass value="${tpl_mass}"/>
-            <inertia ixx="0.0" ixy="0.0" ixz="0.0"
-                     iyy="0.0" iyz="0.0"
-                     izz="0.0}" />
-          </inertial>
-        </link>
+    <xacro:property name="tpl_len" value="0.7" />
+    <xacro:property name="tpl_wid" value="0.2" />
+    <xacro:property name="tpl_hei" value="0.1" />
+    <xacro:property name="tpl_mass" value="300" />
+    <xacro:property name="cyl_width" value="1.0" />
+    <xacro:property name="cyl_radius" value="0.2" />
+    <xacro:macro name="agribot_tpl_base" params="name">
+      <link name="${name}">
+        <visual>
+          <xacro:if value="${name == 'back_tpl_link'}">
+            <material name="white"/>
+          </xacro:if>
+          <xacro:if value="${name == 'front_tpl_link'}">
+            <material name="green"/>
+          </xacro:if>
+          <geometry>
+            <box size="${tpl_len} ${tpl_wid} ${tpl_hei}"/>
+          </geometry>
+        </visual>
+        <collision>
+          <xacro:if value="${name == 'back_tpl_link'}">
+            <material name="white"/>
+          </xacro:if>
+          <xacro:if value="${name == 'front_tpl_link'}">
+            <material name="green"/>
+          </xacro:if>
+          <geometry>
+            <box size="${tpl_len} ${tpl_wid} ${tpl_hei}"/>
+          </geometry>
+        </collision>
+        <inertial>
+          <origin xyz="0.0 0.0 0.0" rpy="0 0 0"/>
+          <!-- Moments of inertia taken from-->
+          <!-- https://en.wikipedia.org/wiki/List_of_moments_of_inertia#List_of_3D_inertia_tensors-->
+          <mass value="${tpl_mass}"/>
+          <inertia ixx="0.0" ixy="0.0" ixz="0.0"
+                   iyy="0.0" iyz="0.0"
+                   izz="0.0" />
+        </inertial>
+      </link>
+    </xacro:macro>
+    <xacro:macro name="agribot_tpl_cylinder" params="name">
+      <link name="${name}">
+        <visual>
+          <xacro:if value="${name == 'back_tpl_link'}">
+            <material name="white"/>
+          </xacro:if>
+          <xacro:if value="${name == 'front_tpl_link'}">
+            <material name="green"/>
+          </xacro:if>
+          <geometry>
+            <cylinder length="${cyl_width}" radius="${cyl_radius}"/>
+          </geometry>
+        </visual>
+        <collision>
+          <xacro:if value="${name == 'back_tpl_link'}">
+            <material name="white"/>
+          </xacro:if>
+          <xacro:if value="${name == 'front_tpl_link'}">
+            <material name="green"/>
+          </xacro:if>
+          <geometry>
+            <box size="${tpl_len} ${tpl_wid} ${tpl_hei}"/>
+          </geometry>
+        </collision>
+        <inertial>
+          <origin xyz="0.0 0.0 0.0" rpy="0 0 0"/>
+          <!-- Moments of inertia taken from-->
+          <!-- https://en.wikipedia.org/wiki/List_of_moments_of_inertia#List_of_3D_inertia_tensors-->
+          <mass value="${tpl_mass}"/>
+          <inertia ixx="0.0" ixy="0.0" ixz="0.0"
+                   iyy="0.0" iyz="0.0"
+                   izz="0.0" />
+        </inertial>
+      </link>
     </xacro:macro>
 </robot>

Commit message: TPL revolute hitches mechanism implemented. Prismatic hitch work in progress

File: urdf/agribot.urdf.xacro (robot description, xacro)
@@ -48,11 +48,13 @@
   </joint>
   <xacro:agribot_cart name="back_cart_link" />
+  <!-- begin front TPL -->
   <joint name="front_tpl_joint" type="fixed">
     <parent link="front_cart_link"/>
-    <child link="front_tpl_link"/>
-    <origin xyz="${(cart_lenght+tpl_len)/2} 0.0 -0.02" rpy="0 0 0"/>
+    <child link="front_tpl_base_link"/>
+    <origin xyz="${(cart_lenght+tpl_base_len)/2} 0.0 -0.02" rpy="0 0 0"/>
     <axis xyz="0 0 1"/>
   </joint>
-  <xacro:agribot_tpl_base name="front_tpl_link" />
+  <xacro:agribot_tpl_base name="front_tpl_base_link" />
+  <!-- end front TPL -->
   <joint name="back_left_wheel_joint" type="continuous">
     <parent link="back_cart_link"/>
@@ -69,18 +71,42 @@
   </joint>
   <xacro:agribot_wheel name="back_right_wheel_link" />
-  <joint name="back_tpl_joint" type="fixed">
+  <!-- begin back TPL -->
+  <joint name="back_tpl_base_joint" type="fixed">
     <parent link="back_cart_link"/>
-    <child link="back_tpl_link"/>
-    <origin xyz="${-(cart_lenght+tpl_len)/2} 0.0 -0.02" rpy="0 0 0"/>
+    <child link="back_tpl_base_link"/>
+    <origin xyz="${-(cart_lenght+tpl_base_len)/2} 0.0 -0.02" rpy="0 0 0"/>
     <axis xyz="0 0 1"/>
   </joint>
-  <xacro:agribot_tpl_base name="back_tpl_link" />
-  <joint name="back_tpl_cyl_joint" type="fixed">
-    <parent link="back_tpl_link"/>
-    <child link="back_tpl_cyl_link"/>
-    <origin xyz="${-(cart_lenght+tpl_len)/2} 0.0 -0.02" rpy="0 0 0"/>
+  <xacro:agribot_tpl_base name="back_tpl_base_link" />
+  <joint name="back_tpl_cylinder_joint" type="revolute">
+    <parent link="back_tpl_base_link"/>
+    <child link="back_tpl_cylinder_link"/>
+    <origin xyz="${-(tpl_base_len)/2} 0.0 0.0" rpy="${M_PI/2} ${-M_PI/18} 0"/>
+    <limit lower="${-60*M_PI/180}" upper="${15*M_PI/180}"  effort="1000.0" velocity="1000.0"/>
     <axis xyz="0 0 1"/>
   </joint>
-  <xacro:agribot_tpl_cylinder name="back_tpl_cyl_link" />
+  <xacro:agribot_tpl_cylinder name="back_tpl_cylinder_link" />
+  <joint name="back_tpl_revolute_hitch_left_joint" type="fixed">
+    <parent link="back_tpl_cylinder_link"/>
+    <child link="back_tpl_revolute_hitch_left_link"/>
+    <origin xyz="${-(tpl_rev_hit_len-tpl_cyl_radius)/2} 0.0 ${-(tpl_cyl_width)/2}" rpy="0 0 0"/>
+    <axis xyz="0 0 1"/>
+  </joint>
+  <xacro:agribot_tpl_revolute_hitch name="back_tpl_revolute_hitch_left_link" />
+  <joint name="back_tpl_revolute_hitch_right_joint" type="fixed">
+    <parent link="back_tpl_cylinder_link"/>
+    <child link="back_tpl_revolute_hitch_right_link"/>
+    <origin xyz="${-(tpl_rev_hit_len-tpl_cyl_radius)/2} 0.0 ${(tpl_cyl_width)/2}" rpy="0 0 0"/>
+    <axis xyz="0 0 1"/>
+  </joint>
+  <xacro:agribot_tpl_revolute_hitch name="back_tpl_revolute_hitch_right_link" />
+  <joint name="back_tpl_bases_joint" type="fixed">
+    <parent link="back_tpl_base_link"/>
+    <child link="back_tpl_up_hit_base"/>
+    <origin xyz="${-(tpl_base_len)/2} 0.0 0.0" rpy="0 0 0"/>
+    <axis xyz="0 0 1"/>
+  </joint>
+  <xacro:agribot_tpl_upper_hitch_base name="back_tpl_up_hit_base" />
+  <!-- end back TPL -->
  <gazebo>
     <plugin name="agribot_controller" filename="libgazebo_ros_agribot.so">

File: urdf/basic_links/tpl.xacro (robot description, xacro)
@@ -1,31 +1,38 @@
 <robot name="tpl" xmlns:xacro="http://ros.org/wiki/xacro">
-    <xacro:property name="tpl_len" value="0.7" />
-    <xacro:property name="tpl_wid" value="0.2" />
-    <xacro:property name="tpl_hei" value="0.1" />
-    <xacro:property name="tpl_mass" value="300" />
-    <xacro:property name="cyl_width" value="1.0" />
-    <xacro:property name="cyl_radius" value="0.2" />
+    <xacro:property name="tpl_base_len" value="0.7" />
+    <xacro:property name="tpl_base_wid" value="0.2" />
+    <xacro:property name="tpl_base_hei" value="0.1" />
+    <xacro:property name="tpl_base_mass" value="300" />
+    <xacro:property name="tpl_cyl_width" value="0.85" />
+    <xacro:property name="tpl_cyl_radius" value="0.05" />
+    <xacro:property name="tpl_cyl_mass" value="50" />
+    <xacro:property name="tpl_rev_hit_len" value="0.5" />
+    <xacro:property name="tpl_rev_hit_wid" value="0.1" />
+    <xacro:property name="tpl_rev_hit_hei" value="0.05" />
+    <xacro:property name="tpl_upper_hit_base_len" value="0.5" />
+    <xacro:property name="tpl_upper_hit_base_wid" value="0.1" />
+    <xacro:property name="tpl_upper_hit_base_hei" value="0.05" />
     <xacro:macro name="agribot_tpl_base" params="name">
       <link name="${name}">
         <visual>
-          <xacro:if value="${name == 'back_tpl_link'}">
+          <xacro:if value="${name == 'back_tpl_base_link'}">
             <material name="white"/>
           </xacro:if>
-          <xacro:if value="${name == 'front_tpl_link'}">
+          <xacro:if value="${name == 'front_tpl_base_link'}">
             <material name="green"/>
           </xacro:if>
           <geometry>
-            <box size="${tpl_len} ${tpl_wid} ${tpl_hei}"/>
+            <box size="${tpl_base_len} ${tpl_base_wid} ${tpl_base_hei}"/>
           </geometry>
         </visual>
         <collision>
-          <xacro:if value="${name == 'back_tpl_link'}">
+          <xacro:if value="${name == 'back_tpl_base_link'}">
             <material name="white"/>
           </xacro:if>
-          <xacro:if value="${name == 'front_tpl_link'}">
+          <xacro:if value="${name == 'front_tpl_base_link'}">
             <material name="green"/>
           </xacro:if>
           <geometry>
-            <box size="${tpl_len} ${tpl_wid} ${tpl_hei}"/>
+            <box size="${tpl_base_len} ${tpl_base_wid} ${tpl_base_hei}"/>
           </geometry>
         </collision>
@@ -34,5 +41,5 @@
           <!-- Moments of inertia taken from-->
           <!-- https://en.wikipedia.org/wiki/List_of_moments_of_inertia#List_of_3D_inertia_tensors-->
-          <mass value="${tpl_mass}"/>
+          <mass value="${tpl_base_mass}"/>
           <inertia ixx="0.0" ixy="0.0" ixz="0.0"
                    iyy="0.0" iyz="0.0"
@@ -44,23 +51,23 @@
       <link name="${name}">
         <visual>
-          <xacro:if value="${name == 'back_tpl_link'}">
+          <xacro:if value="${name == 'back_tpl_cylinder_link'}">
             <material name="white"/>
           </xacro:if>
-          <xacro:if value="${name == 'front_tpl_link'}">
+          <xacro:if value="${name == 'front_tpl_cylinder_link'}">
             <material name="green"/>
           </xacro:if>
           <geometry>
-            <cylinder length="${cyl_width}" radius="${cyl_radius}"/>
+            <cylinder length="${tpl_cyl_width}" radius="${tpl_cyl_radius}"/>
           </geometry>
         </visual>
         <collision>
-          <xacro:if value="${name == 'back_tpl_link'}">
+          <xacro:if value="${name == 'back_tpl_cylinder_link'}">
             <material name="white"/>
           </xacro:if>
-          <xacro:if value="${name == 'front_tpl_link'}">
+          <xacro:if value="${name == 'front_tpl_cylinder_link'}">
             <material name="green"/>
           </xacro:if>
           <geometry>
-            <box size="${tpl_len} ${tpl_wid} ${tpl_hei}"/>
+            <cylinder length="${tpl_cyl_width}" radius="${tpl_cyl_radius}"/>
           </geometry>
         </collision>
@@ -69,5 +76,87 @@
           <!-- Moments of inertia taken from-->
           <!-- https://en.wikipedia.org/wiki/List_of_moments_of_inertia#List_of_3D_inertia_tensors-->
-          <mass value="${tpl_mass}"/>
+          <mass value="${tpl_cyl_mass}"/>
+          <inertia ixx="0.0" ixy="0.0" ixz="0.0"
+                   iyy="0.0" iyz="0.0"
+                   izz="0.0" />
+        </inertial>
+      </link>
+    </xacro:macro>
+    <xacro:macro name="agribot_tpl_revolute_hitch" params="name">
+      <link name="${name}">
+        <visual>
+          <xacro:if value="${name == 'back_tpl_revolute_hitch_right_link'}">
+            <material name="white"/>
+          </xacro:if>
+          <xacro:if value="${name == 'back_tpl_revolute_hitch_left_link'}">
+            <material name="white"/>
+          </xacro:if>
+          <xacro:if value="${name == 'front_tpl_revolute_hitch_right_link'}">
+            <material name="green"/>
+          </xacro:if>
+          <xacro:if value="${name == 'front_tpl_revolute_hitch_left_link'}">
+            <material name="green"/>
+          </xacro:if>
+          <geometry>
+            <box size="${tpl_rev_hit_len} ${tpl_rev_hit_wid} ${tpl_rev_hit_hei}"/>
+          </geometry>
+        </visual>
+        <collision>
+          <xacro:if value="${name == 'back_tpl_revolute_hitch_right_link'}">
+            <material name="white"/>
+          </xacro:if>
+          <xacro:if value="${name == 'back_tpl_revolute_hitch_left_link'}">
+            <material name="white"/>
+          </xacro:if>
+          <xacro:if value="${name == 'front_tpl_revolute_hitch_right_link'}">
+            <material name="green"/>
+          </xacro:if>
+          <xacro:if value="${name == 'front_tpl_revolute_hitch_left_link'}">
+            <material name="green"/>
+          </xacro:if>
+          <geometry>
+            <box size="${tpl_rev_hit_len} ${tpl_rev_hit_wid} ${tpl_rev_hit_hei}"/>
+          </geometry>
+        </collision>
+        <inertial>
+          <origin xyz="0.0 0.0 0.0" rpy="0 0 0"/>
+          <!-- Moments of inertia taken from-->
+          <!-- https://en.wikipedia.org/wiki/List_of_moments_of_inertia#List_of_3D_inertia_tensors-->
+          <mass value="${tpl_base_mass}"/>
+          <inertia ixx="0.0" ixy="0.0" ixz="0.0"
+                   iyy="0.0" iyz="0.0"
+                   izz="0.0" />
+        </inertial>
+      </link>
+    </xacro:macro>
+    <xacro:macro name="agribot_tpl_upper_hitch_base" params="name">
+      <link name="${name}">
+        <visual>
+          <xacro:if value="${name == 'back_tpl_up_hit_base'}">
+            <material name="white"/>
+          </xacro:if>
+          <xacro:if value="${name == 'front_tpl_up_hit_base'}">
+            <material name="green"/>
+          </xacro:if>
+          <geometry>
+            <box size="${tpl_upper_hit_base_len} ${tpl_upper_hit_base_wid} ${tpl_upper_hit_base_hei}"/>
+          </geometry>
+        </visual>
+        <collision>
+          <xacro:if value="${name == 'back_tpl_up_hit_base'}">
+            <material name="white"/>
+          </xacro:if>
+          <xacro:if value="${name == 'front_tpl_up_hit_base'}">
+            <material name="green"/>
+          </xacro:if>
+          <geometry>
+            <box size="${tpl_upper_hit_base_len} ${tpl_upper_hit_base_wid} ${tpl_upper_hit_base_hei}"/>
+          </geometry>
+        </collision>
+        <inertial>
+          <origin xyz="0.0 0.0 0.0" rpy="0 0 0"/>
+          <!-- Moments of inertia taken from-->
+          <!-- https://en.wikipedia.org/wiki/List_of_moments_of_inertia#List_of_3D_inertia_tensors-->
+          <mass value="${tpl_base_mass}"/>
           <inertia ixx="0.0" ixy="0.0" ixz="0.0"
                    iyy="0.0" iyz="0.0"
