Commit message: Revolute as well as prismatic hiches are implemented

File: urdf/agribot.urdf.xacro (robot description, xacro)
@@ -79,5 +79,5 @@
   </joint>
   <xacro:agribot_tpl_base name="back_tpl_base_link" />
-  <joint name="back_tpl_cylinder_joint" type="revolute">
+  <joint name="back_tpl_lower_hitches_revolute_joint" type="revolute">
     <parent link="back_tpl_base_link"/>
     <child link="back_tpl_cylinder_link"/>
@@ -103,9 +103,31 @@
   <joint name="back_tpl_bases_joint" type="fixed">
     <parent link="back_tpl_base_link"/>
-    <child link="back_tpl_up_hit_base"/>
-    <origin xyz="${-(tpl_base_len)/2} 0.0 0.0" rpy="0 0 0"/>
+    <child link="back_tpl_up_hit_base_link"/>
+    <origin xyz="${-(tpl_base_len)/2} 0.0 ${(tpl_upper_hit_base_len)/2}" rpy="0 ${M_PI/2} 0"/>
     <axis xyz="0 0 1"/>
   </joint>
-  <xacro:agribot_tpl_upper_hitch_base name="back_tpl_up_hit_base" />
+  <xacro:agribot_tpl_upper_hitch_base name="back_tpl_up_hit_base_link" />
+  <joint name="back_tpl_upper_hitch_revolute_joint" type="revolute">
+    <parent link="back_tpl_up_hit_base_link"/>
+    <child link="back_tpl_upper_hitch_cylinder_link"/>
+    <origin xyz="${-(tpl_base_len)/2} 0.0 0.0" rpy="${M_PI/2} ${-M_PI/18} 0"/>
+    <limit lower="${-10*M_PI/180}" upper="${80*M_PI/180}"  effort="1000.0" velocity="1000.0"/>
+    <axis xyz="0 0 1"/>
+  </joint>
+  <xacro:agribot_tpl_upper_hitch_cylinder name="back_tpl_upper_hitch_cylinder_link" />
+  <joint name="back_tpl_upper_hitch_prism_joint_base_joint" type="fixed">
+    <parent link="back_tpl_upper_hitch_cylinder_link"/>
+    <child link="back_tpl_upper_hitch_prism_joint_base_link"/>
+    <origin xyz="${-(tpl_upper_hitch_prism_base_len)/2} 0.0 0.0" rpy="0 0 0"/>
+    <axis xyz="0 0 1"/>
+  </joint>
+  <xacro:agribot_tpl_upper_hitch_prism_joint_base name="back_tpl_upper_hitch_prism_joint_base_link" />
+  <joint name="back_tpl_upper_hitch_prismatic_joint" type="prismatic">
+    <parent link="back_tpl_upper_hitch_prism_joint_base_link"/>
+    <child link="back_tpl_upper_hitch_prism_joint_core_link"/>
+    <limit effort="1000.0" lower="${-tpl_upper_hitch_prism_core_len+0.05}" upper="0.0" velocity="0.5"/>
+    <origin rpy="0 0 0" xyz="-0.05 0 0"/>
+  </joint>
+  <xacro:agribot_tpl_upper_hitch_prism_joint_core name="back_tpl_upper_hitch_prism_joint_core_link" />
   <!-- end back TPL -->
  <gazebo>

File: urdf/basic_links/tpl.xacro (robot description, xacro)
@@ -10,7 +10,16 @@
     <xacro:property name="tpl_rev_hit_wid" value="0.1" />
     <xacro:property name="tpl_rev_hit_hei" value="0.05" />
-    <xacro:property name="tpl_upper_hit_base_len" value="0.5" />
-    <xacro:property name="tpl_upper_hit_base_wid" value="0.1" />
-    <xacro:property name="tpl_upper_hit_base_hei" value="0.05" />
+    <xacro:property name="tpl_upper_hit_base_len" value="0.7" />
+    <xacro:property name="tpl_upper_hit_base_wid" value="0.2" />
+    <xacro:property name="tpl_upper_hit_base_hei" value="0.1" />
+    <xacro:property name="tpl_upper_hit_base_cyl_width" value="0.2" />
+    <xacro:property name="tpl_upper_hit_base_cyl_radius" value="0.05" />
+    <xacro:property name="tpl_upper_hit_base_cyl_mass" value="10" />
+    <xacro:property name="tpl_upper_hitch_prism_base_len" value="0.5" />
+    <xacro:property name="tpl_upper_hitch_prism_base_wid" value="0.1" />
+    <xacro:property name="tpl_upper_hitch_prism_base_hei" value="0.1" />
+    <xacro:property name="tpl_upper_hitch_prism_core_len" value="0.5" />
+    <xacro:property name="tpl_upper_hitch_prism_core_wid" value="0.075" />
+    <xacro:property name="tpl_upper_hitch_prism_core_hei" value="0.075" />
     <xacro:macro name="agribot_tpl_base" params="name">
       <link name="${name}">
@@ -133,8 +142,8 @@
       <link name="${name}">
         <visual>
-          <xacro:if value="${name == 'back_tpl_up_hit_base'}">
-            <material name="white"/>
-          </xacro:if>
-          <xacro:if value="${name == 'front_tpl_up_hit_base'}">
+          <xacro:if value="${name == 'back_tpl_up_hit_base_link'}">
+            <material name="white"/>
+          </xacro:if>
+          <xacro:if value="${name == 'front_tpl_up_hit_base_link'}">
             <material name="green"/>
           </xacro:if>
@@ -144,8 +153,8 @@
         </visual>
         <collision>
-          <xacro:if value="${name == 'back_tpl_up_hit_base'}">
-            <material name="white"/>
-          </xacro:if>
-          <xacro:if value="${name == 'front_tpl_up_hit_base'}">
+          <xacro:if value="${name == 'back_tpl_up_hit_base_link'}">
+            <material name="white"/>
+          </xacro:if>
+          <xacro:if value="${name == 'front_tpl_up_hit_base_link'}">
             <material name="green"/>
           </xacro:if>
@@ -165,3 +174,108 @@
       </link>
     </xacro:macro>
+    <xacro:macro name="agribot_tpl_upper_hitch_cylinder" params="name">
+      <link name="${name}">
+        <visual>
+          <xacro:if value="${name == 'back_tpl_upper_hitch_cylinder_link'}">
+            <material name="white"/>
+          </xacro:if>
+          <xacro:if value="${name == 'front_tpl_upper_hitch_cylinder_link'}">
+            <material name="green"/>
+          </xacro:if>
+          <geometry>
+            <cylinder length="${tpl_upper_hit_base_cyl_width}" radius="${tpl_upper_hit_base_cyl_radius}"/>
+          </geometry>
+        </visual>
+        <collision>
+          <xacro:if value="${name == 'back_tpl_upper_hitch_cylinder_link'}">
+            <material name="white"/>
+          </xacro:if>
+          <xacro:if value="${name == 'front_tpl_upper_hitch_cylinder_link'}">
+            <material name="green"/>
+          </xacro:if>
+          <geometry>
+            <cylinder length="${tpl_upper_hit_base_cyl_width}" radius="${tpl_upper_hit_base_cyl_radius}"/>
+          </geometry>
+        </collision>
+        <inertial>
+          <origin xyz="0.0 0.0 0.0" rpy="0 0 0"/>
+          <!-- Moments of inertia taken from-->
+          <!-- https://en.wikipedia.org/wiki/List_of_moments_of_inertia#List_of_3D_inertia_tensors-->
+          <mass value="${tpl_cyl_mass}"/>
+          <inertia ixx="0.0" ixy="0.0" ixz="0.0"
+                   iyy="0.0" iyz="0.0"
+                   izz="0.0" />
+        </inertial>
+      </link>
+    </xacro:macro>
+    <xacro:macro name="agribot_tpl_upper_hitch_prism_joint_base" params="name">
+      <link name="${name}">
+        <visual>
+          <xacro:if value="${name == 'back_tpl_upper_hitch_prism_joint_base_link'}">
+            <material name="white"/>
+          </xacro:if>
+          <xacro:if value="${name == 'front_tpl_upper_hitch_prism_joint_base_link'}">
+            <material name="green"/>
+          </xacro:if>
+          <geometry>
+            <box size="${tpl_upper_hitch_prism_base_len} ${tpl_upper_hitch_prism_base_wid} ${tpl_upper_hitch_prism_base_hei}"/>
+          </geometry>
+        </visual>
+        <collision>
+          <xacro:if value="${name == 'back_tpl_upper_hitch_prism_joint_base_link'}">
+            <material name="white"/>
+          </xacro:if>
+          <xacro:if value="${name == 'front_tpl_upper_hitch_prism_joint_base_link'}">
+            <material name="green"/>
+          </xacro:if>
+          <geometry>
+            <box size="${tpl_upper_hitch_prism_base_len} ${tpl_upper_hitch_prism_base_wid} ${tpl_upper_hitch_prism_base_hei}"/>
+          </geometry>
+        </collision>
+        <inertial>
+          <origin xyz="0.0 0.0 0.0" rpy="0 0 0"/>
+          <!-- Moments of inertia taken from-->
+          <!-- https://en.wikipedia.org/wiki/List_of_moments_of_inertia#List_of_3D_inertia_tensors-->
+          <mass value="${tpl_base_mass}"/>
+          <inertia ixx="0.0" ixy="0.0" ixz="0.0"
+                   iyy="0.0" iyz="0.0"
+                   izz="0.0" />
+        </inertial>
+      </link>
+    </xacro:macro>
+    <xacro:macro name="agribot_tpl_upper_hitch_prism_joint_core" params="name">
+      <link name="${name}">
+        <visual>
+          <xacro:if value="${name == 'back_tpl_upper_hitch_prism_joint_core_link'}">
+            <material name="white"/>
+          </xacro:if>
+          <xacro:if value="${name == 'front_tpl_upper_hitch_prism_joint_core_link'}">
+            <material name="green"/>
+          </xacro:if>
+          <geometry>
+            <box size="${tpl_upper_hitch_prism_core_len} ${tpl_upper_hitch_prism_core_wid} ${tpl_upper_hitch_prism_core_hei}"/>
+          </geometry>
+        </visual>
+        <collision>
+          <xacro:if value="${name == 'back_tpl_upper_hitch_prism_joint_core_link'}">
+            <material name="white"/>
+          </xacro:if>
+          <xacro:if value="${name == 'front_tpl_upper_hitch_prism_joint_core_link'}">
+            <material name="green"/>
+          </xacro:if>
+          <geometry>
+            <box size="${tpl_upper_hitch_prism_core_len} ${tpl_upper_hitch_prism_core_wid} ${tpl_upper_hitch_prism_core_hei}"/>
+          </geometry>
+        </collision>
+        <inertial>
+          <origin xyz="0.0 0.0 0.0" rpy="0 0 0"/>
+          <!-- Moments of inertia taken from-->
+          <!-- https://en.wikipedia.org/wiki/List_of_moments_of_inertia#List_of_3D_inertia_tensors-->
+          <mass value="${tpl_base_mass}"/>
+          <inertia ixx="0.0" ixy="0.0" ixz="0.0"
+                   iyy="0.0" iyz="0.0"
+                   izz="0.0" />
+        </inertial>
+      </link>
+    </xacro:macro>
 </robot>

Commit message: Modified lower hitches

File: urdf/agribot.urdf.xacro (robot description, xacro)
@@ -75,5 +75,5 @@
     <parent link="back_cart_link"/>
     <child link="back_tpl_base_link"/>
-    <origin xyz="${-(cart_lenght+tpl_base_len)/2} 0.0 -0.02" rpy="0 0 0"/>
+    <origin xyz="${-(cart_lenght+tpl_base_len)/2} 0.0 ${(cart_height-tpl_base_hei)/2}" rpy="0 0 0"/>
     <axis xyz="0 0 1"/>
   </joint>
@@ -82,23 +82,37 @@
     <parent link="back_tpl_base_link"/>
     <child link="back_tpl_cylinder_link"/>
-    <origin xyz="${-(tpl_base_len)/2} 0.0 0.0" rpy="${M_PI/2} ${-M_PI/18} 0"/>
+    <origin xyz="${-(tpl_base_len)/2} 0.0 0.0" rpy="${M_PI/2} ${-M_PI/5} 0"/>
     <limit lower="${-60*M_PI/180}" upper="${15*M_PI/180}"  effort="1000.0" velocity="1000.0"/>
     <axis xyz="0 0 1"/>
   </joint>
   <xacro:agribot_tpl_cylinder name="back_tpl_cylinder_link" />
-  <joint name="back_tpl_revolute_hitch_left_joint" type="fixed">
+  <joint name="back_tpl_revolute_hitch_base_left_joint" type="fixed">
     <parent link="back_tpl_cylinder_link"/>
-    <child link="back_tpl_revolute_hitch_left_link"/>
-    <origin xyz="${-(tpl_rev_hit_len-tpl_cyl_radius)/2} 0.0 ${-(tpl_cyl_width)/2}" rpy="0 0 0"/>
+    <child link="back_tpl_revolute_hitch_base_left_link"/>
+    <origin xyz="${-(tpl_rev_hit_base_len-tpl_cyl_radius)/2} 0.0 ${-(tpl_cyl_width)/2}" rpy="0 0 0"/>
     <axis xyz="0 0 1"/>
   </joint>
-  <xacro:agribot_tpl_revolute_hitch name="back_tpl_revolute_hitch_left_link" />
+  <xacro:agribot_tpl_revolute_hitch_base name="back_tpl_revolute_hitch_base_left_link" />
+  <joint name="back_tpl_revolute_hitch_effector_left_joint" type="fixed">
+    <parent link="back_tpl_revolute_hitch_base_left_link"/>
+    <child link="back_tpl_revolute_hitch_effector_left_link"/>
+    <origin xyz="${-0.4*(tpl_rev_hit_base_len+tpl_rev_hit_effector_len)} 0.1 ${-0.22*tpl_rev_hit_effector_len}" rpy="0 ${-M_PI/6} ${-M_PI/6}"/>
+    <axis xyz="0 0 1"/>
+  </joint>
+  <xacro:agribot_tpl_revolute_hitch_effector name="back_tpl_revolute_hitch_effector_left_link" />
   <joint name="back_tpl_revolute_hitch_right_joint" type="fixed">
     <parent link="back_tpl_cylinder_link"/>
-    <child link="back_tpl_revolute_hitch_right_link"/>
-    <origin xyz="${-(tpl_rev_hit_len-tpl_cyl_radius)/2} 0.0 ${(tpl_cyl_width)/2}" rpy="0 0 0"/>
+    <child link="back_tpl_revolute_hitch_base_right_link"/>
+    <origin xyz="${-(tpl_rev_hit_base_len-tpl_cyl_radius)/2} 0.0 ${(tpl_cyl_width)/2}" rpy="0 0 0"/>
     <axis xyz="0 0 1"/>
   </joint>
-  <xacro:agribot_tpl_revolute_hitch name="back_tpl_revolute_hitch_right_link" />
+  <xacro:agribot_tpl_revolute_hitch_base name="back_tpl_revolute_hitch_base_right_link" />
+  <joint name="back_tpl_revolute_hitch_effector_right_joint" type="fixed">
+    <parent link="back_tpl_revolute_hitch_base_right_link"/>
+    <child link="back_tpl_revolute_hitch_effector_right_link"/>
+    <origin xyz="${-0.4*(tpl_rev_hit_base_len+tpl_rev_hit_effector_len)} 0.1 ${0.22*tpl_rev_hit_effector_len}" rpy="0 ${M_PI/6} ${-M_PI/6}"/>
+    <axis xyz="0 0 1"/>
+  </joint>
+  <xacro:agribot_tpl_revolute_hitch_effector name="back_tpl_revolute_hitch_effector_right_link" />
   <joint name="back_tpl_bases_joint" type="fixed">
     <parent link="back_tpl_base_link"/>

File: urdf/basic_links/tpl.xacro (robot description, xacro)
@@ -1,13 +1,16 @@
 <robot name="tpl" xmlns:xacro="http://ros.org/wiki/xacro">
-    <xacro:property name="tpl_base_len" value="0.7" />
-    <xacro:property name="tpl_base_wid" value="0.2" />
-    <xacro:property name="tpl_base_hei" value="0.1" />
+    <xacro:property name="tpl_base_len" value="0.43" />
+    <xacro:property name="tpl_base_wid" value="0.3" />
+    <xacro:property name="tpl_base_hei" value="0.05" />
     <xacro:property name="tpl_base_mass" value="300" />
-    <xacro:property name="tpl_cyl_width" value="0.85" />
-    <xacro:property name="tpl_cyl_radius" value="0.05" />
+    <xacro:property name="tpl_cyl_width" value="0.45" />
+    <xacro:property name="tpl_cyl_radius" value="${tpl_base_hei/2}" />
     <xacro:property name="tpl_cyl_mass" value="50" />
-    <xacro:property name="tpl_rev_hit_len" value="0.5" />
-    <xacro:property name="tpl_rev_hit_wid" value="0.1" />
-    <xacro:property name="tpl_rev_hit_hei" value="0.05" />
+    <xacro:property name="tpl_rev_hit_base_len" value="0.3" />
+    <xacro:property name="tpl_rev_hit_base_wid" value="${2*tpl_base_hei}" />
+    <xacro:property name="tpl_rev_hit_base_hei" value="0.05" />
+    <xacro:property name="tpl_rev_hit_effector_len" value="0.5" />
+    <xacro:property name="tpl_rev_hit_effector_wid" value="${2*tpl_base_hei}" />
+    <xacro:property name="tpl_rev_hit_effector_hei" value="0.05" />
     <xacro:property name="tpl_upper_hit_base_len" value="0.7" />
     <xacro:property name="tpl_upper_hit_base_wid" value="0.2" />
@@ -92,38 +95,85 @@
       </link>
     </xacro:macro>
-    <xacro:macro name="agribot_tpl_revolute_hitch" params="name">
-      <link name="${name}">
-        <visual>
-          <xacro:if value="${name == 'back_tpl_revolute_hitch_right_link'}">
-            <material name="white"/>
-          </xacro:if>
-          <xacro:if value="${name == 'back_tpl_revolute_hitch_left_link'}">
-            <material name="white"/>
-          </xacro:if>
-          <xacro:if value="${name == 'front_tpl_revolute_hitch_right_link'}">
-            <material name="green"/>
-          </xacro:if>
-          <xacro:if value="${name == 'front_tpl_revolute_hitch_left_link'}">
-            <material name="green"/>
-          </xacro:if>
-          <geometry>
-            <box size="${tpl_rev_hit_len} ${tpl_rev_hit_wid} ${tpl_rev_hit_hei}"/>
-          </geometry>
-        </visual>
-        <collision>
-          <xacro:if value="${name == 'back_tpl_revolute_hitch_right_link'}">
-            <material name="white"/>
-          </xacro:if>
-          <xacro:if value="${name == 'back_tpl_revolute_hitch_left_link'}">
-            <material name="white"/>
-          </xacro:if>
-          <xacro:if value="${name == 'front_tpl_revolute_hitch_right_link'}">
-            <material name="green"/>
-          </xacro:if>
-          <xacro:if value="${name == 'front_tpl_revolute_hitch_left_link'}">
-            <material name="green"/>
-          </xacro:if>
-          <geometry>
-            <box size="${tpl_rev_hit_len} ${tpl_rev_hit_wid} ${tpl_rev_hit_hei}"/>
+    <xacro:macro name="agribot_tpl_revolute_hitch_base" params="name">
+      <link name="${name}">
+        <visual>
+          <xacro:if value="${name == 'back_tpl_revolute_hitch_base_right_link'}">
+            <material name="white"/>
+          </xacro:if>
+          <xacro:if value="${name == 'back_tpl_revolute_hitch_base_left_link'}">
+            <material name="white"/>
+          </xacro:if>
+          <xacro:if value="${name == 'front_tpl_revolute_hitch_base_right_link'}">
+            <material name="green"/>
+          </xacro:if>
+          <xacro:if value="${name == 'front_tpl_revolute_hitch_base_left_link'}">
+            <material name="green"/>
+          </xacro:if>
+          <geometry>
+            <box size="${tpl_rev_hit_base_len} ${tpl_rev_hit_base_wid} ${tpl_rev_hit_base_hei}"/>
+          </geometry>
+        </visual>
+        <collision>
+          <xacro:if value="${name == 'back_tpl_revolute_hitch_base_right_link'}">
+            <material name="white"/>
+          </xacro:if>
+          <xacro:if value="${name == 'back_tpl_revolute_hitch_base_left_link'}">
+            <material name="white"/>
+          </xacro:if>
+          <xacro:if value="${name == 'front_tpl_revolute_hitch_base_right_link'}">
+            <material name="green"/>
+          </xacro:if>
+          <xacro:if value="${name == 'front_tpl_revolute_hitch_base_left_link'}">
+            <material name="green"/>
+          </xacro:if>
+          <geometry>
+            <box size="${tpl_rev_hit_base_len} ${tpl_rev_hit_base_wid} ${tpl_rev_hit_base_hei}"/>
+          </geometry>
+        </collision>
+        <inertial>
+          <origin xyz="0.0 0.0 0.0" rpy="0 0 0"/>
+          <!-- Moments of inertia taken from-->
+          <!-- https://en.wikipedia.org/wiki/List_of_moments_of_inertia#List_of_3D_inertia_tensors-->
+          <mass value="${tpl_base_mass}"/>
+          <inertia ixx="0.0" ixy="0.0" ixz="0.0"
+                   iyy="0.0" iyz="0.0"
+                   izz="0.0" />
+        </inertial>
+      </link>
+    </xacro:macro>
+    <xacro:macro name="agribot_tpl_revolute_hitch_effector" params="name">
+      <link name="${name}">
+        <visual>
+          <xacro:if value="${name == 'back_tpl_revolute_hitch_effector_right_link'}">
+            <material name="white"/>
+          </xacro:if>
+          <xacro:if value="${name == 'back_tpl_revolute_hitch_effector_left_link'}">
+            <material name="white"/>
+          </xacro:if>
+          <xacro:if value="${name == 'front_tpl_revolute_hitch_effector_right_link'}">
+            <material name="green"/>
+          </xacro:if>
+          <xacro:if value="${name == 'front_tpl_revolute_hitch_effector_left_link'}">
+            <material name="green"/>
+          </xacro:if>
+          <geometry>
+            <box size="${tpl_rev_hit_effector_len} ${tpl_rev_hit_effector_wid} ${tpl_rev_hit_effector_hei}"/>
+          </geometry>
+        </visual>
+        <collision>
+          <xacro:if value="${name == 'back_tpl_revolute_hitch_effector_right_link'}">
+            <material name="white"/>
+          </xacro:if>
+          <xacro:if value="${name == 'back_tpl_revolute_hitch_effector_left_link'}">
+            <material name="white"/>
+          </xacro:if>
+          <xacro:if value="${name == 'front_tpl_revolute_hitch_effector_right_link'}">
+            <material name="green"/>
+          </xacro:if>
+          <xacro:if value="${name == 'front_tpl_revolute_hitch_effector_left_link'}">
+            <material name="green"/>
+          </xacro:if>
+          <geometry>
+            <box size="${tpl_rev_hit_effector_len} ${tpl_rev_hit_effector_wid} ${tpl_rev_hit_effector_hei}"/>
           </geometry>
         </collision>

Commit message: Upper hitch modified

File: urdf/agribot.urdf.xacro (robot description, xacro)
@@ -83,5 +83,5 @@
     <child link="back_tpl_cylinder_link"/>
     <origin xyz="${-(tpl_base_len)/2} 0.0 0.0" rpy="${M_PI/2} ${-M_PI/5} 0"/>
-    <limit lower="${-60*M_PI/180}" upper="${15*M_PI/180}"  effort="1000.0" velocity="1000.0"/>
+    <limit lower="${-90*M_PI/180}" upper="${15*M_PI/180}"  effort="1000.0" velocity="1000.0"/>
     <axis xyz="0 0 1"/>
   </joint>
@@ -118,5 +118,5 @@
     <parent link="back_tpl_base_link"/>
     <child link="back_tpl_up_hit_base_link"/>
-    <origin xyz="${-(tpl_base_len)/2} 0.0 ${(tpl_upper_hit_base_len)/2}" rpy="0 ${M_PI/2} 0"/>
+    <origin xyz="${-0.82*tpl_base_len} 0.0 ${0.8*(tpl_upper_hit_base_len)/2}" rpy="0 ${M_PI/3.15} 0"/>
     <axis xyz="0 0 1"/>
   </joint>
@@ -125,5 +125,5 @@
     <parent link="back_tpl_up_hit_base_link"/>
     <child link="back_tpl_upper_hitch_cylinder_link"/>
-    <origin xyz="${-(tpl_base_len)/2} 0.0 0.0" rpy="${M_PI/2} ${-M_PI/18} 0"/>
+    <origin xyz="${-tpl_upper_hit_base_len/2} 0.0 0.0" rpy="${M_PI/2} ${-M_PI/18} 0"/>
     <limit lower="${-10*M_PI/180}" upper="${80*M_PI/180}"  effort="1000.0" velocity="1000.0"/>
     <axis xyz="0 0 1"/>

File: urdf/basic_links/tpl.xacro (robot description, xacro)
@@ -13,16 +13,16 @@
     <xacro:property name="tpl_rev_hit_effector_wid" value="${2*tpl_base_hei}" />
     <xacro:property name="tpl_rev_hit_effector_hei" value="0.05" />
-    <xacro:property name="tpl_upper_hit_base_len" value="0.7" />
-    <xacro:property name="tpl_upper_hit_base_wid" value="0.2" />
-    <xacro:property name="tpl_upper_hit_base_hei" value="0.1" />
-    <xacro:property name="tpl_upper_hit_base_cyl_width" value="0.2" />
-    <xacro:property name="tpl_upper_hit_base_cyl_radius" value="0.05" />
+    <xacro:property name="tpl_upper_hit_base_len" value="0.66" />
+    <xacro:property name="tpl_upper_hit_base_wid" value="0.3" />
+    <xacro:property name="tpl_upper_hit_base_hei" value="0.05" />
+    <xacro:property name="tpl_upper_hit_base_cyl_width" value="${tpl_upper_hit_base_wid}" />
+    <xacro:property name="tpl_upper_hit_base_cyl_radius" value="${tpl_cyl_radius}" />
     <xacro:property name="tpl_upper_hit_base_cyl_mass" value="10" />
     <xacro:property name="tpl_upper_hitch_prism_base_len" value="0.5" />
-    <xacro:property name="tpl_upper_hitch_prism_base_wid" value="0.1" />
-    <xacro:property name="tpl_upper_hitch_prism_base_hei" value="0.1" />
+    <xacro:property name="tpl_upper_hitch_prism_base_wid" value="0.075" />
+    <xacro:property name="tpl_upper_hitch_prism_base_hei" value="0.075" />
     <xacro:property name="tpl_upper_hitch_prism_core_len" value="0.5" />
-    <xacro:property name="tpl_upper_hitch_prism_core_wid" value="0.075" />
-    <xacro:property name="tpl_upper_hitch_prism_core_hei" value="0.075" />
+    <xacro:property name="tpl_upper_hitch_prism_core_wid" value="0.05" />
+    <xacro:property name="tpl_upper_hitch_prism_core_hei" value="0.05" />
     <xacro:macro name="agribot_tpl_base" params="name">
       <link name="${name}">
