Commit message: Front and back TPL are visualized

File: urdf/agribot.urdf.xacro (robot description, xacro)
@@ -8,5 +8,4 @@
   <xacro:include filename="$(find agribot_description)/urdf/basic_links/chassis.xacro"/>
   <xacro:include filename="$(find agribot_description)/urdf/basic_links/cart.xacro"/>
-  <xacro:include filename="$(find agribot_description)/urdf/basic_links/tpl/tpl_assembled.xacro"/>
   <xacro:arg name="perception_sensors" default="false" />
   <xacro:arg name="perception_plugins" default="true" />
@@ -48,13 +47,6 @@
   </joint>
   <xacro:agribot_cart name="back_cart_link" />
-  <!-- begin front TPL -->
-  <joint name="front_tpl_joint" type="fixed">
-    <parent link="front_cart_link"/>
-    <child link="front_tpl_base_link"/>
-    <origin xyz="${(cart_lenght+tpl_base_len)/2} 0.0 -0.02" rpy="0 0 0"/>
-    <axis xyz="0 0 1"/>
-  </joint>
-  <xacro:agribot_tpl_base name="front_tpl_base_link" />
-  <!-- end front TPL -->
+  <xacro:property name="sel_tpl" value="front"/>
+  <xacro:include filename="$(find agribot_description)/urdf/basic_links/tpl/tpl_assembled.xacro"/>
   <joint name="back_left_wheel_joint" type="continuous">
     <parent link="back_cart_link"/>
@@ -71,78 +63,6 @@
   </joint>
   <xacro:agribot_wheel name="back_right_wheel_link" />
-  <!-- begin back TPL -->
-  <joint name="back_tpl_base_joint" type="fixed">
-    <parent link="back_cart_link"/>
-    <child link="back_tpl_base_link"/>
-    <origin xyz="${-(cart_lenght+tpl_base_len)/2} 0.0 ${(cart_height-tpl_base_hei)/2}" rpy="0 0 0"/>
-    <axis xyz="0 0 1"/>
-  </joint>
-  <xacro:agribot_tpl_base name="back_tpl_base_link" />
-  <joint name="back_tpl_lower_hitches_revolute_joint" type="revolute">
-    <parent link="back_tpl_base_link"/>
-    <child link="back_tpl_cylinder_link"/>
-    <origin xyz="${-(tpl_base_len)/2} 0.0 0.0" rpy="${M_PI/2} ${-M_PI/5} 0"/>
-    <limit lower="${-90*M_PI/180}" upper="${15*M_PI/180}"  effort="1000.0" velocity="1000.0"/>
-    <axis xyz="0 0 1"/>
-  </joint>
-  <xacro:agribot_tpl_cylinder name="back_tpl_cylinder_link" />
-  <joint name="back_tpl_revolute_hitch_base_left_joint" type="fixed">
-    <parent link="back_tpl_cylinder_link"/>
-    <child link="back_tpl_revolute_hitch_base_left_link"/>
-    <origin xyz="${-(tpl_rev_hit_base_len-tpl_cyl_radius)/2} 0.0 ${-(tpl_cyl_width)/2}" rpy="0 0 0"/>
-    <axis xyz="0 0 1"/>
-  </joint>
-  <xacro:agribot_tpl_revolute_hitch_base name="back_tpl_revolute_hitch_base_left_link" />
-  <joint name="back_tpl_revolute_hitch_effector_left_joint" type="fixed">
-    <parent link="back_tpl_revolute_hitch_base_left_link"/>
-    <child link="back_tpl_revolute_hitch_effector_left_link"/>
-    <origin xyz="${-0.4*(tpl_rev_hit_base_len+tpl_rev_hit_effector_len)} 0.1 ${-0.22*tpl_rev_hit_effector_len}" rpy="0 ${-M_PI/6} ${-M_PI/6}"/>
-    <axis xyz="0 0 1"/>
-  </joint>
-  <xacro:agribot_tpl_revolute_hitch_effector name="back_tpl_revolute_hitch_effector_left_link" />
-  <joint name="back_tpl_revolute_hitch_right_joint" type="fixed">
-    <parent link="back_tpl_cylinder_link"/>
-    <child link="back_tpl_revolute_hitch_base_right_link"/>
-    <origin xyz="${-(tpl_rev_hit_base_len-tpl_cyl_radius)/2} 0.0 ${(tpl_cyl_width)/2}" rpy="0 0 0"/>
-    <axis xyz="0 0 1"/>
-  </joint>
-  <xacro:agribot_tpl_revolute_hitch_base name="back_tpl_revolute_hitch_base_right_link" />
-  <joint name="back_tpl_revolute_hitch_effector_right_joint" type="fixed">
-    <parent link="back_tpl_revolute_hitch_base_right_link"/>
-    <child link="back_tpl_revolute_hitch_effector_right_link"/>
-    <origin xyz="${-0.4*(tpl_rev_hit_base_len+tpl_rev_hit_effector_len)} 0.1 ${0.22*tpl_rev_hit_effector_len}" rpy="0 ${M_PI/6} ${-M_PI/6}"/>
-    <axis xyz="0 0 1"/>
-  </joint>
-  <xacro:agribot_tpl_revolute_hitch_effector name="back_tpl_revolute_hitch_effector_right_link" />
-  <joint name="back_tpl_bases_joint" type="fixed">
-    <parent link="back_tpl_base_link"/>
-    <child link="back_tpl_up_hit_base_link"/>
-    <origin xyz="${-0.82*tpl_base_len} 0.0 ${0.8*(tpl_upper_hit_base_len)/2}" rpy="0 ${M_PI/3.15} 0"/>
-    <axis xyz="0 0 1"/>
-  </joint>
-  <xacro:agribot_tpl_upper_hitch_base name="back_tpl_up_hit_base_link" />
-  <joint name="back_tpl_upper_hitch_revolute_joint" type="revolute">
-    <parent link="back_tpl_up_hit_base_link"/>
-    <child link="back_tpl_upper_hitch_cylinder_link"/>
-    <origin xyz="${-tpl_upper_hit_base_len/2} 0.0 0.0" rpy="${M_PI/2} ${-M_PI/18} 0"/>
-    <limit lower="${-10*M_PI/180}" upper="${80*M_PI/180}"  effort="1000.0" velocity="1000.0"/>
-    <axis xyz="0 0 1"/>
-  </joint>
-  <xacro:agribot_tpl_upper_hitch_cylinder name="back_tpl_upper_hitch_cylinder_link" />
-  <joint name="back_tpl_upper_hitch_prism_joint_base_joint" type="fixed">
-    <parent link="back_tpl_upper_hitch_cylinder_link"/>
-    <child link="back_tpl_upper_hitch_prism_joint_base_link"/>
-    <origin xyz="${-(tpl_upper_hitch_prism_base_len)/2} 0.0 0.0" rpy="0 0 0"/>
-    <axis xyz="0 0 1"/>
-  </joint>
-  <xacro:agribot_tpl_upper_hitch_prism_joint_base name="back_tpl_upper_hitch_prism_joint_base_link" />
-  <joint name="back_tpl_upper_hitch_prismatic_joint" type="prismatic">
-    <parent link="back_tpl_upper_hitch_prism_joint_base_link"/>
-    <child link="back_tpl_upper_hitch_prism_joint_core_link"/>
-    <limit effort="1000.0" lower="${-tpl_upper_hitch_prism_core_len+0.05}" upper="0.0" velocity="0.5"/>
-    <origin rpy="0 0 0" xyz="-0.05 0 0"/>
-  </joint>
-  <xacro:agribot_tpl_upper_hitch_prism_joint_core name="back_tpl_upper_hitch_prism_joint_core_link" />
-  <!-- end back TPL -->
+  <xacro:property name="sel_tpl" value="back"/>
+  <xacro:include filename="$(find agribot_description)/urdf/basic_links/tpl/tpl_assembled.xacro"/>
  <gazebo>
     <plugin name="agribot_controller" filename="libgazebo_ros_agribot.so">

File: urdf/basic_links/tpl/tpl_assembled.xacro (robot description, xacro)
@@ -8,3 +8,153 @@
   <xacro:include filename="$(find agribot_description)/urdf/basic_links/tpl/tpl_upper_hitch_prism_base.xacro"/>
   <xacro:include filename="$(find agribot_description)/urdf/basic_links/tpl/tpl_upper_hitch_prism_core.xacro"/>
+  <!-- Back TPL -->
+  <xacro:if value="${sel_tpl == 'back'}">
+    <joint name="back_tpl_base_joint" type="fixed">
+      <parent link="back_cart_link"/>
+      <child link="back_tpl_base_link"/>
+      <origin xyz="${-(cart_lenght+tpl_base_len)/2} 0.0 ${(cart_height-tpl_base_hei)/2}" rpy="0 0 0"/>
+      <axis xyz="0 0 1"/>
+    </joint>
+    <xacro:agribot_tpl_base name="back_tpl_base_link" />
+    <joint name="back_tpl_lower_hitches_revolute_joint" type="revolute">
+      <parent link="back_tpl_base_link"/>
+      <child link="back_tpl_cylinder_link"/>
+      <origin xyz="${-(tpl_base_len)/2} 0.0 0.0" rpy="${M_PI/2} ${-M_PI/5} 0"/>
+      <limit lower="${-90*M_PI/180}" upper="${15*M_PI/180}"  effort="1000.0" velocity="1000.0"/>
+      <axis xyz="0 0 1"/>
+    </joint>
+    <xacro:agribot_tpl_cylinder name="back_tpl_cylinder_link" />
+    <joint name="back_tpl_revolute_hitch_base_left_joint" type="fixed">
+      <parent link="back_tpl_cylinder_link"/>
+      <child link="back_tpl_revolute_hitch_base_left_link"/>
+      <origin xyz="${-(tpl_rev_hit_base_len-tpl_cyl_radius)/2} 0.0 ${-(tpl_cyl_width)/2}" rpy="0 0 0"/>
+      <axis xyz="0 0 1"/>
+    </joint>
+    <xacro:agribot_tpl_revolute_hitch_base name="back_tpl_revolute_hitch_base_left_link" />
+    <joint name="back_tpl_revolute_hitch_effector_left_joint" type="fixed">
+      <parent link="back_tpl_revolute_hitch_base_left_link"/>
+      <child link="back_tpl_revolute_hitch_effector_left_link"/>
+      <origin xyz="${-0.4*(tpl_rev_hit_base_len+tpl_rev_hit_effector_len)} 0.1 ${-0.22*tpl_rev_hit_effector_len}" rpy="0 ${-M_PI/6} ${-M_PI/6}"/>
+      <axis xyz="0 0 1"/>
+    </joint>
+    <xacro:agribot_tpl_revolute_hitch_effector name="back_tpl_revolute_hitch_effector_left_link" />
+    <joint name="back_tpl_revolute_hitch_right_joint" type="fixed">
+      <parent link="back_tpl_cylinder_link"/>
+      <child link="back_tpl_revolute_hitch_base_right_link"/>
+      <origin xyz="${-(tpl_rev_hit_base_len-tpl_cyl_radius)/2} 0.0 ${(tpl_cyl_width)/2}" rpy="0 0 0"/>
+      <axis xyz="0 0 1"/>
+    </joint>
+    <xacro:agribot_tpl_revolute_hitch_base name="back_tpl_revolute_hitch_base_right_link" />
+    <joint name="back_tpl_revolute_hitch_effector_right_joint" type="fixed">
+      <parent link="back_tpl_revolute_hitch_base_right_link"/>
+      <child link="back_tpl_revolute_hitch_effector_right_link"/>
+      <origin xyz="${-0.4*(tpl_rev_hit_base_len+tpl_rev_hit_effector_len)} 0.1 ${0.22*tpl_rev_hit_effector_len}" rpy="0 ${M_PI/6} ${-M_PI/6}"/>
+      <axis xyz="0 0 1"/>
+    </joint>
+    <xacro:agribot_tpl_revolute_hitch_effector name="back_tpl_revolute_hitch_effector_right_link" />
+    <joint name="back_tpl_upper_hich_base_joint" type="fixed">
+      <parent link="back_tpl_base_link"/>
+      <child link="back_tpl_up_hit_base_link"/>
+      <origin xyz="${-0.82*tpl_base_len} 0.0 ${0.8*(tpl_upper_hit_base_len)/2}" rpy="0 ${M_PI/3.15} 0"/>
+      <axis xyz="0 0 1"/>
+    </joint>
+    <xacro:agribot_tpl_upper_hitch_base name="back_tpl_up_hit_base_link" />
+    <joint name="back_tpl_upper_hitch_revolute_joint" type="revolute">
+      <parent link="back_tpl_up_hit_base_link"/>
+      <child link="back_tpl_upper_hitch_cylinder_link"/>
+      <origin xyz="${-tpl_upper_hit_base_len/2} 0.0 0.0" rpy="${M_PI/2} ${-M_PI/18} 0"/>
+      <limit lower="${-10*M_PI/180}" upper="${80*M_PI/180}"  effort="1000.0" velocity="1000.0"/>
+      <axis xyz="0 0 1"/>
+    </joint>
+    <xacro:agribot_tpl_upper_hitch_cylinder name="back_tpl_upper_hitch_cylinder_link" />
+    <joint name="back_tpl_upper_hitch_prism_joint_base_joint" type="fixed">
+      <parent link="back_tpl_upper_hitch_cylinder_link"/>
+      <child link="back_tpl_upper_hitch_prism_joint_base_link"/>
+      <origin xyz="${-(tpl_upper_hitch_prism_base_len)/2} 0.0 0.0" rpy="0 0 0"/>
+      <axis xyz="0 0 1"/>
+    </joint>
+    <xacro:agribot_tpl_upper_hitch_prism_joint_base name="back_tpl_upper_hitch_prism_joint_base_link" />
+    <joint name="back_tpl_upper_hitch_prismatic_joint" type="prismatic">
+      <parent link="back_tpl_upper_hitch_prism_joint_base_link"/>
+      <child link="back_tpl_upper_hitch_prism_joint_core_link"/>
+      <limit effort="1000.0" lower="${-tpl_upper_hitch_prism_core_len+0.05}" upper="0.0" velocity="0.5"/>
+      <origin rpy="0 0 0" xyz="-0.05 0 0"/>
+    </joint>
+    <xacro:agribot_tpl_upper_hitch_prism_joint_core name="back_tpl_upper_hitch_prism_joint_core_link" />
+  </xacro:if>
+  <!-- Front TPL -->
+  <xacro:if value="${sel_tpl == 'front'}">
+    <joint name="front_tpl_joint" type="fixed">
+      <parent link="front_cart_link"/>
+      <child link="front_tpl_base_link"/>
+      <origin xyz="${(cart_lenght+tpl_base_len)/2} 0.0 ${(cart_height-tpl_base_hei)/2}" rpy="0 0 0"/>
+      <axis xyz="0 0 1"/>
+    </joint>
+    <xacro:agribot_tpl_base name="front_tpl_base_link" />
+    <joint name="front_tpl_lower_hitches_revolute_joint" type="revolute">
+      <parent link="front_tpl_base_link"/>
+      <child link="front_tpl_cylinder_link"/>
+      <origin xyz="${(tpl_base_len)/2} 0.0 0.0" rpy="${-M_PI/2} ${M_PI/5} 0"/>
+      <limit lower="${-90*M_PI/180}" upper="${15*M_PI/180}"  effort="1000.0" velocity="1000.0"/>
+      <axis xyz="0 0 1"/>
+    </joint>
+    <xacro:agribot_tpl_cylinder name="front_tpl_cylinder_link" />
+    <joint name="front_tpl_revolute_hitch_base_left_joint" type="fixed">
+      <parent link="front_tpl_cylinder_link"/>
+      <child link="front_tpl_revolute_hitch_base_right_link"/>
+      <origin xyz="${(tpl_rev_hit_base_len-tpl_cyl_radius)/2} 0.0 ${-(tpl_cyl_width)/2}" rpy="0 0 0"/>
+      <axis xyz="0 0 1"/>
+    </joint>
+    <xacro:agribot_tpl_revolute_hitch_base name="front_tpl_revolute_hitch_base_right_link" />
+    <joint name="front_tpl_revolute_hitch_effector_right_joint" type="fixed">
+      <parent link="front_tpl_revolute_hitch_base_right_link"/>
+      <child link="front_tpl_revolute_hitch_effector_right_link"/>
+      <origin xyz="${0.4*(tpl_rev_hit_base_len+tpl_rev_hit_effector_len)} ${-0.22*tpl_rev_hit_effector_len} -0.1 " rpy="0 ${M_PI/6} ${-M_PI/6}"/>
+      <axis xyz="0 0 1"/>
+    </joint>
+    <xacro:agribot_tpl_revolute_hitch_effector name="front_tpl_revolute_hitch_effector_right_link" />
+    <joint name="front_tpl_revolute_hitch_left_joint" type="fixed">
+      <parent link="front_tpl_cylinder_link"/>
+      <child link="front_tpl_revolute_hitch_base_left_link"/>
+      <origin xyz="${(tpl_rev_hit_base_len-tpl_cyl_radius)/2} 0.0 ${(tpl_cyl_width)/2}" rpy="0 0 0"/>
+      <axis xyz="0 0 1"/>
+    </joint>
+    <xacro:agribot_tpl_revolute_hitch_base name="front_tpl_revolute_hitch_base_left_link" />
+    <joint name="front_tpl_revolute_hitch_effector_left_joint" type="fixed">
+      <parent link="front_tpl_revolute_hitch_base_left_link"/>
+      <child link="front_tpl_revolute_hitch_effector_left_link"/>
+      <origin xyz="${0.4*(tpl_rev_hit_base_len+tpl_rev_hit_effector_len)} ${-0.22*tpl_rev_hit_effector_len} 0.1" rpy="0 ${-M_PI/6} ${-M_PI/6}"/>
+      <axis xyz="0 0 1"/>
+    </joint>
+    <xacro:agribot_tpl_revolute_hitch_effector name="front_tpl_revolute_hitch_effector_left_link" />
+    <joint name="front_tpl_upper_hich_base_joint" type="fixed">
+      <parent link="front_tpl_base_link"/>
+      <child link="front_tpl_up_hit_base_link"/>
+      <origin xyz="${0.82*tpl_base_len} 0.0 ${0.8*(tpl_upper_hit_base_len)/2}" rpy="0 ${-M_PI/3.15} 0"/>
+      <axis xyz="0 0 1"/>
+    </joint>
+    <xacro:agribot_tpl_upper_hitch_base name="front_tpl_up_hit_base_link" />
+    <joint name="front_tpl_upper_hitch_revolute_joint" type="revolute">
+      <parent link="front_tpl_up_hit_base_link"/>
+      <child link="front_tpl_upper_hitch_cylinder_link"/>
+      <origin xyz="${tpl_upper_hit_base_len/2} 0.0 0.0" rpy="${-M_PI/2} ${M_PI/18+M_PI} 0"/>
+      <limit lower="${-10*M_PI/180}" upper="${80*M_PI/180}"  effort="1000.0" velocity="1000.0"/>
+      <axis xyz="0 0 1"/>
+    </joint>
+    <xacro:agribot_tpl_upper_hitch_cylinder name="front_tpl_upper_hitch_cylinder_link" />
+    <joint name="front_tpl_upper_hitch_prism_joint_base_joint" type="fixed">
+      <parent link="front_tpl_upper_hitch_cylinder_link"/>
+      <child link="front_tpl_upper_hitch_prism_joint_base_link"/>
+      <origin xyz="${-(tpl_upper_hitch_prism_base_len)/2} 0.0 0.0" rpy="0 0 0"/>
+      <axis xyz="0 0 1"/>
+    </joint>
+    <xacro:agribot_tpl_upper_hitch_prism_joint_base name="front_tpl_upper_hitch_prism_joint_base_link" />
+    <joint name="front_tpl_upper_hitch_prismatic_joint" type="prismatic">
+      <parent link="front_tpl_upper_hitch_prism_joint_base_link"/>
+      <child link="front_tpl_upper_hitch_prism_joint_core_link"/>
+      <limit effort="1000.0" lower="${-tpl_upper_hitch_prism_core_len+0.05}" upper="0.0" velocity="0.5"/>
+      <origin rpy="0 0 0" xyz="-0.05 0 0"/>
+    </joint>
+    <xacro:agribot_tpl_upper_hitch_prism_joint_core name="front_tpl_upper_hitch_prism_joint_core_link" />
+  </xacro:if>
 </robot>

Commit message: Make TPL urdf as macro

File: urdf/agribot.urdf.xacro (robot description, xacro)
@@ -8,4 +8,5 @@
   <xacro:include filename="$(find agribot_description)/urdf/basic_links/chassis.xacro"/>
   <xacro:include filename="$(find agribot_description)/urdf/basic_links/cart.xacro"/>
+  <xacro:include filename="$(find agribot_description)/urdf/basic_links/tpl.xacro"/>
   <xacro:arg name="perception_sensors" default="false" />
   <xacro:arg name="perception_plugins" default="true" />
@@ -47,6 +48,11 @@
   </joint>
   <xacro:agribot_cart name="back_cart_link" />
-  <xacro:property name="sel_tpl" value="front"/>
-  <xacro:include filename="$(find agribot_description)/urdf/basic_links/tpl/tpl_assembled.xacro"/>
+  <joint name="front_tpl_joint" type="fixed">
+    <parent link="front_cart_link"/>
+    <child link="front_tpl_base_link"/>
+    <origin xyz="${(cart_lenght+tpl_base_len)/2} 0.0 ${(cart_height-tpl_base_hei)/2}" rpy="0 ${-M_PI/36} 0"/>
+    <axis xyz="0 0 1"/>
+  </joint>
+  <xacro:agribot_tpl name="front_tpl" />
   <joint name="back_left_wheel_joint" type="continuous">
     <parent link="back_cart_link"/>
@@ -63,6 +69,11 @@
   </joint>
   <xacro:agribot_wheel name="back_right_wheel_link" />
-  <xacro:property name="sel_tpl" value="back"/>
-  <xacro:include filename="$(find agribot_description)/urdf/basic_links/tpl/tpl_assembled.xacro"/>
+  <joint name="back_tpl_base_joint" type="fixed">
+    <parent link="back_cart_link"/>
+    <child link="back_tpl_base_link"/>
+    <origin xyz="${-(cart_lenght+tpl_base_len)/2} 0.0 ${(cart_height-tpl_base_hei)/2}" rpy="0 ${M_PI/36} 0"/>
+    <axis xyz="0 0 1"/>
+  </joint>
+  <xacro:agribot_tpl name="back_tpl" />
  <gazebo>
     <plugin name="agribot_controller" filename="libgazebo_ros_agribot.so">

Commit message: Load simulation config yaml

File: urdf/agribot.urdf.xacro (robot description, xacro)
@@ -9,4 +9,6 @@
   <xacro:include filename="$(find agribot_description)/urdf/basic_links/cart.xacro"/>
   <xacro:include filename="$(find agribot_description)/urdf/basic_links/tpl.xacro"/>
+  <xacro:property name="yaml_file" value="$(find agribot_common)/config/agribot_simulation_config.yaml" />
+  <xacro:property name="props_simulation" value="${load_yaml(yaml_file)}"/>
   <xacro:arg name="perception_sensors" default="false" />
   <xacro:arg name="perception_plugins" default="true" />

File: urdf/basic_sensors.xacro (robot description, xacro)
@@ -5,9 +5,8 @@
     <xacro:include filename="$(find agribot_description)/urdf/basic_sensors/magnetometer/magnetometer.xacro"/>
     <xacro:macro name="basic_sensors">
-        <!-- Moderna vineyard coordinates -->
-        <xacro:property name="reference_latitude"   value="51.26662409135839"/>
-        <xacro:property name="reference_longitude"  value="17.20327894189977"/>
-        <xacro:property name="reference_heading"    value="158.5507847682035"/>
-        <xacro:property name="reference_altitude"   value="193.7327916698572"/>
+        <xacro:property name="reference_latitude"   value="${props_simulation['simulation_latitude']}"/>
+        <xacro:property name="reference_longitude"  value="${props_simulation['simulation_longitude']}"/>
+        <xacro:property name="reference_heading"    value="${props_simulation['simulation_heading']}"/>
+        <xacro:property name="reference_altitude"   value="${props_simulation['simulation_altitude']}"/>
         <xacro:imu_sensor>
             <origin xyz="0 0 0" rpy="0 0 0" />

Commit message: Change file location

File: urdf/agribot.urdf.xacro (robot description, xacro)
@@ -9,5 +9,5 @@
   <xacro:include filename="$(find agribot_description)/urdf/basic_links/cart.xacro"/>
   <xacro:include filename="$(find agribot_description)/urdf/basic_links/tpl.xacro"/>
-  <xacro:property name="yaml_file" value="$(find agribot_common)/config/agribot_simulation_config.yaml" />
+  <xacro:property name="yaml_file" value="$(find agribot_common)/config/simulation/config.yaml" />
   <xacro:property name="props_simulation" value="${load_yaml(yaml_file)}"/>
   <xacro:arg name="perception_sensors" default="false" />
