Commit message: Move more to params

File: urdf/agribot.urdf.xacro (robot description, xacro)
@@ -9,8 +9,4 @@
   <xacro:include filename="$(find agribot_description)/urdf/basic_links/cart.xacro"/>
   <xacro:include filename="$(find agribot_description)/urdf/basic_links/tpl.xacro"/>
-  <xacro:property name="yaml_file" value="$(find agribot_common)/config/simulation/config.yaml" />
-  <xacro:property name="props_simulation" value="${load_yaml(yaml_file)}"/>
-  <xacro:arg name="perception_sensors" default="false" />
-  <xacro:arg name="perception_plugins" default="true" />
   <link name="base_footprint"/>
   <joint name="chassis_joint" type="fixed">
@@ -100,7 +96,7 @@
   <xacro:tools_sensors/>
   <!-- Load perception sensors -->
-  <xacro:if value="$(arg perception_sensors)">
+  <xacro:if value="${param_simulation['perception_sensors']}">
     <xacro:perception_sensors>
-      <xacro:property name="perception_plugins_arg" value="$(arg perception_plugins)"/>
+      <xacro:property name="perception_plugins_arg" value="${param_simulation['perception_plugins']}"/>
     </xacro:perception_sensors>
   </xacro:if>

File: urdf/basic_links/chassis.xacro (robot description, xacro)
@@ -1,7 +1,7 @@
 <robot name="chassis" xmlns:xacro="http://ros.org/wiki/xacro">
-    <xacro:property name="chassis_length" value="2.42" />
-    <xacro:property name="chassis_width" value="1.05" />
-    <xacro:property name="chassis_height" value="1.65" />
-    <xacro:property name="chassis_mass" value="2000" />
+    <xacro:property name="chassis_length" value="${param_dimension['chassis_length']}" />
+    <xacro:property name="chassis_width" value="${param_dimension['chassis_width']}" />
+    <xacro:property name="chassis_height" value="${param_dimension['chassis_height']}" />
+    <xacro:property name="chassis_mass" value="${param_dimension['chassis_mass']}" />
     <xacro:macro name="agribot_chassis" params="name">
         <link name="${name}">

File: urdf/basic_links/wheel.xacro (robot description, xacro)
@@ -1,6 +1,6 @@
 <robot name="wheel" xmlns:xacro="http://ros.org/wiki/xacro">
-    <xacro:property name="wheel_width" value="0.025" />
-    <xacro:property name="wheel_radius" value="0.16" />
-    <xacro:property name="wheel_mass" value="50" />
+    <xacro:property name="wheel_width" value="${param_dimension['wheel_width']}" />
+    <xacro:property name="wheel_radius" value="${param_dimension['wheel_radius']}" />
+    <xacro:property name="wheel_mass" value="${param_dimension['wheel_mass']}" />
     <xacro:macro name="agribot_wheel" params="name">
         <link name="${name}">

File: urdf/basic_sensors.xacro (robot description, xacro)
@@ -5,8 +5,8 @@
     <xacro:include filename="$(find agribot_description)/urdf/basic_sensors/magnetometer/magnetometer.xacro"/>
     <xacro:macro name="basic_sensors">
-        <xacro:property name="reference_latitude"   value="${props_simulation['simulation_latitude']}"/>
-        <xacro:property name="reference_longitude"  value="${props_simulation['simulation_longitude']}"/>
-        <xacro:property name="reference_heading"    value="${props_simulation['simulation_heading']}"/>
-        <xacro:property name="reference_altitude"   value="${props_simulation['simulation_altitude']}"/>
+        <xacro:property name="reference_latitude"   value="${param_simulation['simulation_latitude']}"/>
+        <xacro:property name="reference_longitude"  value="${param_simulation['simulation_longitude']}"/>
+        <xacro:property name="reference_heading"    value="${param_simulation['simulation_heading']}"/>
+        <xacro:property name="reference_altitude"   value="${param_simulation['simulation_altitude']}"/>
         <xacro:imu_sensor>
             <origin xyz="0 0 0" rpy="0 0 0" />

File: urdf/common_properties.xacro (robot description, xacro)
@@ -1,4 +1,8 @@
 <?xml version="1.0" ?>
 <robot name="xacro_properties" xmlns:xacro="http://ros.org/wiki/xacro">
+  <xacro:property name="simulation_yaml_file" value="$(find agribot_common)/config/simulation/config.yaml" />
+  <xacro:property name="param_simulation" value="${load_yaml(simulation_yaml_file)}"/>
+  <xacro:property name="description_dimensions_file" value="$(find agribot_common)/config/description/dimensions.yaml" />
+  <xacro:property name="param_dimension" value="${load_yaml(description_dimensions_file)}"/>
   <xacro:property name="M_PI" value="3.1415926535897931" />
   <!-- Init colour -->

Commit message: Add robot_length instead of chassis_length

File: urdf/agribot.urdf.xacro (robot description, xacro)
@@ -78,5 +78,5 @@
       <wheelSeparation> ${chassis_width+wheel_width} </wheelSeparation>
       <wheelRadius> ${wheel_radius} </wheelRadius>
-      <chasisLength>${chassis_length-2*wheel_radius}</chasisLength>
+      <chasisLength>${param_dimension['robot_length']}</chasisLength>
       <broadcastTF>false</broadcastTF> <!-- set this paremeter to false when localization is used-->
       <odometryTopic>/agribot/odometry</odometryTopic>

File: urdf/basic_links/chassis.xacro (robot description, xacro)
@@ -1,4 +1,4 @@
 <robot name="chassis" xmlns:xacro="http://ros.org/wiki/xacro">
-    <xacro:property name="chassis_length" value="${param_dimension['chassis_length']}" />
+    <xacro:property name="chassis_length" value="${param_dimension['robot_length']+2*param_dimension['wheel_radius']}" />
     <xacro:property name="chassis_width" value="${param_dimension['chassis_width']}" />
     <xacro:property name="chassis_height" value="${param_dimension['chassis_height']}" />

Commit message: Move config to seperate repo

File: urdf/agribot.urdf.xacro (robot description, xacro)
@@ -9,4 +9,10 @@
   <xacro:include filename="$(find agribot_description)/urdf/basic_links/cart.xacro"/>
   <xacro:include filename="$(find agribot_description)/urdf/basic_links/tpl.xacro"/>
+  <xacro:arg name="perception_sensors" default="false" />
+  <xacro:arg name="perception_plugins" default="false" />
+  <xacro:arg name="simulation_latitude" default="51.26662409135839" />
+  <xacro:arg name="simulation_longitude" default="17.20327894189977" />
+  <xacro:arg name="simulation_heading" default="158.5507847682035" />
+  <xacro:arg name="simulation_altitude" default="193.7327916698572" />
   <link name="base_footprint"/>
   <joint name="chassis_joint" type="fixed">
@@ -96,7 +102,7 @@
   <xacro:tools_sensors/>
   <!-- Load perception sensors -->
-  <xacro:if value="${param_simulation['perception_sensors']}">
+  <xacro:if value="$(arg perception_sensors)">
     <xacro:perception_sensors>
-      <xacro:property name="perception_plugins_arg" value="${param_simulation['perception_plugins']}"/>
+      <xacro:property name="perception_plugins_arg" value="$(arg perception_plugins)"/>
     </xacro:perception_sensors>
   </xacro:if>

File: urdf/basic_sensors.xacro (robot description, xacro)
@@ -5,8 +5,8 @@
     <xacro:include filename="$(find agribot_description)/urdf/basic_sensors/magnetometer/magnetometer.xacro"/>
     <xacro:macro name="basic_sensors">
-        <xacro:property name="reference_latitude"   value="${param_simulation['simulation_latitude']}"/>
-        <xacro:property name="reference_longitude"  value="${param_simulation['simulation_longitude']}"/>
-        <xacro:property name="reference_heading"    value="${param_simulation['simulation_heading']}"/>
-        <xacro:property name="reference_altitude"   value="${param_simulation['simulation_altitude']}"/>
+        <xacro:property name="reference_latitude"   value="$(arg simulation_latitude)"/>
+        <xacro:property name="reference_longitude"  value="$(arg simulation_longitude)"/>
+        <xacro:property name="reference_heading"    value="$(arg simulation_heading)"/>
+        <xacro:property name="reference_altitude"   value="$(arg simulation_altitude)"/>
         <xacro:imu_sensor>
             <origin xyz="0 0 0" rpy="0 0 0" />

File: urdf/common_properties.xacro (robot description, xacro)
@@ -1,7 +1,7 @@
 <?xml version="1.0" ?>
 <robot name="xacro_properties" xmlns:xacro="http://ros.org/wiki/xacro">
-  <xacro:property name="simulation_yaml_file" value="$(find agribot_common)/config/simulation/config.yaml" />
+  <xacro:property name="simulation_yaml_file" value="$(env AGRIBOT_HOME)/agribot/configs/simulation/config.yaml" />
   <xacro:property name="param_simulation" value="${load_yaml(simulation_yaml_file)}"/>
-  <xacro:property name="description_dimensions_file" value="$(find agribot_common)/config/description/dimensions.yaml" />
+  <xacro:property name="description_dimensions_file" value="$(env AGRIBOT_HOME)/agribot/configs/base/description/dimensions.yaml" />
   <xacro:property name="param_dimension" value="${load_yaml(description_dimensions_file)}"/>
   <xacro:property name="M_PI" value="3.1415926535897931" />

Commit message: Adapt to new convention of dimensions config

File: urdf/agribot.urdf.xacro (robot description, xacro)
@@ -26,5 +26,5 @@
     <child link="front_cart_link"/>
     <limit lower="${-45*M_PI/180}" upper="${45*M_PI/180}" effort="1000.0" velocity="1000.0"/>
-    <origin xyz="${(chassis_length/2)-cart_lenght/2} 0.0 ${(chassis_height+cart_height)/(-2)}" rpy="0 0 0"/>
+    <origin xyz="${(chassis_length/2)-cart_length/2} 0.0 ${(chassis_height+cart_height)/(-2)}" rpy="0 0 0"/>
     <axis xyz="0 0 1"/>
   </joint>
@@ -48,5 +48,5 @@
     <child link="back_cart_link"/>
     <limit lower="${-45*M_PI/180}" upper="${45*M_PI/180}"  effort="1000.0" velocity="1000.0"/>
-    <origin xyz="${-(chassis_length/2)+cart_lenght/2} 0.0 ${(chassis_height+cart_height)/(-2)}" rpy="0 0 0"/>
+    <origin xyz="${-(chassis_length/2)+cart_length/2} 0.0 ${(chassis_height+cart_height)/(-2)}" rpy="0 0 0"/>
     <axis xyz="0 0 1"/>
   </joint>
@@ -55,5 +55,5 @@
     <parent link="front_cart_link"/>
     <child link="front_tpl_base_link"/>
-    <origin xyz="${(cart_lenght+tpl_base_len)/2} 0.0 ${(cart_height-tpl_base_hei)/2}" rpy="0 ${-M_PI/36} 0"/>
+    <origin xyz="${(cart_length+tpl_base_len)/2} 0.0 ${(cart_height-tpl_base_hei)/2}" rpy="0 ${-M_PI/36} 0"/>
     <axis xyz="0 0 1"/>
   </joint>
@@ -76,5 +76,5 @@
     <parent link="back_cart_link"/>
     <child link="back_tpl_base_link"/>
-    <origin xyz="${-(cart_lenght+tpl_base_len)/2} 0.0 ${(cart_height-tpl_base_hei)/2}" rpy="0 ${M_PI/36} 0"/>
+    <origin xyz="${-(cart_length+tpl_base_len)/2} 0.0 ${(cart_height-tpl_base_hei)/2}" rpy="0 ${M_PI/36} 0"/>
     <axis xyz="0 0 1"/>
   </joint>
@@ -84,5 +84,5 @@
       <wheelSeparation> ${chassis_width+wheel_width} </wheelSeparation>
       <wheelRadius> ${wheel_radius} </wheelRadius>
-      <chasisLength>${param_dimension['robot_length']}</chasisLength>
+      <chasisLength>${param_dimension['dimensions/robot_axis_to_axis_length']}</chasisLength>
       <broadcastTF>false</broadcastTF> <!-- set this paremeter to false when localization is used-->
       <odometryTopic>/agribot/odometry</odometryTopic>

File: urdf/basic_links/cart.xacro (robot description, xacro)
@@ -1,7 +1,7 @@
 <robot name="base" xmlns:xacro="http://ros.org/wiki/xacro">
-    <xacro:property name="cart_lenght" value="${param_dimension['wheel_radius']*2}" />
-    <xacro:property name="cart_width" value="${param_dimension['chassis_width']}" />
-    <xacro:property name="cart_height" value="${param_dimension['wheel_radius']*2}" />
-    <xacro:property name="cart_mass" value="500" />
+    <xacro:property name="cart_length" value="${param_dimension['dimensions/cart_length']}" />
+    <xacro:property name="cart_width" value="${param_dimension['dimensions/cart_width']}" />
+    <xacro:property name="cart_height" value="${param_dimension['dimensions/cart_height']}" />
+    <xacro:property name="cart_mass" value="${param_dimension['dimensions/cart_mass']}" />
     <xacro:macro name="agribot_cart" params="name">
         <link name="${name}">
@@ -29,5 +29,5 @@
             </xacro:if>
             <geometry>
-               <box size="${cart_lenght} ${cart_width} ${cart_height}" />
+               <box size="${cart_length} ${cart_width} ${cart_height}" />
             </geometry>
           </collision>
@@ -38,6 +38,6 @@
             <mass value="${cart_mass}"/>
             <inertia ixx="${cart_mass*(cart_height*cart_height+cart_width*cart_width)/12}" ixy="0.0" ixz="0.0"
-                     iyy="${cart_mass*(cart_lenght*cart_lenght+cart_height*cart_height)/12}" iyz="0.0"
-                     izz="${cart_mass*(cart_lenght*cart_lenght+cart_width*cart_width)/12}" />
+                     iyy="${cart_mass*(cart_length*cart_length+cart_height*cart_height)/12}" iyz="0.0"
+                     izz="${cart_mass*(cart_length*cart_length+cart_width*cart_width)/12}" />
           </inertial>
         </link>

File: urdf/basic_links/chassis.xacro (robot description, xacro)
@@ -1,11 +1,11 @@
 <robot name="chassis" xmlns:xacro="http://ros.org/wiki/xacro">
-    <xacro:property name="chassis_length" value="${param_dimension['robot_length']+2*param_dimension['wheel_radius']}" />
-    <xacro:property name="chassis_width" value="${param_dimension['chassis_width']}" />
-    <xacro:property name="chassis_height" value="${param_dimension['chassis_height']}" />
-    <xacro:property name="chassis_mass" value="${param_dimension['chassis_mass']}" />
+    <xacro:property name="chassis_length" value="${param_dimension['dimensions/chassis_length']}" />
+    <xacro:property name="chassis_width" value="${param_dimension['dimensions/chassis_width']}" />
+    <xacro:property name="chassis_height" value="${param_dimension['dimensions/chassis_height']}" />
+    <xacro:property name="chassis_mass" value="${param_dimension['dimensions/chassis_mass']}" />
     <xacro:macro name="agribot_chassis" params="name">
         <link name="${name}">
           <visual>
-            <origin xyz="0.0 0.0 0.1" rpy="0 0 1.57"/>
+            <origin xyz="0.0 0.0 0.1" rpy="0 0 ${M_PI/2}"/>
             <geometry>
               <mesh filename="package://agribot_description/meshes/agribot_chassis.stl" scale="0.01 0.01 0.01"/>

File: urdf/basic_links/wheel.xacro (robot description, xacro)
@@ -1,6 +1,6 @@
 <robot name="wheel" xmlns:xacro="http://ros.org/wiki/xacro">
-    <xacro:property name="wheel_width" value="${param_dimension['wheel_width']}" />
-    <xacro:property name="wheel_radius" value="${param_dimension['wheel_radius']}" />
-    <xacro:property name="wheel_mass" value="${param_dimension['wheel_mass']}" />
+    <xacro:property name="wheel_width" value="${param_dimension['dimensions/wheel_width']}" />
+    <xacro:property name="wheel_radius" value="${param_dimension['dimensions/wheel_radius']}" />
+    <xacro:property name="wheel_mass" value="${param_dimension['dimensions/wheel_mass']}" />
     <xacro:macro name="agribot_wheel" params="name">
         <link name="${name}">

Commit message: Fixed description for new controller

File: urdf/agribot.urdf.xacro (robot description, xacro)
@@ -97,4 +97,8 @@
     </plugin>
   </gazebo>
+  <gazebo>
+    <plugin name="gazebo_ros_control" filename="libgazebo_ros_control.so">
+    </plugin>
+  </gazebo>
   <!-- Load basic sensors -->
   <xacro:basic_sensors/>

File: urdf/basic_links/tpl.xacro (robot description, xacro)
@@ -14,12 +14,21 @@
       <child link="${name}_cylinder_link"/>
       <xacro:if value="${name == 'back_tpl'}">
-        <origin xyz="${-(tpl_base_len)/2} 0.0 0.0" rpy="${M_PI/2} ${-M_PI/5} 0"/>
+        <origin xyz="${-(tpl_base_len)/2} 0.0 0.0" rpy="${M_PI/2} ${-M_PI*1.75+M_PI} ${M_PI}"/>
       </xacro:if>
       <xacro:if value="${name == 'front_tpl'}">
-        <origin xyz="${(tpl_base_len)/2} 0.0 0.0" rpy="${-M_PI/2} ${M_PI/5} 0"/>
+        <origin xyz="${(tpl_base_len)/2} 0.0 0.0" rpy="${M_PI/2} ${-M_PI*1.75} 0"/>
       </xacro:if>
-      <limit lower="-0.03" upper="0.9"  effort="1000.0" velocity="1000.0"/>
+      <limit lower="-0.03" upper="0.9"  effort="1.0" velocity="0.5"/>
       <axis xyz="0 0 1"/>
     </joint>
+    <transmission name="${name}_lower_hitches_revolute_joint_transmission">
+      <type>transmission_interface/SimpleTransmission</type>
+      <joint name="${name}_lower_hitches_revolute_joint">
+        <hardwareInterface>hardware_interface/EffortJointInterface</hardwareInterface>
+      </joint>
+      <actuator name="${name}_lower_hitches_revolute_joint_motor">
+        <hardwareInterface>hardware_interface/EffortJointInterface</hardwareInterface>
+      </actuator>
+    </transmission>
     <xacro:agribot_tpl_cylinder name="${name}_cylinder_link" />
     <joint name="${name}_revolute_hitch_base_left_joint" type="fixed">
@@ -27,5 +36,5 @@
       <child link="${name}_revolute_hitch_base_right_link"/>
       <xacro:if value="${name == 'back_tpl'}">
-        <origin xyz="${-(tpl_rev_hit_base_len-tpl_cyl_radius)/2} 0.0 ${(tpl_cyl_width)/2}" rpy="0 0 0"/>
+        <origin xyz="${-(tpl_rev_hit_base_len-tpl_cyl_radius)/2} 0.0 ${(tpl_cyl_width)/2}" rpy="${M_PI} 0 0"/>
       </xacro:if>
       <xacro:if value="${name == 'front_tpl'}">
@@ -39,8 +48,8 @@
       <child link="${name}_revolute_hitch_effector_right_link"/>
       <xacro:if value="${name == 'back_tpl'}">
-        <origin xyz="${-0.43*(tpl_rev_hit_base_len+tpl_rev_hit_effector_len)} 0.12 ${0.28*tpl_rev_hit_effector_len}" rpy="0 ${M_PI/6} ${-M_PI/6}"/>
+        <origin xyz="${-0.43*(tpl_rev_hit_base_len+tpl_rev_hit_effector_len)} 0.12 ${-0.28*tpl_rev_hit_effector_len}" rpy="0 ${-M_PI/6} ${-M_PI/6}"/>
       </xacro:if>
       <xacro:if value="${name == 'front_tpl'}">
-        <origin xyz="${0.43*(tpl_rev_hit_base_len+tpl_rev_hit_effector_len)} ${-0.28*tpl_rev_hit_effector_len} -0.12 " rpy="0 ${M_PI/6} ${-M_PI/6}"/>
+        <origin xyz="${0.43*(tpl_rev_hit_base_len+tpl_rev_hit_effector_len)} ${0.28*tpl_rev_hit_effector_len} -0.12 " rpy="0 ${M_PI/6} ${M_PI/6}"/>
       </xacro:if>
       <axis xyz="0 0 1"/>
@@ -51,5 +60,5 @@
       <child link="${name}_revolute_hitch_base_left_link"/>
       <xacro:if value="${name == 'back_tpl'}">
-        <origin xyz="${-(tpl_rev_hit_base_len-tpl_cyl_radius)/2} 0.0 ${-(tpl_cyl_width)/2}" rpy="0 0 0"/>
+        <origin xyz="${-(tpl_rev_hit_base_len-tpl_cyl_radius)/2} 0.0 ${-(tpl_cyl_width)/2}" rpy="${M_PI} 0 0"/>
       </xacro:if>
       <xacro:if value="${name == 'front_tpl'}">
@@ -63,8 +72,8 @@
       <child link="${name}_revolute_hitch_effector_left_link"/>
       <xacro:if value="${name == 'back_tpl'}">
-        <origin xyz="${-0.43*(tpl_rev_hit_base_len+tpl_rev_hit_effector_len)} 0.12 ${-0.28*tpl_rev_hit_effector_len}" rpy="0 ${-M_PI/6} ${-M_PI/6}"/>
+        <origin xyz="${-0.43*(tpl_rev_hit_base_len+tpl_rev_hit_effector_len)} 0.12 ${0.28*tpl_rev_hit_effector_len}" rpy="0 ${M_PI/6} ${-M_PI/6}"/>
       </xacro:if>
       <xacro:if value="${name == 'front_tpl'}">
-        <origin xyz="${0.43*(tpl_rev_hit_base_len+tpl_rev_hit_effector_len)} ${-0.28*tpl_rev_hit_effector_len} 0.12" rpy="0 ${-M_PI/6} ${-M_PI/6}"/>
+        <origin xyz="${0.43*(tpl_rev_hit_base_len+tpl_rev_hit_effector_len)} ${0.28*tpl_rev_hit_effector_len} 0.12" rpy="0 ${-M_PI/6} ${M_PI/6}"/>
       </xacro:if>
       <axis xyz="0 0 1"/>
@@ -92,5 +101,5 @@
         <origin xyz="${tpl_upper_hit_base_len/2} 0.0 0.0" rpy="${-M_PI/2} ${M_PI/18+M_PI} 0"/>
       </xacro:if>
-      <limit lower="${-10*M_PI/180}" upper="${80*M_PI/180}"  effort="1000.0" velocity="1000.0"/>
+      <limit lower="${-10*M_PI/180}" upper="${80*M_PI/180}"  effort="1.0" velocity="0.5"/>
       <axis xyz="0 0 1"/>
     </joint>
@@ -106,7 +115,16 @@
       <parent link="${name}_upper_hitch_prism_joint_base_link"/>
       <child link="${name}_upper_hitch_prism_joint_core_link"/>
-      <limit effort="1000.0" lower="0.0" upper="0.25" velocity="0.5"/>
-      <origin rpy="0 0 0" xyz="-0.05 0 0"/>
+      <limit effort="1.0" lower="0.0" upper="0.25" velocity="0.5"/>
+      <origin rpy="0 0 ${M_PI}" xyz="-0.05 0 0"/>
     </joint>
+    <transmission name="${name}_upper_hitch_prismatic_joint_transmission">
+      <type>transmission_interface/SimpleTransmission</type>
+      <joint name="${name}_upper_hitch_prismatic_joint">
+        <hardwareInterface>hardware_interface/EffortJointInterface</hardwareInterface>
+      </joint>
+      <actuator name="${name}_upper_hitch_prismatic_joint_motor">
+        <hardwareInterface>hardware_interface/EffortJointInterface</hardwareInterface>
+      </actuator>
+    </transmission>
     <xacro:agribot_tpl_upper_hitch_prism_joint_core name="${name}_upper_hitch_prism_joint_core_link" />  </xacro:macro>
 </robot>

File: urdf/basic_links/tpl/tpl_cyl.xacro (robot description, xacro)
@@ -7,13 +7,13 @@
       <visual>
         <xacro:if value="${name == 'back_tpl_cylinder_link'}">
-          <origin xyz="1.84 -0.68 -0.1" rpy="${M_PI/10} ${M_PI/2} 0"/>
+          <origin xyz="0 0 0" rpy="${M_PI/2} 0 ${M_PI/10}"/>
           <material name="white"/>
         </xacro:if>
         <xacro:if value="${name == 'front_tpl_cylinder_link'}">
-          <origin xyz="-1.84 0.68 -0.1" rpy="${-M_PI+M_PI/10} ${M_PI/2} 0"/>
+          <origin xyz="0 0 0" rpy="${-M_PI/2} ${M_PI} ${M_PI/10}"/>
           <material name="green"/>
         </xacro:if>
         <geometry>
-          <mesh filename="package://agribot_description/meshes/lower_hitches.stl" scale="0.00105 0.00105 0.00105"/>
+          <mesh filename="package://agribot_description/meshes/lower_hitches.stl" scale="0.525 0.525 0.525"/>
         </geometry>
       </visual>

Commit message: Remove perception_sensors from URDF. Perception tf is always broadcasted

File: urdf/agribot.urdf.xacro (robot description, xacro)
@@ -106,8 +106,6 @@
   <xacro:tools_sensors/>
   <!-- Load perception sensors -->
-  <xacro:if value="$(arg perception_sensors)">
-    <xacro:perception_sensors>
-      <xacro:property name="perception_plugins_arg" value="$(arg perception_plugins)"/>
-    </xacro:perception_sensors>
-  </xacro:if>
+  <xacro:perception_sensors>
+    <xacro:property name="perception_plugins_arg" value="$(arg perception_plugins)"/>
+  </xacro:perception_sensors>
 </robot>
