Commit message: Reorganize perception sensors macros

File: urdf/agribot.urdf.xacro (robot description, xacro)
@@ -107,5 +107,5 @@
   <!-- Load perception sensors -->
   <xacro:perception_sensors>
-    <xacro:property name="perception_plugins_arg" value="$(arg perception_plugins)"/>
+    <xacro:property name="perception_plugins" value="$(arg perception_plugins)"/>
   </xacro:perception_sensors>
 </robot>

File: urdf/perception_sensors.xacro (robot description, xacro)
@@ -1,24 +1,16 @@
 <robot name="perception_sensors" xmlns:xacro="http://ros.org/wiki/xacro">
-  <xacro:include filename="$(find agribot_description)/urdf/perception_sensors/lidar/livox_horizon.xacro"/>
-  <xacro:include filename="$(find agribot_description)/urdf/perception_sensors/camera/zed2.xacro"/>
-  <xacro:macro  name="perception_sensors"
-              params="perception_plugins_arg:=^
+  <xacro:include filename="$(find agribot_description)/urdf/perception_sensors/perception_suites/livox_zed2_set.xacro" />
+  <xacro:macro name="perception_sensors" params="perception_plugins:=^
                      ">
     <!-- Lidars -->
-    <xacro:livox_horizon>
-      <origin xyz="2.25 0 1.24" rpy="0 ${18.0*M_PI/180.0} 0" />
-      <xacro:property name="parent"               value="base_footprint"/>
-      <xacro:property name="topic"                value="/agribot/obstacle_detection/front/3d/lidar/point_cloud"/>
-      <xacro:property name="name"                 value="front_lidar"/>
-      <xacro:property name="hz"                   value="1.0"/>
-      <xacro:property name="visualize"            value="false"/>
-      <xacro:property name="perception_plugins"   value="${perception_plugins_arg}"/>
-    </xacro:livox_horizon>
-    <!-- ZED2 camera -->
-    <xacro:zed2>
-      <origin xyz="2.25 0 1.24" rpy="0 ${18.0*M_PI/180.0} 0" />
-      <xacro:property name="parent"               value="base_footprint"/>
-      <xacro:property name="camera_name"          value="zed2"/>
-    </xacro:zed2>
+    <xacro:livox_zed2_set>
+      <origin xyz="2.25 0 1.24" rpy="0 ${25.0*M_PI/180.0} 0" />
+      <xacro:property name="parent" value="base_footprint" />
+      <xacro:property name="suite_name" value="front_livox_zed2_set" />
+      <xacro:property name="livox_name" value="front_lidar" />
+      <xacro:property name="livox_topic" value="/agribot/obstacle_detection/front/3d/lidar/point_cloud" />
+      <xacro:property name="livox_hz" value="1.0" />
+      <xacro:property name="livox_visualize" value="false" />
+    </xacro:livox_zed2_set>
   </xacro:macro>
 </robot>

File: urdf/perception_sensors/camera/zed2.xacro (robot description, xacro)
@@ -1,78 +1,77 @@
 <robot name="zed2" xmlns:xacro="http://ros.org/wiki/xacro">
   <material name="zed2_mat">
-    <color rgba="0.25 0.25 0.25 0.99"/>
+    <color rgba="0.25 0.25 0.25 0.99" />
   </material>
-  <xacro:macro name="zed2"
-               params="*origin
+  <xacro:macro name="zed2" params="*origin
                        parent:=^
                        camera_name:=^
                       ">
     <!-- Properties -->
-    <xacro:property name="M_PI"     value="3.1415926535897931" />
+    <xacro:property name="M_PI" value="3.1415926535897931" />
     <xacro:property name="baseline" value="0.12" />
     <!-- Camera Center -->
     <joint name="${camera_name}_camera_center_joint" type="fixed">
-        <parent link="${parent}"/>
-        <child link="${camera_name}_camera_center"/>
-        <xacro:insert_block name="origin" />
+      <parent link="${parent}" />
+      <child link="${camera_name}_camera_center" />
+      <xacro:insert_block name="origin" />
     </joint>
     <link name="${camera_name}_camera_center">
-        <visual>
-            <origin xyz="0 0 0" rpy="0 0 0"/>
-            <geometry>
-                <mesh filename="package://agribot_description/meshes/zed2.stl" />
-            </geometry>
-            <material name="zed2_mat" />
-        </visual>
+      <visual>
+        <origin xyz="0 0 0" rpy="0 0 0" />
+        <geometry>
+          <mesh filename="package://agribot_description/meshes/zed2.stl" />
+        </geometry>
+        <material name="zed2_mat" />
+      </visual>
     </link>
     <!-- Left Camera -->
     <joint name="${camera_name}_left_camera_joint" type="fixed">
-        <parent link="${camera_name}_camera_center"/>
-        <child link="${camera_name}_left_camera_frame"/>
-        <origin xyz="0 ${baseline/2} 0" rpy="0 0 0" />
+      <parent link="${camera_name}_camera_center" />
+      <child link="${camera_name}_left_camera_frame" />
+      <origin xyz="0 ${baseline/2} 0" rpy="0 0 0" />
     </joint>
     <link name="${camera_name}_left_camera_frame" />
     <joint name="${camera_name}_left_camera_optical_joint" type="fixed">
-        <origin xyz="0 0 0" rpy="-${M_PI/2} 0.0 -${M_PI/2}"/>
-        <parent link="${camera_name}_left_camera_frame"/>
-        <child link="${camera_name}_left_camera_optical_frame"/>
+      <origin xyz="0 0 0" rpy="-${M_PI/2} 0.0 -${M_PI/2}" />
+      <parent link="${camera_name}_left_camera_frame" />
+      <child link="${camera_name}_left_camera_optical_frame" />
     </joint>
-    <link name="${camera_name}_left_camera_optical_frame"/>
+    <link name="${camera_name}_left_camera_optical_frame" />
     <!-- Right Camera -->
     <joint name="${camera_name}_right_camera_joint" type="fixed">
-        <parent link="${camera_name}_camera_center"/>
-        <child link="${camera_name}_right_camera_frame"/>
-        <origin xyz="0 -${baseline/2} 0" rpy="0 0 0" />
+      <parent link="${camera_name}_camera_center" />
+      <child link="${camera_name}_right_camera_frame" />
+      <origin xyz="0 -${baseline/2} 0" rpy="0 0 0" />
     </joint>
     <link name="${camera_name}_right_camera_frame" />
     <joint name="${camera_name}_right_camera_optical_joint" type="fixed">
-        <origin xyz="0 0 0" rpy="-${M_PI/2} 0.0 -${M_PI/2}"/>
-        <parent link="${camera_name}_right_camera_frame"/>
-        <child link="${camera_name}_right_camera_optical_frame"/>
+      <origin xyz="0 0 0" rpy="-${M_PI/2} 0.0 -${M_PI/2}" />
+      <parent link="${camera_name}_right_camera_frame" />
+      <child link="${camera_name}_right_camera_optical_frame" />
     </joint>
-    <link name="${camera_name}_right_camera_optical_frame"/>
+    <link name="${camera_name}_right_camera_optical_frame" />
     <!-- ZED2 Sensors -->
     <joint name="${camera_name}_mag_joint" type="fixed">
-        <parent link="${camera_name}_camera_center"/>
-        <child link="${camera_name}_mag_link"/>
-        <origin xyz="0 0 0" rpy="0 0 0" />
+      <parent link="${camera_name}_camera_center" />
+      <child link="${camera_name}_mag_link" />
+      <origin xyz="0 0 0" rpy="0 0 0" />
     </joint>
     <link name="${camera_name}_mag_link" />
     <joint name="${camera_name}_baro_joint" type="fixed">
-        <parent link="${camera_name}_camera_center"/>
-        <child link="${camera_name}_baro_link"/>
-        <origin xyz="0 0 0" rpy="0 0 0" />
+      <parent link="${camera_name}_camera_center" />
+      <child link="${camera_name}_baro_link" />
+      <origin xyz="0 0 0" rpy="0 0 0" />
     </joint>
     <link name="${camera_name}_baro_link" />
     <joint name="${camera_name}_temp_left_joint" type="fixed">
-        <parent link="${camera_name}_left_camera_frame"/>
-        <child link="${camera_name}_temp_left_link"/>
-        <origin xyz="0 0 0" rpy="0 0 0" />
+      <parent link="${camera_name}_left_camera_frame" />
+      <child link="${camera_name}_temp_left_link" />
+      <origin xyz="0 0 0" rpy="0 0 0" />
     </joint>
     <link name="${camera_name}_temp_left_link" />
     <joint name="${camera_name}_temp_right_joint" type="fixed">
-        <parent link="${camera_name}_right_camera_frame"/>
-        <child link="${camera_name}_temp_right_link"/>
-        <origin xyz="0 0 0" rpy="0 0 0" />
+      <parent link="${camera_name}_right_camera_frame" />
+      <child link="${camera_name}_temp_right_link" />
+      <origin xyz="0 0 0" rpy="0 0 0" />
     </joint>
     <link name="${camera_name}_temp_right_link" />

File: urdf/perception_sensors/lidar/livox_horizon.xacro (robot description, xacro)
@@ -1,7 +1,6 @@
 <robot name="livox_horizon" xmlns:xacro="http://ros.org/wiki/xacro">
-    <xacro:property name="M_PI" value="3.1415926535897931" />
-    <xacro:include filename="$(find agribot_description)/urdf/perception_sensors/lidar/velodyne.xacro"/>
-    <xacro:macro    name="livox_horizon"
-                    params="*origin
+  <xacro:property name="M_PI" value="3.1415926535897931" />
+  <xacro:include filename="$(find agribot_description)/urdf/perception_sensors/lidar/lidar_plugin.xacro" />
+  <xacro:macro name="livox_horizon" params="*origin
                             parent:=^
                             name:=^
@@ -11,24 +10,36 @@
                             perception_plugins:=^
                             ">
-        <!-- Call basic velodyne lidar and pass arguments -->
-        <xacro:velodyne parent="${parent}"
-                        name="${name}"
-                        topic="${topic}"
-                        hz="${hz}"
-                        >
-            <xacro:insert_block name="origin" />
-            <!-- Sensor specific arguments -->
-            <xacro:property name="lasers"                   value="64"/>
-            <xacro:property name="samples"                  value="320"/>
-            <xacro:property name="min_range"                value="0.5"/>
-            <xacro:property name="max_range"                value="260.0"/>
-            <xacro:property name="noise"                    value="0.01"/>
-            <xacro:property name="min_horizontal_angle"     value="-${40.85*M_PI/180.0}"/>
-            <xacro:property name="max_horizontal_angle"     value="${40.85*M_PI/180.0}"/>
-            <xacro:property name="min_vertical_angle"       value="-${12.55*M_PI/180.0}"/>
-            <xacro:property name="max_vertical_angle"       value="${12.55*M_PI/180.0}"/>
-            <xacro:property name="resolution"               value="0.001"/>
-            <xacro:property name="perception_plugins_arg"       value="${perception_plugins}"/>
-        </xacro:velodyne>
-    </xacro:macro>
+    <link name="${name}_base_link">
+      <!-- TODO(olek) - add inertial, visual and collision -->
+    </link>
+    <joint name="${name}_base_mount_joint" type="fixed">
+      <xacro:insert_block name="origin" />
+      <parent link="${parent}" />
+      <child link="${name}_base_link" />
+    </joint>
+    <!-- Optical (scan) origin -->
+    <link name="${name}_link" />
+    <joint name="${name}_base_scan_joint" type="fixed">
+      <origin xyz="0 0 0.0501" rpy="0 0 0" />
+      <parent link="${name}_base_link" />
+      <child link="${name}_link" />
+    </joint>
+    <!-- Run lidar plugin, if perception_plugins_arg set to true -->
+    <xacro:if value="${perception_plugins}">
+      <xacro:lidar_plugin name="${name}" topic="${topic}" hz="${hz}">
+        <xacro:insert_block name="origin" />
+        <!-- Sensor specific arguments -->
+        <xacro:property name="vertical_samples" value="64" />
+        <xacro:property name="horizontal_samples" value="320" />
+        <xacro:property name="min_range" value="0.5" />
+        <xacro:property name="max_range" value="260.0" />
+        <xacro:property name="noise" value="0.01" />
+        <xacro:property name="min_horizontal_angle" value="-${40.85*M_PI/180.0}" />
+        <xacro:property name="max_horizontal_angle" value="${40.85*M_PI/180.0}" />
+        <xacro:property name="min_vertical_angle" value="-${12.55*M_PI/180.0}" />
+        <xacro:property name="max_vertical_angle" value="${12.55*M_PI/180.0}" />
+        <xacro:property name="resolution" value="0.001" />
+      </xacro:lidar_plugin>
+    </xacro:if>
+  </xacro:macro>
 </robot>

Commit message: Update dimention of rotation of cart to center of the robot

File: urdf/agribot.urdf.xacro (robot description, xacro)
@@ -26,5 +26,5 @@
     <child link="front_cart_link"/>
     <limit lower="${-45*M_PI/180}" upper="${45*M_PI/180}" effort="1000.0" velocity="1000.0"/>
-    <origin xyz="${(chassis_length/2)-cart_length/2} 0.0 ${(chassis_height+cart_height)/(-2)}" rpy="0 0 0"/>
+    <origin xyz="1.11 0.0 ${(chassis_height+cart_height)/(-2)}" rpy="0 0 0"/>
     <axis xyz="0 0 1"/>
   </joint>
@@ -48,5 +48,5 @@
     <child link="back_cart_link"/>
     <limit lower="${-45*M_PI/180}" upper="${45*M_PI/180}"  effort="1000.0" velocity="1000.0"/>
-    <origin xyz="${-(chassis_length/2)+cart_length/2} 0.0 ${(chassis_height+cart_height)/(-2)}" rpy="0 0 0"/>
+    <origin xyz="-1.11 0.0 ${(chassis_height+cart_height)/(-2)}" rpy="0 0 0"/>
     <axis xyz="0 0 1"/>
   </joint>
