Commit message: Remove sonars from simulation

File: urdf/perception_sensors.xacro (robot description, xacro)
@@ -5,6 +5,4 @@
   <xacro:include filename="$(find agribot_description)/urdf/basic_sensors/lidar/livox_horizon.xacro"/>
   <xacro:include filename="$(find agribot_description)/urdf/basic_sensors/lidar/robosense_bpearl.xacro"/>
-  <xacro:include filename="$(find agribot_description)/urdf/basic_sensors/sonar/bosch_sonar.xacro"/>
-  <xacro:include filename="$(find agribot_description)/urdf/basic_sensors/sonar/balluff_sonar.xacro"/>
   <xacro:macro  name="perception_sensors"
               params="perception_plugins_arg:=^
@@ -44,133 +42,4 @@
       <xacro:property name="visualize"            value="false"/>
     </xacro:robosense_bpearl> -->
-      <!-- Front bumper sonars -->
-    <xacro:bosch_sonar>
-      <origin xyz="0.7 0.4 0.55" rpy="0 0 ${90*M_PI/180.0}" />
-      <xacro:property name="parent"               value="front_cart_link"/>
-      <xacro:property name="topic"                value="/bumper/front/sonar/left_side"/>
-      <xacro:property name="name"                 value="bumper_front_sonar_left_side"/>
-      <xacro:property name="hz"                   value="10.0"/>
-      <xacro:property name="visualize"            value="true"/>
-      <xacro:property name="perception_plugins"   value="${perception_plugins_arg}"/>
-    </xacro:bosch_sonar>
-    <xacro:bosch_sonar>
-      <origin xyz="0.8 0.2 0.55" rpy="0 0 ${45*M_PI/180.0}" />
-      <xacro:property name="parent"               value="front_cart_link"/>
-      <xacro:property name="topic"                value="/bumper/front/sonar/left"/>
-      <xacro:property name="name"                 value="bumper_front_sonar_left"/>
-      <xacro:property name="hz"                   value="10.0"/>
-      <xacro:property name="visualize"            value="true"/>
-      <xacro:property name="perception_plugins"   value="${perception_plugins_arg}"/>
-    </xacro:bosch_sonar>
-    <xacro:balluff_sonar>
-      <origin xyz="0.9 0 0.55" rpy="0 0 0" />
-      <xacro:property name="parent"               value="front_cart_link"/>
-      <xacro:property name="topic"                value="/bumper/front/sonar/center"/>
-      <xacro:property name="name"                 value="bumper_front_sonar_center"/>
-      <xacro:property name="hz"                   value="10.0"/>
-      <xacro:property name="visualize"            value="true"/>
-    </xacro:balluff_sonar>
-    <xacro:bosch_sonar>
-      <origin xyz="0.8 -0.2 0.55" rpy="0 0 -${45*M_PI/180.0}" />
-      <xacro:property name="parent"               value="front_cart_link"/>
-      <xacro:property name="topic"                value="/bumper/front/sonar/right"/>
-      <xacro:property name="name"                 value="bumper_front_sonar_right"/>
-      <xacro:property name="hz"                   value="10.0"/>
-      <xacro:property name="visualize"            value="true"/>
-      <xacro:property name="perception_plugins"   value="${perception_plugins_arg}"/>
-    </xacro:bosch_sonar>
-    <xacro:bosch_sonar>
-      <origin xyz="0.7 -0.4 0.55" rpy="0 0 -${90*M_PI/180.0}" />
-      <xacro:property name="parent"               value="front_cart_link"/>
-      <xacro:property name="topic"                value="/bumper/front/sonar/right_side"/>
-      <xacro:property name="name"                 value="bumper_front_sonar_right_side"/>
-      <xacro:property name="hz"                   value="10.0"/>
-      <xacro:property name="visualize"            value="true"/>
-      <xacro:property name="perception_plugins"   value="${perception_plugins_arg}"/>
-    </xacro:bosch_sonar>
-    <!-- Left side sonars -->
-    <xacro:bosch_sonar>
-      <origin xyz="0.45 0.5 0.0" rpy="0 0 ${90*M_PI/180.0}" />
-      <xacro:property name="parent"               value="chassis_link"/>
-      <xacro:property name="topic"                value="/agribot/sonar/left/front"/>
-      <xacro:property name="name"                 value="agribot_sonar_left_front"/>
-      <xacro:property name="hz"                   value="10.0"/>
-      <xacro:property name="visualize"            value="true"/>
-      <xacro:property name="perception_plugins"   value="${perception_plugins_arg}"/>
-    </xacro:bosch_sonar>
-    <xacro:bosch_sonar>
-      <origin xyz="-0.45 0.5 0.0" rpy="0 0 ${90*M_PI/180.0}" />
-      <xacro:property name="parent"               value="chassis_link"/>
-      <xacro:property name="topic"                value="/agribot/sonar/left/back"/>
-      <xacro:property name="name"                 value="agribot_sonar_left_back"/>
-      <xacro:property name="hz"                   value="10.0"/>
-      <xacro:property name="visualize"            value="true"/>
-      <xacro:property name="perception_plugins"   value="${perception_plugins_arg}"/>
-    </xacro:bosch_sonar>
-    <!-- Right side sonars -->
-    <xacro:bosch_sonar>
-      <origin xyz="0.45 -0.5 0.0" rpy="0 0 -${90*M_PI/180.0}" />
-      <xacro:property name="parent"               value="chassis_link"/>
-      <xacro:property name="topic"                value="/agribot/sonar/right/front"/>
-      <xacro:property name="name"                 value="agribot_sonar_right_front"/>
-      <xacro:property name="hz"                   value="10.0"/>
-      <xacro:property name="visualize"            value="true"/>
-      <xacro:property name="perception_plugins"   value="${perception_plugins_arg}"/>
-    </xacro:bosch_sonar>
-    <xacro:bosch_sonar>
-      <origin xyz="-0.45 -0.5 0.0" rpy="0 0 -${90*M_PI/180.0}" />
-      <xacro:property name="parent"               value="chassis_link"/>
-      <xacro:property name="topic"                value="/agribot/sonar/right/back"/>
-      <xacro:property name="name"                 value="agribot_sonar_right_back"/>
-      <xacro:property name="hz"                   value="10.0"/>
-      <xacro:property name="visualize"            value="true"/>
-      <xacro:property name="perception_plugins"   value="${perception_plugins_arg}"/>
-    </xacro:bosch_sonar>
-    <!-- Back bumper sonars -->
-    <xacro:bosch_sonar>
-      <origin xyz="-0.7 0.4 0.55" rpy="0 0 ${90*M_PI/180.0}" />
-      <xacro:property name="parent"               value="back_cart_link"/>
-      <xacro:property name="topic"                value="/bumper/back/sonar/left_side"/>
-      <xacro:property name="name"                 value="bumper_back_sonar_left_side"/>
-      <xacro:property name="hz"                   value="10.0"/>
-      <xacro:property name="visualize"            value="true"/>
-      <xacro:property name="perception_plugins"   value="${perception_plugins_arg}"/>
-    </xacro:bosch_sonar>
-    <xacro:bosch_sonar>
-      <origin xyz="-0.8 0.2 0.55" rpy="0 0 ${135*M_PI/180.0}" />
-      <xacro:property name="parent"               value="back_cart_link"/>
-      <xacro:property name="topic"                value="/bumper/back/sonar/left"/>
-      <xacro:property name="name"                 value="bumper_back_sonar_left"/>
-      <xacro:property name="hz"                   value="10.0"/>
-      <xacro:property name="visualize"            value="true"/>
-      <xacro:property name="perception_plugins"   value="${perception_plugins_arg}"/>
-    </xacro:bosch_sonar>
-    <xacro:balluff_sonar>
-      <origin xyz="-0.9 0 0.55" rpy="0 0 ${180*M_PI/180.0}" />
-      <xacro:property name="parent"               value="back_cart_link"/>
-      <xacro:property name="topic"                value="/bumper/back/sonar/center"/>
-      <xacro:property name="name"                 value="bumper_back_sonar_center"/>
-      <xacro:property name="hz"                   value="10.0"/>
-      <xacro:property name="visualize"            value="true"/>
-      <xacro:property name="perception_plugins"   value="${perception_plugins_arg}"/>
-    </xacro:balluff_sonar>
-    <xacro:bosch_sonar>
-      <origin xyz="-0.8 -0.2 0.55" rpy="0 0 -${135*M_PI/180.0}" />
-      <xacro:property name="parent"               value="back_cart_link"/>
-      <xacro:property name="topic"                value="/bumper/back/sonar/right"/>
-      <xacro:property name="name"                 value="bumper_back_sonar_right"/>
-      <xacro:property name="hz"                   value="10.0"/>
-      <xacro:property name="visualize"            value="true"/>
-      <xacro:property name="perception_plugins"   value="${perception_plugins_arg}"/>
-    </xacro:bosch_sonar>
-    <xacro:bosch_sonar>
-      <origin xyz="-0.7 -0.4 0.55" rpy="0 0 -${90*M_PI/180.0}" />
-      <xacro:property name="parent"               value="back_cart_link"/>
-      <xacro:property name="topic"                value="/bumper/back/sonar/right_side"/>
-      <xacro:property name="name"                 value="bumper_back_sonar_right_side"/>
-      <xacro:property name="hz"                   value="10.0"/>
-      <xacro:property name="visualize"            value="true"/>
-      <xacro:property name="perception_plugins"   value="${perception_plugins_arg}"/>
-    </xacro:bosch_sonar>
   </xacro:macro>
 </robot>

Commit message: Change lidar position to avoid collision with tools

File: urdf/perception_sensors.xacro (robot description, xacro)
@@ -28,5 +28,5 @@
     </xacro:benewake_ce30_c> -->
     <xacro:livox_horizon>
-      <origin xyz="1.3 0 1.25" rpy="0 0.2 0" />
+      <origin xyz="2.25 0 1.0" rpy="0 0.2 0" />
       <xacro:property name="parent"               value="base_footprint"/>
       <xacro:property name="topic"                value="/bumper/front/lidar"/>

Commit message: Add lidar mount on robot

File: urdf/perception_sensors.xacro (robot description, xacro)
@@ -26,5 +26,5 @@
     </xacro:benewake_ce30_c> -->
     <xacro:livox_horizon>
-      <origin xyz="2.25 0 1.0" rpy="0 0.2 0" />
+      <origin xyz="2.25 0 1.24" rpy="0 ${18.0*M_PI/180.0} 0" />
       <xacro:property name="parent"               value="base_footprint"/>
       <xacro:property name="topic"                value="/bumper/front/lidar"/>

Commit message: Add ZED2 joint. Also remove old commented lidar plugins

File: urdf/perception_sensors.xacro (robot description, xacro)
@@ -1,4 +1,4 @@
 <robot name="perception_sensors" xmlns:xacro="http://ros.org/wiki/xacro">
-  <xacro:property name="M_PI" value="3.1415926535897931" />
+  <xacro:include filename="$(find agribot_description)/urdf/common_properties.xacro"/>
   <xacro:include filename="$(find agribot_description)/urdf/basic_sensors/lidar/velodyne16.xacro"/>
   <xacro:include filename="$(find agribot_description)/urdf/basic_sensors/lidar/benewake_ce30_c.xacro"/>
@@ -9,37 +9,20 @@
                      ">
     <!-- Lidars -->
-    <!-- <xacro:velodyne16>
-      <origin xyz="1.3 0 1.25" rpy="0 0.35 0" />
-      <xacro:property name="parent"               value="base_footprint"/>
-      <xacro:property name="topic"                value="/agribot/front_lidar/v16/pc2"/>
-      <xacro:property name="name"                 value="front_lidar_v16"/>
-      <xacro:property name="hz"                   value="1.0"/>
-      <xacro:property name="visualize"            value="false"/>
-    </xacro:velodyne16> -->
-    <!-- <xacro:benewake_ce30_c>
-      <origin xyz="1.3 0 1.25" rpy="0 0.5 0" />
-      <xacro:property name="parent"               value="base_footprint"/>
-      <xacro:property name="topic"                value="/agribot/front_lidar/ce30c/pc2"/>
-      <xacro:property name="name"                 value="front_lidar_ce30c"/>
-      <xacro:property name="hz"                   value="1.0"/>
-      <xacro:property name="visualize"            value="false"/>
-    </xacro:benewake_ce30_c> -->
     <xacro:livox_horizon>
       <origin xyz="2.25 0 1.24" rpy="0 ${18.0*M_PI/180.0} 0" />
       <xacro:property name="parent"               value="base_footprint"/>
-      <xacro:property name="topic"                value="/bumper/front/lidar"/>
-      <xacro:property name="name"                 value="bumper_front_lidar"/>
+      <xacro:property name="topic"                value="/agribot/obstacle_detection/front/3d/lidar/point_cloud"/>
+      <xacro:property name="name"                 value="front_lidar"/>
       <xacro:property name="hz"                   value="1.0"/>
       <xacro:property name="visualize"            value="false"/>
       <xacro:property name="perception_plugins"   value="${perception_plugins_arg}"/>
     </xacro:livox_horizon>
-    <!-- <xacro:robosense_bpearl>
-      <origin xyz="1.3 0 1.25" rpy="0 ${M_PI/2} 0" />
-      <xacro:property name="parent"               value="base_footprint"/>
-      <xacro:property name="topic"                value="/agribot/front_lidar/robosense_bpearl/pc2"/>
-      <xacro:property name="name"                 value="front_lidar_robosense_bpearl"/>
-      <xacro:property name="hz"                   value="1.0"/>
-      <xacro:property name="visualize"            value="false"/>
-    </xacro:robosense_bpearl> -->
+    <!-- ZED2 camera -->
+    <!-- TODO(olek) - add plugin and inertial/collision info-->
+    <joint name="zed2_camera_base_joint" type="fixed">
+      <origin xyz="2.2 0 1.2991" rpy="0 ${18.0*M_PI/180.0} 0" />
+      <parent link="base_footprint"/>
+      <child link="zed2_camera_base_link" />
+    </joint>
   </xacro:macro>
 </robot>

Commit message: Add zed2 macro

File: urdf/perception_sensors.xacro (robot description, xacro)
@@ -18,10 +18,9 @@
     </xacro:livox_horizon>
     <!-- ZED2 camera -->
-    <!-- TODO(olek) - add plugin and inertial/collision info-->
-    <joint name="zed2_camera_base_joint" type="fixed">
-      <origin xyz="2.2 0 1.2991" rpy="0 ${18.0*M_PI/180.0} 0" />
-      <parent link="base_footprint"/>
-      <child link="zed2_camera_base_link" />
-    </joint>
+    <xacro:zed2>
+      <origin xyz="2.25 0 1.24" rpy="0 ${18.0*M_PI/180.0} 0" />
+      <xacro:property name="parent"               value="base_footprint"/>
+      <xacro:property name="camera_name"          value="zed2"/>
+    </xacro:zed2>
   </xacro:macro>
 </robot>

Commit message: Move camera, lidar and sonar macros to perception_sensors directory

File: urdf/perception_sensors.xacro (robot description, xacro)
@@ -1,5 +1,5 @@
 <robot name="perception_sensors" xmlns:xacro="http://ros.org/wiki/xacro">
-  <xacro:include filename="$(find agribot_description)/urdf/basic_sensors/lidar/livox_horizon.xacro"/>
-  <xacro:include filename="$(find agribot_description)/urdf/basic_sensors/camera/zed2.xacro"/>
+  <xacro:include filename="$(find agribot_description)/urdf/perception_sensors/lidar/livox_horizon.xacro"/>
+  <xacro:include filename="$(find agribot_description)/urdf/perception_sensors/camera/zed2.xacro"/>
   <xacro:macro  name="perception_sensors"
               params="perception_plugins_arg:=^

File: urdf/perception_sensors/lidar/benewake_ce30_c.xacro (robot description, xacro)
@@ -1,6 +1,6 @@
-<robot name="livox_horizon" xmlns:xacro="http://ros.org/wiki/xacro">
+<robot name="benewake_ce30_c" xmlns:xacro="http://ros.org/wiki/xacro">
     <xacro:property name="M_PI" value="3.1415926535897931" />
-    <xacro:include filename="$(find agribot_description)/urdf/basic_sensors/lidar/velodyne.xacro"/>
-    <xacro:macro    name="livox_horizon"
+    <xacro:include filename="$(find agribot_description)/urdf/perception_sensors/lidar/velodyne.xacro"/>
+    <xacro:macro    name="benewake_ce30_c"
                     params="*origin
                             parent:=^
@@ -9,5 +9,4 @@
                             hz:=^
                             visualize:=^
-                            perception_plugins:=^
                             ">
         <!-- Call basic velodyne lidar and pass arguments -->
@@ -19,15 +18,14 @@
             <xacro:insert_block name="origin" />
             <!-- Sensor specific arguments -->
-            <xacro:property name="lasers"                   value="64"/>
+            <xacro:property name="lasers"                   value="24"/>
             <xacro:property name="samples"                  value="320"/>
-            <xacro:property name="min_range"                value="0.5"/>
-            <xacro:property name="max_range"                value="260.0"/>
+            <xacro:property name="min_range"                value="0.1"/>
+            <xacro:property name="max_range"                value="4.0"/>
             <xacro:property name="noise"                    value="0.01"/>
-            <xacro:property name="min_horizontal_angle"     value="-${40.85*M_PI/180.0}"/>
-            <xacro:property name="max_horizontal_angle"     value="${40.85*M_PI/180.0}"/>
-            <xacro:property name="min_vertical_angle"       value="-${12.55*M_PI/180.0}"/>
-            <xacro:property name="max_vertical_angle"       value="${12.55*M_PI/180.0}"/>
+            <xacro:property name="min_horizontal_angle"     value="-${66.0*M_PI/180.0}"/>
+            <xacro:property name="max_horizontal_angle"     value="${66.0*M_PI/180.0}"/>
+            <xacro:property name="min_vertical_angle"       value="-${4.5*M_PI/180.0}"/>
+            <xacro:property name="max_vertical_angle"       value="${4.5*M_PI/180.0}"/>
             <xacro:property name="resolution"               value="0.001"/>
-            <xacro:property name="perception_plugins_arg"       value="${perception_plugins}"/>
         </xacro:velodyne>
     </xacro:macro>

File: urdf/perception_sensors/lidar/livox_horizon.xacro (robot description, xacro)
@@ -1,6 +1,6 @@
-<robot name="benewake_ce30_c" xmlns:xacro="http://ros.org/wiki/xacro">
+<robot name="livox_horizon" xmlns:xacro="http://ros.org/wiki/xacro">
     <xacro:property name="M_PI" value="3.1415926535897931" />
-    <xacro:include filename="$(find agribot_description)/urdf/basic_sensors/lidar/velodyne.xacro"/>
-    <xacro:macro    name="benewake_ce30_c"
+    <xacro:include filename="$(find agribot_description)/urdf/perception_sensors/lidar/velodyne.xacro"/>
+    <xacro:macro    name="livox_horizon"
                     params="*origin
                             parent:=^
@@ -9,4 +9,5 @@
                             hz:=^
                             visualize:=^
+                            perception_plugins:=^
                             ">
         <!-- Call basic velodyne lidar and pass arguments -->
@@ -18,14 +19,15 @@
             <xacro:insert_block name="origin" />
             <!-- Sensor specific arguments -->
-            <xacro:property name="lasers"                   value="24"/>
+            <xacro:property name="lasers"                   value="64"/>
             <xacro:property name="samples"                  value="320"/>
-            <xacro:property name="min_range"                value="0.1"/>
-            <xacro:property name="max_range"                value="4.0"/>
+            <xacro:property name="min_range"                value="0.5"/>
+            <xacro:property name="max_range"                value="260.0"/>
             <xacro:property name="noise"                    value="0.01"/>
-            <xacro:property name="min_horizontal_angle"     value="-${66.0*M_PI/180.0}"/>
-            <xacro:property name="max_horizontal_angle"     value="${66.0*M_PI/180.0}"/>
-            <xacro:property name="min_vertical_angle"       value="-${4.5*M_PI/180.0}"/>
-            <xacro:property name="max_vertical_angle"       value="${4.5*M_PI/180.0}"/>
+            <xacro:property name="min_horizontal_angle"     value="-${40.85*M_PI/180.0}"/>
+            <xacro:property name="max_horizontal_angle"     value="${40.85*M_PI/180.0}"/>
+            <xacro:property name="min_vertical_angle"       value="-${12.55*M_PI/180.0}"/>
+            <xacro:property name="max_vertical_angle"       value="${12.55*M_PI/180.0}"/>
             <xacro:property name="resolution"               value="0.001"/>
+            <xacro:property name="perception_plugins_arg"       value="${perception_plugins}"/>
         </xacro:velodyne>
     </xacro:macro>

File: urdf/perception_sensors/lidar/robosense_bpearl.xacro (robot description, xacro)
@@ -1,5 +1,5 @@
 <robot name="robosense_bpearl" xmlns:xacro="http://ros.org/wiki/xacro">
     <xacro:property name="M_PI" value="3.1415926535897931" />
-    <xacro:include filename="$(find agribot_description)/urdf/basic_sensors/lidar/velodyne.xacro"/>
+    <xacro:include filename="$(find agribot_description)/urdf/perception_sensors/lidar/velodyne.xacro"/>
     <xacro:macro    name="robosense_bpearl"
                     params="*origin

File: urdf/perception_sensors/lidar/velodyne16.xacro (robot description, xacro)
@@ -1,5 +1,5 @@
 <robot name="velodyne16" xmlns:xacro="http://ros.org/wiki/xacro">
     <xacro:property name="M_PI" value="3.1415926535897931" />
-    <xacro:include filename="$(find agribot_description)/urdf/basic_sensors/lidar/velodyne.xacro"/>
+    <xacro:include filename="$(find agribot_description)/urdf/perception_sensors/lidar/velodyne.xacro"/>
     <xacro:macro    name="velodyne16"
                     params="*origin

File: urdf/perception_sensors/sonar/balluff_sonar.xacro (robot description, xacro)
@@ -1,5 +1,5 @@
 <robot name="balluff_sonar" xmlns:xacro="http://ros.org/wiki/xacro">
     <xacro:property name="M_PI" value="3.1415926535897931" />
-    <xacro:include filename="$(find agribot_description)/urdf/basic_sensors/sonar/sonar.xacro"/>
+    <xacro:include filename="$(find agribot_description)/urdf/perception_sensors/sonar/sonar.xacro"/>
     <xacro:macro    name="balluff_sonar"
                     params="*origin

File: urdf/perception_sensors/sonar/bosch_sonar.xacro (robot description, xacro)
@@ -1,5 +1,5 @@
 <robot name="bosch_sonar" xmlns:xacro="http://ros.org/wiki/xacro">
     <xacro:property name="M_PI" value="3.1415926535897931" />
-    <xacro:include filename="$(find agribot_description)/urdf/basic_sensors/sonar/sonar.xacro"/>
+    <xacro:include filename="$(find agribot_description)/urdf/perception_sensors/sonar/sonar.xacro"/>
     <xacro:macro    name="bosch_sonar"
                     params="*origin

Commit message: Mount livox_zed2_set with respect to front_cart_link instead of base_footprint

File: urdf/perception_sensors.xacro (robot description, xacro)
@@ -5,6 +5,6 @@
     <!-- Lidars -->
     <xacro:livox_zed2_set>
-      <origin xyz="2.25 0 1.24" rpy="0 ${25.0*M_PI/180.0} 0" />
-      <xacro:property name="parent" value="base_footprint" />
+      <origin xyz="1.47 0 0.98" rpy="0 ${25.0*M_PI/180.0} 0" />
+      <xacro:property name="parent" value="front_cart_link" />
       <xacro:property name="suite_name" value="front_livox_zed2_set" />
       <xacro:property name="livox_name" value="front_lidar" />

Commit message: Mount zed-livox set on the chassis

File: urdf/perception_sensors.xacro (robot description, xacro)
@@ -5,6 +5,6 @@
     <!-- Lidars -->
     <xacro:livox_zed2_set>
-      <origin xyz="1.47 0 0.98" rpy="0 ${25.0*M_PI/180.0} 0" />
-      <xacro:property name="parent" value="front_cart_link" />
+      <origin xyz="1.15 0 2.05" rpy="0 ${28.9*M_PI/180.0} 0" />
+      <xacro:property name="parent" value="base_footprint" />
       <xacro:property name="suite_name" value="front_livox_zed2_set" />
       <xacro:property name="livox_name" value="front_lidar" />
