Commit message: Changed point cloud topic to mimic real zed2 topic

File: urdf/perception_sensors.xacro (robot description, xacro)
@@ -10,4 +10,5 @@
       <xacro:property name="livox_name" value="front_lidar" />
       <xacro:property name="livox_topic" value="/agribot/obstacle_detection/front/3d/lidar/point_cloud" />
+      <xacro:property name="zed2_topic" value="/agribot/obstacle_detection/front/3d/stereo_camera" />
       <xacro:property name="livox_hz" value="1.0" />
       <xacro:property name="livox_visualize" value="false" />

File: urdf/perception_sensors/camera/zed2.xacro (robot description, xacro)
@@ -7,4 +7,5 @@
                        parent:=^
                        camera_name:=^
+                       topic:=^
                       ">
     <!-- Properties -->
@@ -87,9 +88,8 @@
         <update_rate>20</update_rate>
         <camera>
-          <horizontal_fov>1.047198</horizontal_fov>
-          <vertical_fov></vertical_fov>
+          <horizontal_fov>1.9198621772</horizontal_fov>
           <image>
-            <width>640</width>
-            <height>480</height>
+            <width>1280</width>
+            <height>720</height>
             <format>R8G8B8</format>
           </image>
@@ -100,25 +100,25 @@
         </camera>
         <plugin name="${camera_name}_controller" filename="libgazebo_ros_openni_kinect.so">
-          <baseline>0.2</baseline>
+          <baseline>0.12</baseline>
           <alwaysOn>true</alwaysOn>
           <updateRate>0</updateRate>
           <cameraName>${camera_name}_ir</cameraName>
-          <imageTopicName>/${camera_name}/color/image_raw</imageTopicName>
-          <cameraInfoTopicName>/${camera_name}/color/camera_info</cameraInfoTopicName>
-          <depthImageTopicName>/${camera_name}/depth/image_raw</depthImageTopicName>
-          <depthImageInfoTopicName>/${camera_name}/depth/camera_info</depthImageInfoTopicName>
-          <pointCloudTopicName>/${camera_name}/depth/points</pointCloudTopicName>
+          <imageTopicName>/${topic}/color/image_raw</imageTopicName>
+          <cameraInfoTopicName>/${topic}/color/camera_info</cameraInfoTopicName>
+          <depthImageTopicName>/${topic}/image_raw</depthImageTopicName>
+          <depthImageInfoTopicName>${topic}/camera_info</depthImageInfoTopicName>
+          <pointCloudTopicName>${topic}/point_cloud</pointCloudTopicName>
           <frameName>${camera_name}_center_camera_optical_frame</frameName>
-          <pointCloudCutoff>0.2</pointCloudCutoff>
-          <pointCloudCutoffMax>10.0</pointCloudCutoffMax>
-          <distortionK1>0.00000001</distortionK1>
-          <distortionK2>0.00000001</distortionK2>
-          <distortionK3>0.00000001</distortionK3>
-          <distortionT1>0.00000001</distortionT1>
-          <distortionT2>0.00000001</distortionT2>
+          <pointCloudCutoff>0.3</pointCloudCutoff>
+          <pointCloudCutoffMax>20.0</pointCloudCutoffMax>
+          <distortionK1>0</distortionK1>
+          <distortionK2>0</distortionK2>
+          <distortionK3>0.0</distortionK3>
+          <distortionT1>0</distortionT1>
+          <distortionT2>0</distortionT2>
           <CxPrime>0</CxPrime>
           <Cx>0</Cx>
           <Cy>0</Cy>
-          <focalLength>0</focalLength>
+          <focalLength>0.00212</focalLength>
           <hackBaseline>0</hackBaseline>
         </plugin>

File: urdf/perception_sensors/perception_suites/livox_zed2_set.xacro (robot description, xacro)
@@ -7,4 +7,5 @@
                           livox_name:=^
                           livox_topic:=^
+                          zed2_topic:=^
                           livox_hz:=^
                           livox_visualize:=^
@@ -37,4 +38,5 @@
       <xacro:property name="parent" value="${suite_name}_link" />
       <xacro:property name="camera_name" value="zed2" />
+      <xacro:property name="topic" value="${zed2_topic}" />
     </xacro:zed2>
   </xacro:macro>

Commit message: Added seperate parameters for topics

File: urdf/perception_sensors.xacro (robot description, xacro)
@@ -10,5 +10,9 @@
       <xacro:property name="livox_name" value="front_lidar" />
       <xacro:property name="livox_topic" value="/agribot/obstacle_detection/front/3d/lidar/point_cloud" />
-      <xacro:property name="zed2_topic" value="/agribot/obstacle_detection/front/3d/stereo_camera" />
+      <xacro:property name="zed2_point_cloud_topic" value="/agribot/obstacle_detection/front/3d/stereo_camera/point_cloud" />
+      <xacro:property name="zed2_image_topic" />
+      <xacro:property name="zed2_image_camera_info_topic" />
+      <xacro:property name="zed2_depth_image_topic" />
+      <xacro:property name="zed2_depth_image_camera_info_topic" />
       <xacro:property name="livox_hz" value="1.0" />
       <xacro:property name="livox_visualize" value="false" />

File: urdf/perception_sensors/camera/zed2.xacro (robot description, xacro)
@@ -6,5 +6,9 @@
                        parent:=^
                        camera_name:=^
-                       topic:=^
+                       point_cloud_topic:=^
+                       depth_image_topic:=^
+                       depth_image_camera_info_topic:=^
+                       image_topic:=^
+                       image_camera_info_topic:=^
                       ">
     <!-- Properties -->
@@ -52,5 +56,5 @@
     </joint>
     <link name="${camera_name}_right_camera_optical_frame" />
-     <joint name="${camera_name}_center_camera_optical_joint" type="fixed">
+    <joint name="${camera_name}_center_camera_optical_joint" type="fixed">
       <origin xyz="0 0 0" rpy="-${M_PI/2} 0.0 -${M_PI/2}" />
       <parent link="${camera_name}_camera_center" />
@@ -85,5 +89,5 @@
     <gazebo reference="${camera_name}_camera_center">
       <sensor name="${camera_name}_camera" type="depth">
-        <update_rate>20</update_rate>
+        <update_rate>5</update_rate>
         <camera>
           <horizontal_fov>1.9198621772</horizontal_fov>
@@ -94,6 +98,6 @@
           </image>
           <clip>
-            <near>0.02</near>
-            <far>300</far>
+            <near>0.3</near>
+            <far>20.0</far>
           </clip>
         </camera>
@@ -102,23 +106,23 @@
           <alwaysOn>true</alwaysOn>
           <updateRate>0</updateRate>
-          <cameraName>${camera_name}_ir</cameraName>
-          <imageTopicName>/${topic}/image_raw</imageTopicName>
-          <cameraInfoTopicName>/${topic}/camera_info</cameraInfoTopicName>
-          <depthImageTopicName>/${topic}/depth_image</depthImageTopicName>
-          <depthImageInfoTopicName>${topic}/depth_camera_info</depthImageInfoTopicName>
-          <pointCloudTopicName>${topic}/point_cloud</pointCloudTopicName>
+          <cameraName>${camera_name}</cameraName>
+          <imageTopicName>${image_topic}</imageTopicName>
+          <cameraInfoTopicName>${image_camera_info_topic}</cameraInfoTopicName>
+          <depthImageTopicName>${depth_image_topic}</depthImageTopicName>
+          <depthImageCameraInfoTopicName>${depth_image_camera_info_topic}</depthImageCameraInfoTopicName>
+          <pointCloudTopicName>${point_cloud_topic}</pointCloudTopicName>
           <frameName>${camera_name}_center_camera_optical_frame</frameName>
           <pointCloudCutoff>0.3</pointCloudCutoff>
           <pointCloudCutoffMax>20.0</pointCloudCutoffMax>
-          <distortionK1>0</distortionK1>
-          <distortionK2>0</distortionK2>
+          <distortionK1>0.0</distortionK1>
+          <distortionK2>0.0</distortionK2>
           <distortionK3>0.0</distortionK3>
-          <distortionT1>0</distortionT1>
-          <distortionT2>0</distortionT2>
-          <CxPrime>0</CxPrime>
-          <Cx>0</Cx>
-          <Cy>0</Cy>
-          <focalLength>0</focalLength>
-          <hackBaseline>0</hackBaseline>
+          <distortionT1>0.0</distortionT1>
+          <distortionT2>0.0</distortionT2>
+          <CxPrime>0.0</CxPrime>
+          <Cx>0.0</Cx>
+          <Cy>0.0</Cy>
+          <focalLength>0.0</focalLength>
+          <hackBaseline>0.0</hackBaseline>
         </plugin>
       </sensor>

File: urdf/perception_sensors/perception_suites/livox_zed2_set.xacro (robot description, xacro)
@@ -7,5 +7,5 @@
                           livox_name:=^
                           livox_topic:=^
-                          zed2_topic:=^
+                          zed2_topic_namespace:=^
                           livox_hz:=^
                           livox_visualize:=^
@@ -38,5 +38,9 @@
       <xacro:property name="parent" value="${suite_name}_link" />
       <xacro:property name="camera_name" value="zed2" />
-      <xacro:property name="topic" value="${zed2_topic}" />
+      <xacro:property name="point_cloud_topic" value="${zed2_point_cloud_topic}" />
+      <xacro:property name="depth_image_topic" value="${zed2_depth_image_topic}" />
+      <xacro:property name="depth_image_camera_info_topic" value="${zed2_depth_image_camera_info_topic}" />
+      <xacro:property name="image_topic" value="${zed2_image_topic}" />
+      <xacro:property name="image_camera_info_topic" value="${zed2_image_camera_info_topic}" />
     </xacro:zed2>
   </xacro:macro>

Commit message: Changed topics for zed2 gazebo

File: urdf/perception_sensors.xacro (robot description, xacro)
@@ -11,8 +11,8 @@
       <xacro:property name="livox_topic" value="/agribot/obstacle_detection/front/3d/lidar/point_cloud" />
       <xacro:property name="zed2_point_cloud_topic" value="/agribot/obstacle_detection/front/3d/stereo_camera/point_cloud" />
-      <xacro:property name="zed2_image_topic" />
-      <xacro:property name="zed2_image_camera_info_topic" />
-      <xacro:property name="zed2_depth_image_topic" />
-      <xacro:property name="zed2_depth_image_camera_info_topic" />
+      <xacro:property name="zed2_image_topic" value="/zed2_node/rgb/image_rect_color" />
+      <xacro:property name="zed2_image_camera_info_topic" value="/zed2_node/rgb/camera_info" />
+      <xacro:property name="zed2_depth_image_topic" value="/zed2_node/stereo/image_rect_color" />
+      <xacro:property name="zed2_depth_image_camera_info_topic" value="/zed2_node/stereo/camera_info" />
       <xacro:property name="livox_hz" value="1.0" />
       <xacro:property name="livox_visualize" value="false" />

File: urdf/perception_sensors/perception_suites/livox_zed2_set.xacro (robot description, xacro)
@@ -7,5 +7,9 @@
                           livox_name:=^
                           livox_topic:=^
-                          zed2_topic_namespace:=^
+                          zed2_image_topic:=^
+                          zed2_image_camera_info_topic:=^
+                          zed2_depth_image_topic:=^
+                          zed2_depth_image_camera_info_topic:=^
+                          zed2_point_cloud_topic:=^
                           livox_hz:=^
                           livox_visualize:=^
