Commit message: Fixed problem with gazebo gui in sim

File: urdf/basic_links/tpl/tpl_base.xacro (robot description, xacro)
@@ -14,5 +14,5 @@
         </xacro:if>
         <geometry>
-          <box size="0 0 0"/>
+          <box size="0.0001 0.0001 0.0001"/>
         </geometry>
       </visual>

File: urdf/basic_links/tpl/tpl_rev_hit_base.xacro (robot description, xacro)
@@ -20,5 +20,5 @@
         </xacro:if>
         <geometry>
-          <box size="0 0 0"/>
+          <box size="0.0001 0.0001 0.0001"/>
         </geometry>
       </visual>

File: urdf/basic_links/tpl/tpl_rev_hit_effector.xacro (robot description, xacro)
@@ -20,5 +20,5 @@
           </xacro:if>
           <geometry>
-            <box size="0 0 0"/>
+            <box size="0.0001 0.0001 0.0001"/>
           </geometry>
         </visual>

File: urdf/basic_links/tpl/tpl_upper_hit_base.xacro (robot description, xacro)
@@ -14,5 +14,5 @@
           </xacro:if>
           <geometry>
-            <box size="0 0 0"/>
+            <box size="0.0001 0.0001 0.0001"/>
           </geometry>
         </visual>

File: urdf/basic_links/tpl/tpl_upper_hit_base_cyl.xacro (robot description, xacro)
@@ -13,5 +13,5 @@
           </xacro:if>
           <geometry>
-            <cylinder length="0" radius="0"/>
+            <cylinder length="0.0001" radius="0.0001"/>
           </geometry>
         </visual>

Commit message: Agribot is moving like before TPL addition

File: urdf/basic_links/tpl/tpl_base.xacro (robot description, xacro)
@@ -3,5 +3,5 @@
   <xacro:property name="tpl_base_wid" value="0.3" />
   <xacro:property name="tpl_base_hei" value="0.05" />
-  <xacro:property name="tpl_base_mass" value="300" />
+  <xacro:property name="tpl_base_mass" value="0.001" />
   <xacro:macro name="agribot_tpl_base" params="name">
     <link name="${name}">

File: urdf/basic_links/tpl/tpl_cyl.xacro (robot description, xacro)
@@ -2,5 +2,5 @@
   <xacro:property name="tpl_cyl_width" value="0.45" />
   <xacro:property name="tpl_cyl_radius" value="${tpl_base_hei/2}" />
-  <xacro:property name="tpl_cyl_mass" value="50" />
+  <xacro:property name="tpl_cyl_mass" value="0.001" />
   <xacro:macro name="agribot_tpl_cylinder" params="name">
     <link name="${name}">

File: urdf/basic_links/tpl/tpl_rev_hit_base.xacro (robot description, xacro)
@@ -3,5 +3,5 @@
   <xacro:property name="tpl_rev_hit_base_wid" value="${2*tpl_base_hei}" />
   <xacro:property name="tpl_rev_hit_base_hei" value="0.05" />
-  <xacro:property name="tpl_rev_hit_base_mass" value="20.0" />
+  <xacro:property name="tpl_rev_hit_base_mass" value="0.001" />
   <xacro:macro name="agribot_tpl_revolute_hitch_base" params="name">
     <link name="${name}">

File: urdf/basic_links/tpl/tpl_rev_hit_effector.xacro (robot description, xacro)
@@ -3,5 +3,5 @@
     <xacro:property name="tpl_rev_hit_effector_wid" value="${3.5*tpl_base_hei}" />
     <xacro:property name="tpl_rev_hit_effector_hei" value="0.05" />
-    <xacro:property name="tpl_rev_hit_effector_mass" value="25.0" />
+    <xacro:property name="tpl_rev_hit_effector_mass" value="0.001" />
     <xacro:macro name="agribot_tpl_revolute_hitch_effector" params="name">
       <link name="${name}">

File: urdf/basic_links/tpl/tpl_upper_hit_base.xacro (robot description, xacro)
@@ -3,5 +3,5 @@
     <xacro:property name="tpl_upper_hit_base_wid" value="0.3" />
     <xacro:property name="tpl_upper_hit_base_hei" value="0.05" />
-    <xacro:property name="tpl_upper_hit_base_mass" value="15.0" />
+    <xacro:property name="tpl_upper_hit_base_mass" value="0.001" />
     <xacro:macro name="agribot_tpl_upper_hitch_base" params="name">
       <link name="${name}">

File: urdf/basic_links/tpl/tpl_upper_hit_base_cyl.xacro (robot description, xacro)
@@ -2,5 +2,5 @@
     <xacro:property name="tpl_upper_hit_base_cyl_width" value="${tpl_upper_hit_base_wid}" />
     <xacro:property name="tpl_upper_hit_base_cyl_radius" value="${tpl_cyl_radius}" />
-    <xacro:property name="tpl_upper_hit_base_cyl_mass" value="10" />
+    <xacro:property name="tpl_upper_hit_base_cyl_mass" value="0.001" />
     <xacro:macro name="agribot_tpl_upper_hitch_cylinder" params="name">
       <link name="${name}">

File: urdf/basic_links/tpl/tpl_upper_hitch_prism_base.xacro (robot description, xacro)
@@ -3,5 +3,5 @@
     <xacro:property name="tpl_upper_hitch_prism_base_wid" value="0.05" />
     <xacro:property name="tpl_upper_hitch_prism_base_hei" value="0.05" />
-    <xacro:property name="tpl_upper_hitch_prism_base_mass" value="10.0" />
+    <xacro:property name="tpl_upper_hitch_prism_base_mass" value="0.001" />
     <xacro:macro name="agribot_tpl_upper_hitch_prism_joint_base" params="name">
       <link name="${name}">

File: urdf/basic_links/tpl/tpl_upper_hitch_prism_core.xacro (robot description, xacro)
@@ -3,5 +3,5 @@
     <xacro:property name="tpl_upper_hitch_prism_core_wid" value="0.025" />
     <xacro:property name="tpl_upper_hitch_prism_core_hei" value="0.025" />
-    <xacro:property name="tpl_upper_hitch_prism_core_mass" value="8.0" />
+    <xacro:property name="tpl_upper_hitch_prism_core_mass" value="0.001" />
     <xacro:macro name="agribot_tpl_upper_hitch_prism_joint_core" params="name">
       <link name="${name}">

File: urdf/basic_links/wheel.xacro (robot description, xacro)
@@ -28,6 +28,6 @@
         </link>
         <gazebo reference="${name}">
-          <mu1>0.1</mu1>
-          <mu2>0.1</mu2>
+          <mu1>0.5</mu1>
+          <mu2>0.5</mu2>
           <kp>5e9</kp>
           <kd>10.0</kd>
