Commit message: Add COLLADA meshes instead of simple boxes

File: urdf/basic_links/cart.xacro (robot description, xacro)
@@ -8,9 +8,13 @@
         <link name="${name}">
           <visual>
-            <origin xyz="0.0 0.0 0.0" rpy="0 0 0"/>
+            <xacro:if value="${name == 'back_cart_link'}">
+              <origin xyz="${cart_width} 0.0 0.0" rpy="1.57 0 1.57"/>
+            </xacro:if>
+            <xacro:if value="${name == 'front_cart_link'}">
+              <origin xyz="-${cart_width} 0.0 0.0" rpy="1.57 0 -1.57"/>
+            </xacro:if>
             <geometry>
-               <box size="${cart_lenght} ${cart_width} ${cart_height}" />
+              <mesh filename="package://agribot_description/meshes/agribot_cart.dae" scale="1 1 1"/>
             </geometry>
-            <material name="blue"/>
           </visual>
           <collision>

File: urdf/basic_links/chassis.xacro (robot description, xacro)
@@ -9,9 +9,8 @@
         <link name="${name}">
           <visual>
-            <origin xyz="0.0 0.0 0.0" rpy="0 0 0"/>
+            <origin xyz="0.0 0.0 -${chassis_width}" rpy="1.57 0 1.57"/>
             <geometry>
-               <box size="${chassis_length} ${chassis_width} ${chassis_height}" />
+              <mesh filename="package://agribot_description/meshes/agribot_chassis.dae" scale="1 1 1"/>
             </geometry>
-            <material name="blue"/>
           </visual>
           <collision>

File: urdf/basic_links/wheel.xacro (robot description, xacro)
@@ -6,11 +6,4 @@
     <xacro:macro name="agribot_wheel" params="name">
         <link name="${name}">
-          <visual>
-            <origin xyz="0 0 0" rpy="0 0 0"/>
-            <geometry>
-                <cylinder length="${wheel_width}" radius="${wheel_radius}"/>
-            </geometry>
-            <material name="blue"/>
-          </visual>
           <collision>
             <origin rpy="0 0 0" xyz="0 0 0"/>

Commit message: Change COLLADA meshes to STL

File: urdf/basic_links/cart.xacro (robot description, xacro)
@@ -9,11 +9,13 @@
           <visual>
             <xacro:if value="${name == 'back_cart_link'}">
-              <origin xyz="${cart_width} 0.0 0.0" rpy="1.57 0 1.57"/>
+              <origin xyz="-0.25 0.0 0.3" rpy="0 0 1.57"/>
+              <material name="white"/>
             </xacro:if>
             <xacro:if value="${name == 'front_cart_link'}">
-              <origin xyz="-${cart_width} 0.0 0.0" rpy="1.57 0 -1.57"/>
+              <origin xyz="0.25 0.0 0.3" rpy="0 0 -1.57"/>
+              <material name="green"/>
             </xacro:if>
             <geometry>
-              <mesh filename="package://agribot_description/meshes/agribot_cart.dae" scale="1 1 1"/>
+              <mesh filename="package://agribot_description/meshes/agribot_cart.stl" scale="0.01 0.01 0.01"/>
             </geometry>
           </visual>

File: urdf/basic_links/chassis.xacro (robot description, xacro)
@@ -9,8 +9,9 @@
         <link name="${name}">
           <visual>
-            <origin xyz="0.0 0.0 -${chassis_width}" rpy="1.57 0 1.57"/>
+            <origin xyz="0.0 0.0 0" rpy="0 0 1.57"/>
             <geometry>
-              <mesh filename="package://agribot_description/meshes/agribot_chassis.dae" scale="1 1 1"/>
+              <mesh filename="package://agribot_description/meshes/agribot_chassis.stl" scale="0.01 0.01 0.01"/>
             </geometry>
+            <material name="green"/>
           </visual>
           <collision>

Commit message: Update collission model

File: urdf/basic_links/cart.xacro (robot description, xacro)
@@ -21,7 +21,14 @@
           </visual>
           <collision>
-            <origin xyz="0.0 0.0 0.0" rpy="0 0 0"/>
+            <xacro:if value="${name == 'back_cart_link'}">
+              <origin xyz="-0.25 0.0 0.3" rpy="0 0 1.57"/>
+              <material name="white"/>
+            </xacro:if>
+            <xacro:if value="${name == 'front_cart_link'}">
+              <origin xyz="0.25 0.0 0.3" rpy="0 0 -1.57"/>
+              <material name="green"/>
+            </xacro:if>
             <geometry>
-              <box size="${cart_lenght} ${cart_width} ${cart_height}"/>
+              <mesh filename="package://agribot_description/meshes/agribot_cart.stl" scale="0.01 0.01 0.01"/>
             </geometry>
           </collision>

File: urdf/basic_links/chassis.xacro (robot description, xacro)
@@ -16,8 +16,9 @@
           </visual>
           <collision>
-            <origin xyz="0.0 0.0 0.0" rpy="0 0 0"/>
+            <origin xyz="0.0 0.0 0" rpy="0 0 1.57"/>
             <geometry>
-              <box size="${chassis_length} ${chassis_width} ${chassis_height}"/>
+              <mesh filename="package://agribot_description/meshes/agribot_chassis.stl" scale="0.01 0.01 0.01"/>
             </geometry>
+            <material name="green"/>
           </collision>
           <inertial>

File: urdf/basic_links/support.xacro (robot description, xacro)
@@ -17,6 +17,7 @@
             <origin xyz="0.0 0.0 0.0" rpy="0 0 0"/>
             <geometry>
-              <box size="${support_length} ${support_width} ${support_height}"/>
+               <box size="${support_length} ${support_width} ${support_height}" />
             </geometry>
+            <material name="blue"/>
           </collision>
           <inertial>

Commit message: STL replacement in progress

File: urdf/basic_links/cart.xacro (robot description, xacro)
@@ -8,13 +8,13 @@
           <visual>
             <xacro:if value="${name == 'back_cart_link'}">
-              <origin xyz="-0.25 0.0 0.3" rpy="0 0 1.57"/>
+              <origin xyz="0.0 0.0 0.0" rpy="${M_PI/2} 0 ${M_PI/2}"/>
               <material name="white"/>
             </xacro:if>
             <xacro:if value="${name == 'front_cart_link'}">
-              <origin xyz="0.25 0.0 0.3" rpy="0 0 -1.57"/>
+              <origin xyz="-0.9 -0.1 0.0" rpy="${M_PI/2} 0 ${-M_PI/2}"/>
               <material name="green"/>
             </xacro:if>
             <geometry>
-              <mesh filename="package://agribot_description/meshes/agribot_cart.stl" scale="0.01 0.01 0.01"/>
+              <mesh filename="package://agribot_description/meshes/agribot_cart.stl" scale="0.001 0.001 0.001"/>
             </geometry>
           </visual>

Commit message: Model changed to fit new STLs

File: urdf/basic_links/cart.xacro (robot description, xacro)
@@ -8,13 +8,13 @@
           <visual>
             <xacro:if value="${name == 'back_cart_link'}">
-              <origin xyz="0.0 0.0 0.0" rpy="${M_PI/2} 0 ${M_PI/2}"/>
+              <origin xyz="1.155 0.1 0.092" rpy="${M_PI/2} 0 ${M_PI/2}"/>
               <material name="white"/>
             </xacro:if>
             <xacro:if value="${name == 'front_cart_link'}">
-              <origin xyz="-0.9 -0.1 0.0" rpy="${M_PI/2} 0 ${-M_PI/2}"/>
+              <origin xyz="-1.155 -0.1 0.092" rpy="${M_PI/2} 0 ${-M_PI/2}"/>
               <material name="green"/>
             </xacro:if>
             <geometry>
-              <mesh filename="package://agribot_description/meshes/agribot_cart.stl" scale="0.001 0.001 0.001"/>
+              <mesh filename="package://agribot_description/meshes/agribot_cart.stl" scale="0.00105 0.00105 0.00105"/>
             </geometry>
           </visual>

File: urdf/basic_links/chassis.xacro (robot description, xacro)
@@ -2,10 +2,10 @@
     <xacro:property name="chassis_length" value="2.42" />
     <xacro:property name="chassis_width" value="1.05" />
-    <xacro:property name="chassis_height" value="1.3" />
+    <xacro:property name="chassis_height" value="1.65" />
     <xacro:property name="chassis_mass" value="2000" />
     <xacro:macro name="agribot_chassis" params="name">
         <link name="${name}">
           <visual>
-            <origin xyz="0.0 0.0 0" rpy="0 0 1.57"/>
+            <origin xyz="0.0 0.0 0.1" rpy="0 0 1.57"/>
             <geometry>
               <mesh filename="package://agribot_description/meshes/agribot_chassis.stl" scale="0.01 0.01 0.01"/>

File: urdf/basic_links/tpl/tpl_assembled.xacro (robot description, xacro)
@@ -13,5 +13,5 @@
       <parent link="back_cart_link"/>
       <child link="back_tpl_base_link"/>
-      <origin xyz="${-(cart_lenght+tpl_base_len)/2} 0.0 ${(cart_height-tpl_base_hei)/2}" rpy="0 0 0"/>
+      <origin xyz="${-(cart_lenght+tpl_base_len)/2} 0.0 ${(cart_height-tpl_base_hei)/2}" rpy="0 ${M_PI/36} 0"/>
       <axis xyz="0 0 1"/>
     </joint>
@@ -35,5 +35,5 @@
       <parent link="back_tpl_revolute_hitch_base_left_link"/>
       <child link="back_tpl_revolute_hitch_effector_left_link"/>
-      <origin xyz="${-0.4*(tpl_rev_hit_base_len+tpl_rev_hit_effector_len)} 0.1 ${-0.22*tpl_rev_hit_effector_len}" rpy="0 ${-M_PI/6} ${-M_PI/6}"/>
+      <origin xyz="${-0.43*(tpl_rev_hit_base_len+tpl_rev_hit_effector_len)} 0.12 ${-0.28*tpl_rev_hit_effector_len}" rpy="0 ${-M_PI/6} ${-M_PI/6}"/>
       <axis xyz="0 0 1"/>
     </joint>
@@ -49,5 +49,5 @@
       <parent link="back_tpl_revolute_hitch_base_right_link"/>
       <child link="back_tpl_revolute_hitch_effector_right_link"/>
-      <origin xyz="${-0.4*(tpl_rev_hit_base_len+tpl_rev_hit_effector_len)} 0.1 ${0.22*tpl_rev_hit_effector_len}" rpy="0 ${M_PI/6} ${-M_PI/6}"/>
+      <origin xyz="${-0.43*(tpl_rev_hit_base_len+tpl_rev_hit_effector_len)} 0.12 ${0.28*tpl_rev_hit_effector_len}" rpy="0 ${M_PI/6} ${-M_PI/6}"/>
       <axis xyz="0 0 1"/>
     </joint>
@@ -56,5 +56,5 @@
       <parent link="back_tpl_base_link"/>
       <child link="back_tpl_up_hit_base_link"/>
-      <origin xyz="${-0.82*tpl_base_len} 0.0 ${0.8*(tpl_upper_hit_base_len)/2}" rpy="0 ${M_PI/3.15} 0"/>
+      <origin xyz="${-0.78*tpl_base_len} 0.0 ${0.8*(tpl_upper_hit_base_len)/2}" rpy="0 ${M_PI/3.43} 0"/>
       <axis xyz="0 0 1"/>
     </joint>
@@ -88,5 +88,5 @@
       <parent link="front_cart_link"/>
       <child link="front_tpl_base_link"/>
-      <origin xyz="${(cart_lenght+tpl_base_len)/2} 0.0 ${(cart_height-tpl_base_hei)/2}" rpy="0 0 0"/>
+      <origin xyz="${(cart_lenght+tpl_base_len)/2} 0.0 ${(cart_height-tpl_base_hei)/2}" rpy="0 ${-M_PI/36} 0"/>
       <axis xyz="0 0 1"/>
     </joint>
@@ -110,5 +110,5 @@
       <parent link="front_tpl_revolute_hitch_base_right_link"/>
       <child link="front_tpl_revolute_hitch_effector_right_link"/>
-      <origin xyz="${0.4*(tpl_rev_hit_base_len+tpl_rev_hit_effector_len)} ${-0.22*tpl_rev_hit_effector_len} -0.1 " rpy="0 ${M_PI/6} ${-M_PI/6}"/>
+      <origin xyz="${0.43*(tpl_rev_hit_base_len+tpl_rev_hit_effector_len)} ${-0.28*tpl_rev_hit_effector_len} -0.12 " rpy="0 ${M_PI/6} ${-M_PI/6}"/>
       <axis xyz="0 0 1"/>
     </joint>
@@ -124,5 +124,5 @@
       <parent link="front_tpl_revolute_hitch_base_left_link"/>
       <child link="front_tpl_revolute_hitch_effector_left_link"/>
-      <origin xyz="${0.4*(tpl_rev_hit_base_len+tpl_rev_hit_effector_len)} ${-0.22*tpl_rev_hit_effector_len} 0.1" rpy="0 ${-M_PI/6} ${-M_PI/6}"/>
+      <origin xyz="${0.43*(tpl_rev_hit_base_len+tpl_rev_hit_effector_len)} ${-0.28*tpl_rev_hit_effector_len} 0.12" rpy="0 ${-M_PI/6} ${-M_PI/6}"/>
       <axis xyz="0 0 1"/>
     </joint>

File: urdf/basic_links/tpl/tpl_base.xacro (robot description, xacro)
@@ -1,4 +1,4 @@
 <robot name="tpl_assembled" xmlns:xacro="http://ros.org/wiki/xacro">
-  <xacro:property name="tpl_base_len" value="0.43" />
+  <xacro:property name="tpl_base_len" value="0.64" />
   <xacro:property name="tpl_base_wid" value="0.3" />
   <xacro:property name="tpl_base_hei" value="0.05" />
@@ -14,5 +14,5 @@
         </xacro:if>
         <geometry>
-          <box size="${tpl_base_len} ${tpl_base_wid} ${tpl_base_hei}"/>
+          <box size="0 0 0"/>
         </geometry>
       </visual>

File: urdf/basic_links/tpl/tpl_cyl.xacro (robot description, xacro)
@@ -7,11 +7,13 @@
       <visual>
         <xacro:if value="${name == 'back_tpl_cylinder_link'}">
+          <origin xyz="1.84 -0.68 -0.1" rpy="${M_PI/10} ${M_PI/2} 0"/>
           <material name="white"/>
         </xacro:if>
         <xacro:if value="${name == 'front_tpl_cylinder_link'}">
+          <origin xyz="-1.84 0.68 -0.1" rpy="${-M_PI+M_PI/10} ${M_PI/2} 0"/>
           <material name="green"/>
         </xacro:if>
         <geometry>
-          <cylinder length="${tpl_cyl_width}" radius="${tpl_cyl_radius}"/>
+          <mesh filename="package://agribot_description/meshes/lower_hitches.stl" scale="0.00105 0.00105 0.00105"/>
         </geometry>
       </visual>

File: urdf/basic_links/tpl/tpl_rev_hit_base.xacro (robot description, xacro)
@@ -20,5 +20,5 @@
         </xacro:if>
         <geometry>
-          <box size="${tpl_rev_hit_base_len} ${tpl_rev_hit_base_wid} ${tpl_rev_hit_base_hei}"/>
+          <box size="0 0 0"/>
         </geometry>
       </visual>

File: urdf/basic_links/tpl/tpl_rev_hit_effector.xacro (robot description, xacro)
@@ -1,5 +1,5 @@
 <robot name="tpl_assembled" xmlns:xacro="http://ros.org/wiki/xacro">
-    <xacro:property name="tpl_rev_hit_effector_len" value="0.5" />
-    <xacro:property name="tpl_rev_hit_effector_wid" value="${2*tpl_base_hei}" />
+    <xacro:property name="tpl_rev_hit_effector_len" value="0.55" />
+    <xacro:property name="tpl_rev_hit_effector_wid" value="${3.5*tpl_base_hei}" />
     <xacro:property name="tpl_rev_hit_effector_hei" value="0.05" />
     <xacro:property name="tpl_rev_hit_effector_mass" value="25.0" />
@@ -20,5 +20,5 @@
           </xacro:if>
           <geometry>
-            <box size="${tpl_rev_hit_effector_len} ${tpl_rev_hit_effector_wid} ${tpl_rev_hit_effector_hei}"/>
+            <box size="0 0 0"/>
           </geometry>
         </visual>

File: urdf/basic_links/tpl/tpl_upper_hit_base.xacro (robot description, xacro)
@@ -14,5 +14,5 @@
           </xacro:if>
           <geometry>
-            <box size="${tpl_upper_hit_base_len} ${tpl_upper_hit_base_wid} ${tpl_upper_hit_base_hei}"/>
+            <box size="0 0 0"/>
           </geometry>
         </visual>

File: urdf/basic_links/tpl/tpl_upper_hit_base_cyl.xacro (robot description, xacro)
@@ -13,5 +13,5 @@
           </xacro:if>
           <geometry>
-            <cylinder length="${tpl_upper_hit_base_cyl_width}" radius="${tpl_upper_hit_base_cyl_radius}"/>
+            <cylinder length="0" radius="0"/>
           </geometry>
         </visual>

File: urdf/basic_links/tpl/tpl_upper_hitch_prism_base.xacro (robot description, xacro)
@@ -1,6 +1,6 @@
 <robot name="tpl_assembled" xmlns:xacro="http://ros.org/wiki/xacro">
     <xacro:property name="tpl_upper_hitch_prism_base_len" value="0.5" />
-    <xacro:property name="tpl_upper_hitch_prism_base_wid" value="0.075" />
-    <xacro:property name="tpl_upper_hitch_prism_base_hei" value="0.075" />
+    <xacro:property name="tpl_upper_hitch_prism_base_wid" value="0.05" />
+    <xacro:property name="tpl_upper_hitch_prism_base_hei" value="0.05" />
     <xacro:property name="tpl_upper_hitch_prism_base_mass" value="10.0" />
     <xacro:macro name="agribot_tpl_upper_hitch_prism_joint_base" params="name">

File: urdf/basic_links/tpl/tpl_upper_hitch_prism_core.xacro (robot description, xacro)
@@ -1,6 +1,6 @@
 <robot name="tpl_assembled" xmlns:xacro="http://ros.org/wiki/xacro">
     <xacro:property name="tpl_upper_hitch_prism_core_len" value="0.5" />
-    <xacro:property name="tpl_upper_hitch_prism_core_wid" value="0.05" />
-    <xacro:property name="tpl_upper_hitch_prism_core_hei" value="0.05" />
+    <xacro:property name="tpl_upper_hitch_prism_core_wid" value="0.025" />
+    <xacro:property name="tpl_upper_hitch_prism_core_hei" value="0.025" />
     <xacro:property name="tpl_upper_hitch_prism_core_mass" value="8.0" />
     <xacro:macro name="agribot_tpl_upper_hitch_prism_joint_core" params="name">

Commit message: read wheel_radius and chassis_width from params in cart.xacro

File: urdf/basic_links/cart.xacro (robot description, xacro)
@@ -1,6 +1,6 @@
 <robot name="base" xmlns:xacro="http://ros.org/wiki/xacro">
-    <xacro:property name="cart_lenght" value="${wheel_radius*2}" />
-    <xacro:property name="cart_width" value="${chassis_width}" />
-    <xacro:property name="cart_height" value="${wheel_radius*2}" />
+    <xacro:property name="cart_lenght" value="${param_dimension['wheel_radius']*2}" />
+    <xacro:property name="cart_width" value="${param_dimension['chassis_width']}" />
+    <xacro:property name="cart_height" value="${param_dimension['wheel_radius']*2}" />
     <xacro:property name="cart_mass" value="500" />
     <xacro:macro name="agribot_cart" params="name">
