Commit message: Inertia values adding in progress

File: urdf/basic_links/tpl.xacro (robot description, xacro)
@@ -54,7 +54,7 @@
           <!-- https://en.wikipedia.org/wiki/List_of_moments_of_inertia#List_of_3D_inertia_tensors-->
           <mass value="${tpl_base_mass}"/>
-          <inertia ixx="0.0" ixy="0.0" ixz="0.0"
-                   iyy="0.0" iyz="0.0"
-                   izz="0.0" />
+          <inertia ixx="${tpl_base_mass*(tpl_base_hei*tpl_base_hei+tpl_base_wid*tpl_base_wid)/12}" ixy="0.0" ixz="0.0"
+                   iyy="${tpl_base_mass*(tpl_base_len*tpl_base_len+tpl_base_hei*tpl_base_hei)/12}" iyz="0.0"
+                   izz="${tpl_base_mass*(tpl_base_len*tpl_base_len+tpl_base_wid*tpl_base_wid)/12}" />
         </inertial>
       </link>
@@ -89,7 +89,7 @@
           <!-- https://en.wikipedia.org/wiki/List_of_moments_of_inertia#List_of_3D_inertia_tensors-->
           <mass value="${tpl_cyl_mass}"/>
-          <inertia ixx="0.0" ixy="0.0" ixz="0.0"
-                   iyy="0.0" iyz="0.0"
-                   izz="0.0" />
+            <inertia ixx="${tpl_cyl_mass*(3*tpl_cyl_radius*tpl_cyl_radius+tpl_cyl_width*tpl_cyl_width)/12}" ixy="0.0" ixz="0.0"
+                     iyy="${tpl_cyl_mass*(3*tpl_cyl_radius*tpl_cyl_radius+tpl_cyl_width*tpl_cyl_width)/12}" iyz="0.0"
+                     izz="${tpl_cyl_mass*(tpl_cyl_radius*tpl_cyl_radius)/2}" />
         </inertial>
       </link>

Commit message: Modified macro to work with front and back TPL

File: urdf/basic_links/tpl.xacro (robot description, xacro)
@@ -1,3 +1,3 @@
-<robot name="base" xmlns:xacro="http://ros.org/wiki/xacro">
+<robot name="tpl" xmlns:xacro="http://ros.org/wiki/xacro">
   <xacro:include filename="$(find agribot_description)/urdf/basic_links/tpl/tpl_base.xacro"/>
   <xacro:include filename="$(find agribot_description)/urdf/basic_links/tpl/tpl_cyl.xacro"/>
@@ -26,5 +26,10 @@
       <parent link="${name}_cylinder_link"/>
       <child link="${name}_revolute_hitch_base_right_link"/>
-      <origin xyz="${(tpl_rev_hit_base_len-tpl_cyl_radius)/2} 0.0 ${-(tpl_cyl_width)/2}" rpy="0 0 0"/>
+      <xacro:if value="${name == 'back_tpl'}">
+        <origin xyz="${-(tpl_rev_hit_base_len-tpl_cyl_radius)/2} 0.0 ${(tpl_cyl_width)/2}" rpy="0 0 0"/>
+      </xacro:if>
+      <xacro:if value="${name == 'front_tpl'}">
+        <origin xyz="${(tpl_rev_hit_base_len-tpl_cyl_radius)/2} 0.0 ${-(tpl_cyl_width)/2}" rpy="0 0 0"/>
+      </xacro:if>
       <axis xyz="0 0 1"/>
     </joint>
@@ -33,5 +38,10 @@
       <parent link="${name}_revolute_hitch_base_right_link"/>
       <child link="${name}_revolute_hitch_effector_right_link"/>
-      <origin xyz="${0.43*(tpl_rev_hit_base_len+tpl_rev_hit_effector_len)} ${-0.28*tpl_rev_hit_effector_len} -0.12 " rpy="0 ${M_PI/6} ${-M_PI/6}"/>
+      <xacro:if value="${name == 'back_tpl'}">
+        <origin xyz="${-0.43*(tpl_rev_hit_base_len+tpl_rev_hit_effector_len)} 0.12 ${0.28*tpl_rev_hit_effector_len}" rpy="0 ${M_PI/6} ${-M_PI/6}"/>
+      </xacro:if>
+      <xacro:if value="${name == 'front_tpl'}">
+        <origin xyz="${0.43*(tpl_rev_hit_base_len+tpl_rev_hit_effector_len)} ${-0.28*tpl_rev_hit_effector_len} -0.12 " rpy="0 ${M_PI/6} ${-M_PI/6}"/>
+      </xacro:if>
       <axis xyz="0 0 1"/>
     </joint>
@@ -40,5 +50,10 @@
       <parent link="${name}_cylinder_link"/>
       <child link="${name}_revolute_hitch_base_left_link"/>
-      <origin xyz="${(tpl_rev_hit_base_len-tpl_cyl_radius)/2} 0.0 ${(tpl_cyl_width)/2}" rpy="0 0 0"/>
+      <xacro:if value="${name == 'back_tpl'}">
+        <origin xyz="${-(tpl_rev_hit_base_len-tpl_cyl_radius)/2} 0.0 ${-(tpl_cyl_width)/2}" rpy="0 0 0"/>
+      </xacro:if>
+      <xacro:if value="${name == 'front_tpl'}">
+        <origin xyz="${(tpl_rev_hit_base_len-tpl_cyl_radius)/2} 0.0 ${(tpl_cyl_width)/2}" rpy="0 0 0"/>
+      </xacro:if>
       <axis xyz="0 0 1"/>
     </joint>
@@ -47,5 +62,10 @@
       <parent link="${name}_revolute_hitch_base_left_link"/>
       <child link="${name}_revolute_hitch_effector_left_link"/>
-      <origin xyz="${0.43*(tpl_rev_hit_base_len+tpl_rev_hit_effector_len)} ${-0.28*tpl_rev_hit_effector_len} 0.12" rpy="0 ${-M_PI/6} ${-M_PI/6}"/>
+      <xacro:if value="${name == 'back_tpl'}">
+        <origin xyz="${-0.43*(tpl_rev_hit_base_len+tpl_rev_hit_effector_len)} 0.12 ${-0.28*tpl_rev_hit_effector_len}" rpy="0 ${-M_PI/6} ${-M_PI/6}"/>
+      </xacro:if>
+      <xacro:if value="${name == 'front_tpl'}">
+        <origin xyz="${0.43*(tpl_rev_hit_base_len+tpl_rev_hit_effector_len)} ${-0.28*tpl_rev_hit_effector_len} 0.12" rpy="0 ${-M_PI/6} ${-M_PI/6}"/>
+      </xacro:if>
       <axis xyz="0 0 1"/>
     </joint>
@@ -54,5 +74,10 @@
       <parent link="${name}_base_link"/>
       <child link="${name}_up_hit_base_link"/>
-      <origin xyz="${0.82*tpl_base_len} 0.0 ${0.8*(tpl_upper_hit_base_len)/2}" rpy="0 ${-M_PI/3.15} 0"/>
+      <xacro:if value="${name == 'back_tpl'}">
+        <origin xyz="${-0.78*tpl_base_len} 0.0 ${0.8*(tpl_upper_hit_base_len)/2}" rpy="0 ${M_PI/3.43} 0"/>
+      </xacro:if>
+      <xacro:if value="${name == 'front_tpl'}">
+        <origin xyz="${0.82*tpl_base_len} 0.0 ${0.8*(tpl_upper_hit_base_len)/2}" rpy="0 ${-M_PI/3.15} 0"/>
+      </xacro:if>
       <axis xyz="0 0 1"/>
     </joint>
@@ -61,5 +86,10 @@
       <parent link="${name}_up_hit_base_link"/>
       <child link="${name}_upper_hitch_cylinder_link"/>
-      <origin xyz="${tpl_upper_hit_base_len/2} 0.0 0.0" rpy="${-M_PI/2} ${M_PI/18+M_PI} 0"/>
+      <xacro:if value="${name == 'back_tpl'}">
+        <origin xyz="${-tpl_upper_hit_base_len/2} 0.0 0.0" rpy="${M_PI/2} ${-M_PI/18} 0"/>
+      </xacro:if>
+      <xacro:if value="${name == 'front_tpl'}">
+        <origin xyz="${tpl_upper_hit_base_len/2} 0.0 0.0" rpy="${-M_PI/2} ${M_PI/18+M_PI} 0"/>
+      </xacro:if>
       <limit lower="${-10*M_PI/180}" upper="${80*M_PI/180}"  effort="1000.0" velocity="1000.0"/>
       <axis xyz="0 0 1"/>

Commit message: Not shaking version

File: urdf/basic_links/tpl.xacro (robot description, xacro)
@@ -23,5 +23,4 @@
     </joint>
     <xacro:agribot_tpl_cylinder name="${name}_cylinder_link" />
-<!--
     <joint name="${name}_revolute_hitch_base_left_joint" type="fixed">
       <parent link="${name}_cylinder_link"/>
@@ -72,5 +71,4 @@
     </joint>
     <xacro:agribot_tpl_revolute_hitch_effector name="${name}_revolute_hitch_effector_left_link" />
--->
     <joint name="${name}_upper_hich_base_joint" type="fixed">
       <parent link="${name}_base_link"/>

File: urdf/basic_links/tpl/tpl_rev_hit_base.xacro (robot description, xacro)
@@ -3,5 +3,5 @@
   <xacro:property name="tpl_rev_hit_base_wid" value="${2*tpl_base_hei}" />
   <xacro:property name="tpl_rev_hit_base_hei" value="0.05" />
-  <xacro:property name="tpl_rev_hit_base_mass" value="20" />
+  <xacro:property name="tpl_rev_hit_base_mass" value="20.0" />
   <xacro:macro name="agribot_tpl_revolute_hitch_base" params="name">
     <link name="${name}">

Commit message: Extended joint limits for control purposes

File: urdf/basic_links/tpl.xacro (robot description, xacro)
@@ -19,5 +19,5 @@
         <origin xyz="${(tpl_base_len)/2} 0.0 0.0" rpy="${-M_PI/2} ${M_PI/5} 0"/>
       </xacro:if>
-      <limit lower="${-90*M_PI/180}" upper="${15*M_PI/180}"  effort="1000.0" velocity="1000.0"/>
+      <limit lower="${-90*M_PI/180}" upper="${90*M_PI/180}"  effort="1000.0" velocity="1000.0"/>
       <axis xyz="0 0 1"/>
     </joint>

Commit message: Changed limits for those measured from robot

File: urdf/basic_links/tpl.xacro (robot description, xacro)
@@ -19,5 +19,5 @@
         <origin xyz="${(tpl_base_len)/2} 0.0 0.0" rpy="${-M_PI/2} ${M_PI/5} 0"/>
       </xacro:if>
-      <limit lower="${-90*M_PI/180}" upper="${90*M_PI/180}"  effort="1000.0" velocity="1000.0"/>
+      <limit lower="-0.03" upper="0.9"  effort="1000.0" velocity="1000.0"/>
       <axis xyz="0 0 1"/>
     </joint>
@@ -106,5 +106,5 @@
       <parent link="${name}_upper_hitch_prism_joint_base_link"/>
       <child link="${name}_upper_hitch_prism_joint_core_link"/>
-      <limit effort="1000.0" lower="${-tpl_upper_hitch_prism_core_len+0.05}" upper="0.0" velocity="0.5"/>
+      <limit effort="1000.0" lower="0.0" upper="0.25" velocity="0.5"/>
       <origin rpy="0 0 0" xyz="-0.05 0 0"/>
     </joint>
