Commit message: Adjust zed2 position

File: urdf/perception_sensors/perception_suites/livox_zed2_set.xacro (robot description, xacro)
@@ -11,5 +11,6 @@
                           perception_plugins:=^
                          ">
-    <!-- This link is "origin" of the livox_zed2_set and ia assumed to be  -->
+    <!-- This link is "origin" of the livox_zed2_set and ia assumed to be at the
+      (x axis - front, y axis - center, z axis - bottom) of the lidar  -->
     <link name="${suite_name}_link" />
     <joint name="livox_zed2_set" type="fixed">
@@ -27,6 +28,10 @@
     </xacro:livox_horizon>
     <!-- ZED2 camera -->
+    <xacro:property name="livox_height" value="0.0841" />
+    <xacro:property name="plate_height" value="0.0102" />
+    <xacro:property name="zed2_height" value="0.03" />
+    <xacro:property name="suite_base_to_zed2_center_z" value="${livox_height + plate_height + zed2_height/2}" />
     <xacro:zed2>
-      <origin xyz="-0.05 0 0.0571" rpy="0 0 0" />
+      <origin xyz="-0.018 0 ${suite_base_to_zed2_center_z}" rpy="0 0 0" />
       <xacro:property name="parent" value="${suite_name}_link" />
       <xacro:property name="camera_name" value="zed2" />

Commit message: Add livox pitch offset

File: urdf/perception_sensors/perception_suites/livox_zed2_set.xacro (robot description, xacro)
@@ -20,5 +20,6 @@
     </joint>
     <xacro:livox_horizon>
-      <origin xyz="0 0 0" rpy="0 0 0" />
+    <!-- TODO(olek) - monitor if this pitch offset (-2.5deg) is necessary  -->
+    <origin xyz="0 0 0" rpy="0 ${-2.5*M_PI/180.0} 0" />
       <xacro:property name="parent" value="${suite_name}_link" />
       <xacro:property name="topic" value="${livox_topic}" />
