Commit message: Fixed cloud point position to fit optical frame

File: urdf/perception_sensors/camera/zed2.xacro (robot description, xacro)
@@ -52,4 +52,10 @@
     </joint>
     <link name="${camera_name}_right_camera_optical_frame" />
+     <joint name="${camera_name}_center_camera_optical_joint" type="fixed">
+      <origin xyz="0 0 0" rpy="-${M_PI/2} 0.0 -${M_PI/2}" />
+      <parent link="${camera_name}_camera_center" />
+      <child link="${camera_name}_center_camera_optical_frame" />
+    </joint>
+    <link name="${camera_name}_center_camera_optical_frame" />
     <!-- ZED2 Sensors -->
     <joint name="${camera_name}_mag_joint" type="fixed">
@@ -82,4 +88,5 @@
         <camera>
           <horizontal_fov>1.047198</horizontal_fov>
+          <vertical_fov></vertical_fov>
           <image>
             <width>640</width>
@@ -102,5 +109,5 @@
           <depthImageInfoTopicName>/${camera_name}/depth/camera_info</depthImageInfoTopicName>
           <pointCloudTopicName>/${camera_name}/depth/points</pointCloudTopicName>
-          <frameName>${camera_name}_camera_center</frameName>
+          <frameName>${camera_name}_center_camera_optical_frame</frameName>
           <pointCloudCutoff>0.2</pointCloudCutoff>
           <pointCloudCutoffMax>10.0</pointCloudCutoffMax>
